Commit message: separate controllers among base, arm, gripper

File: src/tidybot_description/urdf/ros2_control.xacro (robot description, xacro)
@@ -1,5 +1,5 @@
 <?xml version="1.0"?>
 <robot name="ros2_control" xmlns:xacro="http://ros.org/wiki/xacro">
-    <xacro:macro name="load_ros2_control" params="config_path">
+    <xacro:macro name="load_ros2_control" params="config_path hardware_plugin">
         <xacro:macro name="add_joint" params="name gain cmd_interface">
             <joint name="${name}">
@@ -12,5 +12,5 @@
         <ros2_control name="GazeboSystem" type="system">
         <hardware>
-            <plugin>gz_ros2_control/GazeboSimSystem</plugin>
+            <plugin>${hardware_plugin}</plugin>
         </hardware>
         <xacro:add_joint name="joint_x" gain="0.1" cmd_interface="velocity"/>

File: src/tidybot_description/urdf/tidybot.xacro (robot description, xacro)
@@ -1,4 +1,5 @@
 <?xml version="1.0"?>
 <robot name="tidybot" xmlns:xacro="http://ros.org/wiki/xacro">
+    <xacro:arg name="hardware_plugin" default="mock_components/GenericSystem" />
     <xacro:arg name="arm" default="gen3_lite" />
     <xacro:arg name="gripper" default="gen3_lite_2f" />
@@ -11,4 +12,4 @@
     <!-- configure ros2_control joints -->
     <xacro:include filename="$(find tidybot_description)/urdf/ros2_control.xacro" />
-    <xacro:load_ros2_control config_path="$(arg ros2_control_config_path)"/>
+    <xacro:load_ros2_control config_path="$(arg ros2_control_config_path)" hardware_plugin="$(arg hardware_plugin)" />
 </robot>

File: src/tidybot_moveit_config/config/tidybot.urdf.xacro (robot description, xacro)
@@ -2,8 +2,6 @@
 <robot xmlns:xacro="http://www.ros.org/wiki/xacro" name="tidybot">
     <xacro:arg name="initial_positions_file" default="initial_positions.yaml" />
+    <xacro:arg name="ros2_control_config_path" default="$(find tidybot_description)/config/tidybot_controllers.yaml"/>
     <!-- Import tidybot urdf file -->
     <xacro:include filename="$(find tidybot_description)/urdf/tidybot.xacro" />
-    <!-- Import control_xacro -->
-    <xacro:include filename="tidybot.ros2_control.xacro" />
-    <xacro:tidybot_ros2_control name="FakeSystem" initial_positions_file="$(arg initial_positions_file)"/>
 </robot>
