Commit message: fixed tidybot.xacro and drive.launch.py

File: src/tidybot_description/urdf/tidybot.xacro (robot description, xacro)
@@ -1,1006 +1,19 @@
-<?xml version="1.0" ?>
-<!-- =================================================================================== -->
-<!-- |    This document was autogenerated by xacro from tidybot.urdf                   | -->
-<!-- |    EDITING THIS FILE BY HAND IS NOT RECOMMENDED                                 | -->
-<!-- =================================================================================== -->
-<!-- =================================================================================== -->
-<!-- |    This document was autogenerated by xacro from tidybot.xacro                  | -->
-<!-- |    EDITING THIS FILE BY HAND IS NOT RECOMMENDED                                 | -->
-<!-- =================================================================================== -->
-<robot name="tidybot">
-  <!-- <xacro:load_base prefix=""/> -->
-  <link name="world"/>
-  <link name="base">
-    <inertial>
-      <origin rpy="0.0 0.0 0.0" xyz="0.0 0.0 0.035"/>
-      <mass value="60.0"/>
-      <inertia ixx="0.001" ixy="0" ixz="0" iyy="0.001" iyz="0" izz="0.001"/>
-    </inertial>
-    <visual name="bumper">
-      <origin rpy="-2.442021632452952 -1.5707963267948966 0.0" xyz="-1.3915598211675165e-07 -2.058962502098711e-07 0.05386474576457055"/>
-      <geometry>
-        <mesh filename="file:///home/janchen/Documents/tidybot_platform/install/tidybot_description/share/tidybot_description/meshes/base/bumper.stl"/>
-      </geometry>
-      <material name="white"/>
-    </visual>
-    <collision name="bumper">
-      <origin rpy="-2.442021632452952 -1.5707963267948966 0.0" xyz="-1.3915598211675165e-07 -2.058962502098711e-07 0.05386474576457055"/>
-      <geometry>
-        <mesh filename="file:///home/janchen/Documents/tidybot_platform/install/tidybot_description/share/tidybot_description/meshes/base/bumper.stl"/>
-      </geometry>
-    </collision>
-    <visual name="bottom_plate">
-      <origin rpy="1.6659662035857206 -1.5707963267948966 0.0" xyz="4.155854111430312e-11 1.8201972332496634e-11 0.08495000004768373"/>
-      <geometry>
-        <mesh filename="file:///home/janchen/Documents/tidybot_platform/install/tidybot_description/share/tidybot_description/meshes/base/bottom_plate.stl"/>
-      </geometry>
-      <material name="white"/>
-    </visual>
-    <collision name="bottom_plate">
-      <origin rpy="1.6659662035857206 -1.5707963267948966 0.0" xyz="4.155854111430312e-11 1.8201972332496634e-11 0.08495000004768373"/>
-      <geometry>
-        <mesh filename="file:///home/janchen/Documents/tidybot_platform/install/tidybot_description/share/tidybot_description/meshes/base/bottom_plate.stl"/>
-      </geometry>
-    </collision>
-    <visual name="body">
-      <origin rpy="-1.5707963267948966 -1.570779305272103 3.141592653589793" xyz="7.590768644441668e-06 -6.000635064190085e-10 0.20330222068596052"/>
-      <geometry>
-        <mesh filename="file:///home/janchen/Documents/tidybot_platform/install/tidybot_description/share/tidybot_description/meshes/base/body.stl"/>
-      </geometry>
-      <material name="white"/>
-    </visual>
-    <collision name="body">
-      <origin rpy="-1.5707963267948966 -1.570779305272103 3.141592653589793" xyz="7.590768644441668e-06 -6.000635064190085e-10 0.20330222068596052"/>
-      <geometry>
-        <mesh filename="file:///home/janchen/Documents/tidybot_platform/install/tidybot_description/share/tidybot_description/meshes/base/body.stl"/>
-      </geometry>
-    </collision>
-    <visual name="top_plate">
-      <origin rpy="1.6906681075416252 -1.5707963267948966 0.0" xyz="-2.9658670629084936e-11 -3.476524862019053e-11 0.3216499984264373"/>
-      <geometry>
-        <mesh filename="file:///home/janchen/Documents/tidybot_platform/install/tidybot_description/share/tidybot_description/meshes/base/top_plate.stl"/>
-      </geometry>
-      <material name="white"/>
-    </visual>
-    <collision name="top_plate">
-      <origin rpy="1.6906681075416252 -1.5707963267948966 0.0" xyz="-2.9658670629084936e-11 -3.476524862019053e-11 0.3216499984264373"/>
-      <geometry>
-        <mesh filename="file:///home/janchen/Documents/tidybot_platform/install/tidybot_description/share/tidybot_description/meshes/base/top_plate.stl"/>
-      </geometry>
-    </collision>
-    <visual name="arm_plate">
-      <origin rpy="1.5707963267948966 -1.5707963267948966 0.0" xyz="-2.7580994002430455e-12 -3.3382504263355704e-12 0.32999999883475684"/>
-      <geometry>
-        <mesh filename="file:///home/janchen/Documents/tidybot_platform/install/tidybot_description/share/tidybot_description/meshes/base/arm_plate.stl"/>
-      </geometry>
-      <material name="white"/>
-    </visual>
-    <collision name="arm_plate">
-      <origin rpy="1.5707963267948966 -1.5707963267948966 0.0" xyz="-2.7580994002430455e-12 -3.3382504263355704e-12 0.32999999883475684"/>
-      <geometry>
-        <mesh filename="file:///home/janchen/Documents/tidybot_platform/install/tidybot_description/share/tidybot_description/meshes/base/arm_plate.stl"/>
-      </geometry>
-    </collision>
-  </link>
-  <link name="joint_x_jointbody">
-    <inertial>
-      <origin rpy="0.0 0.0 0.0" xyz="0.0 0.0 0.0"/>
-      <mass value="0.001"/>
-      <inertia ixx="1e-09" ixy="0" ixz="0" iyy="1e-09" iyz="0" izz="1e-09"/>
-    </inertial>
-  </link>
-  <joint name="joint_x" type="prismatic">
-    <origin rpy="0.0 0.0 0.0" xyz="0.0 0.0 0.0"/>
-    <parent link="world"/>
-    <child link="joint_x_jointbody"/>
-    <axis xyz="1 0 0"/>
-    <limit effort="100" lower="-10.0" upper="10.0" velocity="1"/>
-    <dynamics damping="1.0" friction="1.0"/>
-  </joint>
-  <link name="joint_y_jointbody">
-    <inertial>
-      <origin rpy="0.0 0.0 0.0" xyz="0.0 0.0 0.0"/>
-      <mass value="0.001"/>
-      <inertia ixx="1e-09" ixy="0" ixz="0" iyy="1e-09" iyz="0" izz="1e-09"/>
-    </inertial>
-  </link>
-  <joint name="joint_y" type="prismatic">
-    <origin rpy="0.0 0.0 0.0" xyz="0.0 0.0 0.0"/>
-    <parent link="joint_x_jointbody"/>
-    <child link="joint_y_jointbody"/>
-    <axis xyz="0 1 0"/>
-    <limit effort="100" lower="-10.0" upper="10.0" velocity="1"/>
-    <dynamics damping="1.0" friction="1.0"/>
-  </joint>
-  <link name="joint_th_jointbody">
-    <inertial>
-      <origin rpy="0.0 0.0 0.0" xyz="0.0 0.0 0.0"/>
-      <mass value="0.001"/>
-      <inertia ixx="1e-09" ixy="0" ixz="0" iyy="1e-09" iyz="0" izz="1e-09"/>
-    </inertial>
-  </link>
-  <joint name="joint_th" type="revolute">
-    <origin rpy="0.0 0.0 0.0" xyz="0.0 0.0 0.0"/>
-    <parent link="joint_y_jointbody"/>
-    <child link="joint_th_jointbody"/>
-    <axis xyz="0.0 0.0 1.0"/>
-    <limit effort="100" lower="-10" upper="10" velocity="1"/>
-    <dynamics damping="1.0" friction="1.0"/>
-  </joint>
-  <joint name="joint_th_offset" type="fixed">
-    <origin rpy="0.0 0.0 0.0" xyz="-0.0 -0.0 -0.0"/>
-    <parent link="joint_th_jointbody"/>
-    <child link="base"/>
-    <axis xyz="0.0 0.0 1.0"/>
-    <limit effort="100" lower="0.0" upper="0.0" velocity="100"/>
-  </joint>
-  <material name="white">
-    <color rgba="1 1 1 1"/>
-  </material>
-  <joint name="arm_base_joint" type="fixed">
-    <origin rpy="0 0 0" xyz="0 0 0.33"/>
-    <parent link="base"/>
-    <child link="arm_base_link"/>
-  </joint>
-  <link name="arm_base_link">
-    <inertial>
-      <origin rpy="0 0 0" xyz="-0.000648 -0.000166 0.084487"/>
-      <mass value="1.697"/>
-      <inertia ixx="0.004622" ixy="9E-06" ixz="6E-05" iyy="0.004495" iyz="9E-06" izz="0.002079"/>
-    </inertial>
-    <visual>
-      <origin rpy="0 0 0" xyz="0 0 0"/>
-      <geometry>
-        <mesh filename="file:///home/janchen/Documents/tidybot_platform/install/tidybot_description/share/tidybot_description/meshes/arms/gen3_7dof/base_link.STL"/>
-      </geometry>
-      <material name="">
-        <color rgba="0.75294 0.75294 0.75294 1"/>
-      </material>
-    </visual>
-    <collision>
-      <origin rpy="0 0 0" xyz="0 0 0"/>
-      <geometry>
-        <mesh filename="file:///home/janchen/Documents/tidybot_platform/install/tidybot_description/share/tidybot_description/meshes/arms/gen3_7dof/base_link.STL"/>
-      </geometry>
-    </collision>
-  </link>
-  <gazebo reference="arm_base_link">
-    <material>Gazebo/Gray</material>
-  </gazebo>
-  <link name="shoulder_link">
-    <inertial>
-      <origin rpy="0 0 0" xyz="-2.3E-05 -0.010364 -0.07336"/>
-      <mass value="1.3773"/>
-      <inertia ixx="0.00457" ixy="1E-06" ixz="2E-06" iyy="0.004831" iyz="0.000448" izz="0.001409"/>
-    </inertial>
-    <visual>
-      <origin rpy="0 0 0" xyz="0 0 0"/>
-      <geometry>
-        <mesh filename="file:///home/janchen/Documents/tidybot_platform/install/tidybot_description/share/tidybot_description/meshes/arms/gen3_7dof/shoulder_link.STL"/>
-      </geometry>
-      <material name="">
-        <color rgba="0.75294 0.75294 0.75294 1"/>
-      </material>
-    </visual>
-    <collision>
-      <origin rpy="0 0 0" xyz="0 0 0"/>
-      <geometry>
-        <mesh filename="file:///home/janchen/Documents/tidybot_platform/install/tidybot_description/share/tidybot_description/meshes/arms/gen3_7dof/shoulder_link.STL"/>
-      </geometry>
-    </collision>
-  </link>
-  <gazebo reference="shoulder_link">
-    <material>Gazebo/Gray</material>
-  </gazebo>
-  <joint name="joint_1" type="continuous">
-    <origin rpy="3.1416 2.7629E-18 -4.9305E-36" xyz="0 0 0.15643"/>
-    <parent link="arm_base_link"/>
-    <child link="shoulder_link"/>
-    <axis xyz="0 0 1"/>
-    <limit effort="39" velocity="1.3963"/>
-  </joint>
-  <link name="half_arm_1_link">
-    <inertial>
-      <origin rpy="0 0 0" xyz="-4.4E-05 -0.09958 -0.013278"/>
-      <mass value="1.1636"/>
-      <inertia ixx="0.011088" ixy="5E-06" ixz="0" iyy="0.001072" iyz="-0.000691" izz="0.011255"/>
-    </inertial>
-    <visual>
-      <origin rpy="0 0 0" xyz="0 0 0"/>
-      <geometry>
-        <mesh filename="file:///home/janchen/Documents/tidybot_platform/install/tidybot_description/share/tidybot_description/meshes/arms/gen3_7dof/half_arm_1_link.STL"/>
-      </geometry>
-      <material name="">
-        <color rgba="0.75294 0.75294 0.75294 1"/>
-      </material>
-    </visual>
-    <collision>
-      <origin rpy="0 0 0" xyz="0 0 0"/>
-      <geometry>
-        <mesh filename="file:///home/janchen/Documents/tidybot_platform/install/tidybot_description/share/tidybot_description/meshes/arms/gen3_7dof/half_arm_1_link.STL"/>
-      </geometry>
-    </collision>
-  </link>
-  <gazebo reference="half_arm_1_link">
-    <material>Gazebo/Gray</material>
-  </gazebo>
-  <joint name="joint_2" type="revolute">
-    <origin rpy="1.5708 2.1343E-17 -1.1102E-16" xyz="0 0.005375 -0.12838"/>
-    <parent link="shoulder_link"/>
-    <child link="half_arm_1_link"/>
-    <axis xyz="0 0 1"/>
-    <limit effort="39" lower="-2.24" upper="2.24" velocity="1.3963"/>
-  </joint>
-  <link name="half_arm_2_link">
-    <inertial>
-      <origin rpy="0 0 0" xyz="-4.4E-05 -0.006641 -0.117892"/>
-      <mass value="1.1636"/>
-      <inertia ixx="0.010932" ixy="0" ixz="-7E-06" iyy="0.011127" iyz="0.000606" izz="0.001043"/>
-    </inertial>
-    <visual>
-      <origin rpy="0 0 0" xyz="0 0 0"/>
-      <geometry>
-        <mesh filename="file:///home/janchen/Documents/tidybot_platform/install/tidybot_description/share/tidybot_description/meshes/arms/gen3_7dof/half_arm_2_link.STL"/>
-      </geometry>
-      <material name="">
-        <color rgba="0.75294 0.75294 0.75294 1"/>
-      </material>
-    </visual>
-    <collision>
-      <origin rpy="0 0 0" xyz="0 0 0"/>
-      <geometry>
-        <mesh filename="file:///home/janchen/Documents/tidybot_platform/install/tidybot_description/share/tidybot_description/meshes/arms/gen3_7dof/half_arm_2_link.STL"/>
-      </geometry>
-    </collision>
-  </link>
-  <gazebo reference="half_arm_2_link">
-    <material>Gazebo/Gray</material>
-  </gazebo>
-  <joint name="joint_3" type="continuous">
-    <origin rpy="-1.5708 1.2326E-32 -2.9122E-16" xyz="0 -0.21038 -0.006375"/>
-    <parent link="half_arm_1_link"/>
-    <child link="half_arm_2_link"/>
-    <axis xyz="0 0 1"/>
-    <limit effort="39" velocity="1.3963"/>
-  </joint>
-  <link name="forearm_link">
-    <inertial>
-      <origin rpy="0 0 0" xyz="-1.8E-05 -0.075478 -0.015006"/>
-      <mass value="0.9302"/>
-      <inertia ixx="0.008147" ixy="-1E-06" ixz="0" iyy="0.000631" iyz="-0.0005" izz="0.008316"/>
-    </inertial>
-    <visual>
-      <origin rpy="0 0 0" xyz="0 0 0"/>
-      <geometry>
-        <mesh filename="file:///home/janchen/Documents/tidybot_platform/install/tidybot_description/share/tidybot_description/meshes/arms/gen3_7dof/forearm_link.STL"/>
-      </geometry>
-      <material name="">
-        <color rgba="0.75294 0.75294 0.75294 1"/>
-      </material>
-    </visual>
-    <collision>
-      <origin rpy="0 0 0" xyz="0 0 0"/>
-      <geometry>
-        <mesh filename="file:///home/janchen/Documents/tidybot_platform/install/tidybot_description/share/tidybot_description/meshes/arms/gen3_7dof/forearm_link.STL"/>
-      </geometry>
-    </collision>
-  </link>
-  <gazebo reference="forearm_link">
-    <material>Gazebo/Gray</material>
-  </gazebo>
-  <joint name="joint_4" type="revolute">
-    <origin rpy="1.5708 -6.6954E-17 -1.6653E-16" xyz="0 0.006375 -0.21038"/>
-    <parent link="half_arm_2_link"/>
-    <child link="forearm_link"/>
-    <axis xyz="0 0 1"/>
-    <limit effort="39" lower="-2.57" upper="2.57" velocity="1.3963"/>
-  </joint>
-  <link name="spherical_wrist_1_link">
-    <inertial>
-      <origin rpy="0 0 0" xyz="1E-06 -0.009432 -0.063883"/>
-      <mass value="0.6781"/>
-      <inertia ixx="0.001596" ixy="0" ixz="0" iyy="0.001607" iyz="0.000256" izz="0.000399"/>
-    </inertial>
-    <visual>
-      <origin rpy="0 0 0" xyz="0 0 0"/>
-      <geometry>
-        <mesh filename="file:///home/janchen/Documents/tidybot_platform/install/tidybot_description/share/tidybot_description/meshes/arms/gen3_7dof/spherical_wrist_1_link.STL"/>
-      </geometry>
-      <material name="">
-        <color rgba="0.75294 0.75294 0.75294 1"/>
-      </material>
-    </visual>
-    <collision>
-      <origin rpy="0 0 0" xyz="0 0 0"/>
-      <geometry>
-        <mesh filename="file:///home/janchen/Documents/tidybot_platform/install/tidybot_description/share/tidybot_description/meshes/arms/gen3_7dof/spherical_wrist_1_link.STL"/>
-      </geometry>
-    </collision>
-  </link>
-  <gazebo reference="spherical_wrist_1_link">
-    <material>Gazebo/Gray</material>
-  </gazebo>
-  <joint name="joint_5" type="continuous">
-    <origin rpy="-1.5708 2.2204E-16 -6.373E-17" xyz="0 -0.20843 -0.006375"/>
-    <parent link="forearm_link"/>
-    <child link="spherical_wrist_1_link"/>
-    <axis xyz="0 0 1"/>
-    <limit effort="9" velocity="1.2218"/>
-  </joint>
-  <link name="spherical_wrist_2_link">
-    <inertial>
-      <origin rpy="0 0 0" xyz="1E-06 -0.045483 -0.00965"/>
-      <mass value="0.6781"/>
-      <inertia ixx="0.001641" ixy="0" ixz="0" iyy="0.00041" iyz="-0.000278" izz="0.001641"/>
-    </inertial>
-    <visual>
-      <origin rpy="0 0 0" xyz="0 0 0"/>
-      <geometry>
-        <mesh filename="file:///home/janchen/Documents/tidybot_platform/install/tidybot_description/share/tidybot_description/meshes/arms/gen3_7dof/spherical_wrist_2_link.STL"/>
-      </geometry>
-      <material name="">
-        <color rgba="0.75294 0.75294 0.75294 1"/>
-      </material>
-    </visual>
-    <collision>
-      <origin rpy="0 0 0" xyz="0 0 0"/>
-      <geometry>
-        <mesh filename="file:///home/janchen/Documents/tidybot_platform/install/tidybot_description/share/tidybot_description/meshes/arms/gen3_7dof/spherical_wrist_2_link.STL"/>
-      </geometry>
-    </collision>
-  </link>
-  <gazebo reference="spherical_wrist_2_link">
-    <material>Gazebo/Gray</material>
-  </gazebo>
-  <joint name="joint_6" type="revolute">
-    <origin rpy="1.5708 9.2076E-28 -8.2157E-15" xyz="0 0.00017505 -0.10593"/>
-    <parent link="spherical_wrist_1_link"/>
-    <child link="spherical_wrist_2_link"/>
-    <axis xyz="0 0 1"/>
-    <limit effort="9" lower="-2.09" upper="2.09" velocity="1.2218"/>
-  </joint>
-  <link name="bracelet_link">
-    <inertial>
-      <origin rpy="0 0 0" xyz="0.000281 0.011402 -0.029798"/>
-      <mass value="0.5"/>
-      <inertia ixx="0.000587" ixy="3E-06" ixz="3E-06" iyy="0.000369" iyz="-0.000118" izz="0.000609"/>
-    </inertial>
-    <visual>
-      <origin rpy="0 0 0" xyz="0 0 0"/>
-      <geometry>
-        <mesh filename="file:///home/janchen/Documents/tidybot_platform/install/tidybot_description/share/tidybot_description/meshes/arms/gen3_7dof/bracelet_with_vision_link.STL"/>
-      </geometry>
-      <material name="">
-        <color rgba="0.75294 0.75294 0.75294 1"/>
-      </material>
-    </visual>
-    <collision>
-      <origin rpy="0 0 0" xyz="0 0 0"/>
-      <geometry>
-        <mesh filename="file:///home/janchen/Documents/tidybot_platform/install/tidybot_description/share/tidybot_description/meshes/arms/gen3_7dof/bracelet_with_vision_link.STL"/>
-      </geometry>
-    </collision>
-  </link>
-  <gazebo reference="bracelet_link">
-    <material>Gazebo/Gray</material>
-  </gazebo>
-  <joint name="joint_7" type="continuous">
-    <origin rpy="-1.5708 -5.5511E-17 9.6396E-17" xyz="0 -0.10593 -0.00017505"/>
-    <parent link="spherical_wrist_2_link"/>
-    <child link="bracelet_link"/>
-    <axis xyz="0 0 1"/>
-    <limit effort="9" velocity="1.2218"/>
-  </joint>
-  <link name="end_effector_link"/>
-  <joint name="end_effector" type="fixed">
-    <origin rpy="3.14159265358979 1.09937075168372E-32 0" xyz="0 0 -0.0615250000000001"/>
-    <parent link="bracelet_link"/>
-    <child link="end_effector_link"/>
-    <axis xyz="0 0 0"/>
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