Commit message: implement the reset_env function

File: src/tidybot_description/urdf/tidybot.gazebo.xacro (robot description, xacro)
@@ -5,7 +5,7 @@
       <plugin name="gz_ros2_control::GazeboSimROS2ControlPlugin" filename="gz_ros2_control-system">
           <parameters>${config_path}</parameters>
-          <robot_description_param>robot_description</robot_description_param>
+          <!-- <robot_description_param>robot_description</robot_description_param> -->
       </plugin>
-      <self_collide>true</self_collide>
+      <!-- <self_collide>true</self_collide> -->
   </gazebo>
   <gazebo>

File: src/tidybot_description/urdf/tidybot.ros2_control.xacro (robot description, xacro)
@@ -10,5 +10,5 @@
             </joint>
         </xacro:macro>
-        <ros2_control name="GazeboSystem" type="system">
+        <ros2_control name="TidybotSystem" type="system">
         <hardware>
             <plugin>${hardware_plugin}</plugin>

File: src/tidybot_description/urdf/tidybot.urdf (robot description, URDF)
Before this commit: robot tidybot, 18 links, 17 joints
Links:
- link arm_base_link: geometry collision mesh filename=file:///home/janchen/Documents/ros2/tidybot_ws/install/tidy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; visual mesh filename=file:///home/janchen/Documents/ros2/tidybot_ws/install/tidy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
- link arm_link: geometry collision mesh filename=file:///home/janchen/Documents/ros2/tidybot_ws/install/tidy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; visual mesh filename=file:///home/janchen/Documents/ros2/tidybot_ws/install/tidy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
- link base: geometry collision mesh filename=file:///home/janchen/Documents/ros2/tidybot_ws/install/tidy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; collision mesh filename=file:///home/janchen/Documents/ros2/tidybot_ws/install/tidy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
- link forearm_link: geometry collision mesh filename=file:///home/janchen/Documents/ros2/tidybot_ws/install/tidy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; visual mesh filename=file:///home/janchen/Documents/ros2/tidybot_ws/install/tidy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
- link gripper_base_link: geometry visual mesh filename=file:///home/janchen/Documents/ros2/tidybot_ws/install/tidy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
- link left_finger_dist_link: geometry visual mesh filename=file:///home/janchen/Documents/ros2/tidybot_ws/install/tidy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
- link left_finger_prox_link: geometry visual mesh filename=file:///home/janchen/Documents/ros2/tidybot_ws/install/tidy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
- link lower_wrist_link: geometry collision mesh filename=file:///home/janchen/Documents/ros2/tidybot_ws/install/tidy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; visual mesh filename=file:///home/janchen/Documents/ros2/tidybot_ws/install/tidy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
- link right_finger_dist_link: geometry visual mesh filename=file:///home/janchen/Documents/ros2/tidybot_ws/install/tidy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
- link right_finger_prox_link: geometry visual mesh filename=file:///home/janchen/Documents/ros2/tidybot_ws/install/tidy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
- link shoulder_link: geometry collision mesh filename=file:///home/janchen/Documents/ros2/tidybot_ws/install/tidy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; visual mesh filename=file:///home/janchen/Documents/ros2/tidybot_ws/install/tidy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
- link upper_wrist_link: geometry collision mesh filename=file:///home/janchen/Documents/ros2/tidybot_ws/install/tidy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; visual mesh filename=file:///home/janchen/Documents/ros2/tidybot_ws/install/tidy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

File: src/tidybot_description/urdf/tidybot.xacro (robot description, xacro)
@@ -1,5 +1,6 @@
 <?xml version="1.0"?>
 <robot name="tidybot" xmlns:xacro="http://ros.org/wiki/xacro">
-    <xacro:arg name="hardware_plugin" default="mock_components/GenericSystem" />
+    <!-- <xacro:arg name="hardware_plugin" default="mock_components/GenericSystem" />     -->
+    <xacro:arg name="hardware_plugin" default="gz_ros2_control/GazeboSimSystem" />
     <xacro:arg name="arm" default="gen3_lite" />
     <xacro:arg name="gripper" default="gen3_lite_2f" />

Commit message: add openvla action node

File: src/tidybot_description/urdf/tidybot.gazebo.xacro (robot description, xacro)
@@ -25,5 +25,5 @@
         <update_rate>30</update_rate>
         <visualize>true</visualize>
-        <pose>0 -0.01 0.03 0 4.7124 1.5708</pose>
+        <pose>0 -0.01 0.01 0 4.7124 1.5708</pose>
 				<topic>/camera</topic>
         <gz_frame_id>${prefix}camera_link</gz_frame_id>
@@ -36,6 +36,33 @@
           </image>
           <clip>
-            <near>0.03</near>
+            <near>0.01</near>
             <far>3.0</far>
+          </clip>
+          <noise>
+            <type>gaussian</type>
+            <mean>0.0</mean>
+            <stddev>0.007</stddev>
+          </noise>
+        </camera>
+      </sensor>
+    </gazebo>
+    <gazebo reference="${prefix}base">
+      <sensor name="${prefix}third_person_camera" type="rgbd_camera">
+        <always_on>1</always_on>
+        <update_rate>30</update_rate>
+        <visualize>true</visualize>
+        <pose>0.5 -1.75 1 0 0.2 1.57</pose>
+				<topic>/third_person_camera</topic>
+        <frame_name>${prefix}base</frame_name>
+        <camera>
+          <horizontal_fov>1.547</horizontal_fov>
+          <image>
+            <width>640</width>
+            <height>480</height>
+            <format>R8G8B8</format>
+          </image>
+          <clip>
+            <near>0.01</near>
+            <far>20.0</far>
           </clip>
           <noise>

File: src/tidybot_description/urdf/tidybot.urdf (robot description, URDF)
Before this commit: robot tidybot, 29 links, 28 joints
Links:
- link base: mass 60.0 -> 34; geometry collision mesh filename=file:///home/yuandi/tidybot_platform/install/tidybot_descri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; visual mesh filename=file:///home/yuandi/tidybot_platform/install/tidybot_descri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
- link left_inner_finger: geometry collision mesh filename=file:///home/yuandi/tidybot_platform/install/tidybot_descri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 scale=0.001 0.001 0.001; visual mesh filename=file:///home/yuandi/tidybot_platform/install/tidybot_descri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 scale=0.001 0.001 0.001
- link left_inner_finger_pad: geometry collision box size=0.022 0.00635 0.0375; visual box size=0.022 0.00635 0.0375
- link left_inner_knuckle: geometry collision mesh filename=file:///home/yuandi/tidybot_platform/install/tidybot_descri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 scale=0.001 0.001 0.001; visual mesh filename=file:///home/yuandi/tidybot_platform/install/tidybot_descri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 scale=0.001 0.001 0.001
- link left_outer_finger: geometry collision mesh filename=file:///home/yuandi/tidybot_platform/install/tidybot_descri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 scale=0.001 0.001 0.001; visual mesh filename=file:///home/yuandi/tidybot_platform/install/tidybot_descri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 scale=0.001 0.001 0.001
- link left_outer_knuckle: geometry collision mesh filename=file:///home/yuandi/tidybot_platform/install/tidybot_descri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 scale=0.001 0.001 0.001; visual mesh filename=file:///home/yuandi/tidybot_platform/install/tidybot_descri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 scale=0.001 0.001 0.001
- link right_inner_finger: geometry collision mesh filename=file:///home/yuandi/tidybot_platform/install/tidybot_descri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 scale=0.001 0.001 0.001; visual mesh filename=file:///home/yuandi/tidybot_platform/install/tidybot_descri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 scale=0.001 0.001 0.001
- link right_inner_finger_pad: geometry collision box size=0.022 0.00635 0.0375; visual box size=0.022 0.00635 0.0375
- link right_inner_knuckle: geometry collision mesh filename=file:///home/yuandi/tidybot_platform/install/tidybot_descri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 scale=0.001 0.001 0.001; visual mesh filename=file:///home/yuandi/tidybot_platform/install/tidybot_descri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 scale=0.001 0.001 0.001
- link right_outer_finger: geometry collision mesh filename=file:///home/yuandi/tidybot_platform/install/tidybot_descri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 scale=0.001 0.001 0.001; visual mesh filename=file:///home/yuandi/tidybot_platform/install/tidybot_descri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 scale=0.001 0.001 0.001
- link right_outer_knuckle: geometry collision mesh filename=file:///home/yuandi/tidybot_platform/install/tidybot_descri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 scale=0.001 0.001 0.001; visual mesh filename=file:///home/yuandi/tidybot_platform/install/tidybot_descri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 scale=0.001 0.001 0.001
Joints:
- joint arm_base_joint: origin xyz=0 0 0.33 rpy=0 0 0 -> xyz=0.12 3.76986e-15 0.374775 rpy=0 0 0
- joint left_inner_knuckle_joint: limit lower=0 upper=0.8757 effort=1000 velocity=2.0 -> lower=-0.01 upper=0.8757 effort=1000 velocity=2.0
- joint left_outer_knuckle_joint: limit lower=0 upper=0.8 effort=1000 velocity=2.0 -> lower=-0.01 upper=0.8 effort=1000 velocity=2.0
- joint right_inner_knuckle_joint: limit lower=0 upper=0.8757 effort=1000 velocity=2.0 -> lower=-0.01 upper=0.8757 effort=1000 velocity=2.0
- joint right_outer_knuckle_joint: limit lower=0 upper=0.81 effort=1000 velocity=2.0 -> lower=-0.01 upper=0.81 effort=1000 velocity=2.0
