Commit message: adjust the initial postion of the robot

File: src/tidybot_description/urdf/tidybot.ros2_control.xacro (robot description, xacro)
@@ -2,8 +2,10 @@
 <robot name="ros2_control" xmlns:xacro="http://ros.org/wiki/xacro">
     <xacro:macro name="load_ros2_control" params="hardware_plugin arm gripper">
-        <xacro:macro name="add_joint" params="name gain cmd_interface">
+        <xacro:macro name="add_joint" params="name gain cmd_interface init_pos">
             <joint name="${name}">
                 <command_interface name="${cmd_interface}"/>
-                <state_interface name="position"/>
+                <state_interface name="position">
+                    <param name="initial_value">${init_pos}</param>
+                </state_interface>
                 <state_interface name="velocity"/>
                 <param name="position_proportional_gain">${gain}</param>
@@ -14,29 +16,31 @@
             <plugin>${hardware_plugin}</plugin>
         </hardware>
-        <xacro:add_joint name="joint_x" gain="0.1" cmd_interface="velocity"/>
-        <xacro:add_joint name="joint_x" gain="0.1" cmd_interface="position"/>
-        <xacro:add_joint name="joint_y" gain="0.1" cmd_interface="velocity"/>
-        <xacro:add_joint name="joint_y" gain="0.1" cmd_interface="position"/>
-        <xacro:add_joint name="joint_th" gain="0.1" cmd_interface="velocity"/>
-        <xacro:add_joint name="joint_th" gain="0.1" cmd_interface="position"/>
-        <xacro:add_joint name="joint_1" gain="0.1" cmd_interface="position"/>
-        <xacro:add_joint name="joint_2" gain="0.1" cmd_interface="position"/>
-        <xacro:add_joint name="joint_3" gain="0.1" cmd_interface="position"/>
-        <xacro:add_joint name="joint_4" gain="0.1" cmd_interface="position"/>
-        <xacro:add_joint name="joint_5" gain="0.1" cmd_interface="position"/>
-        <xacro:add_joint name="joint_6" gain="0.1" cmd_interface="position"/>
+        <xacro:add_joint name="joint_x" gain="0.1" cmd_interface="velocity" init_pos="0.0"/>
+        <xacro:add_joint name="joint_x" gain="0.1" cmd_interface="position" init_pos="0.0"/>
+        <xacro:add_joint name="joint_y" gain="0.1" cmd_interface="velocity" init_pos="0.0"/>
+        <xacro:add_joint name="joint_y" gain="0.1" cmd_interface="position" init_pos="0.0"/>
+        <xacro:add_joint name="joint_th" gain="0.1" cmd_interface="velocity" init_pos="0.0"/>
+        <xacro:add_joint name="joint_th" gain="0.1" cmd_interface="position" init_pos="0.0"/>
+        <xacro:add_joint name="joint_1" gain="0.1" cmd_interface="position" init_pos="0.0"/>
+        <xacro:add_joint name="joint_2" gain="0.1" cmd_interface="position" init_pos="-0.348927"/>
+        <xacro:add_joint name="joint_3" gain="0.1" cmd_interface="position" init_pos="3.141522"/>
+        <xacro:add_joint name="joint_4" gain="0.1" cmd_interface="position" init_pos="-2.548368"/>
+        <xacro:add_joint name="joint_5" gain="0.1" cmd_interface="position" init_pos="-3.195793"/>
+        <xacro:add_joint name="joint_6" gain="0.1" cmd_interface="position" init_pos="0.872947"/>
         <xacro:if value="${arm == 'gen3_7dof'}">
-            <xacro:add_joint name="joint_7" gain="0.1" cmd_interface="position"/>
+            <xacro:add_joint name="joint_7" gain="0.1" cmd_interface="position" init_pos="-1.574186"/>
         </xacro:if>
         <xacro:if value="${gripper == 'gen3_lite_2f'}">
-            <xacro:add_joint name="right_finger_bottom_joint" gain="0.1" cmd_interface="position"/>
-            <xacro:add_joint name="right_finger_tip_joint" gain="0.1" cmd_interface="position"/>
-            <xacro:add_joint name="left_finger_bottom_joint" gain="0.1" cmd_interface="position"/>
-            <xacro:add_joint name="left_finger_tip_joint" gain="0.1" cmd_interface="position"/>
+            <xacro:add_joint name="right_finger_bottom_joint" gain="0.1" cmd_interface="position" init_pos="0.0"/>
+            <xacro:add_joint name="right_finger_tip_joint" gain="0.1" cmd_interface="position" init_pos="0.0"/>
+            <xacro:add_joint name="left_finger_bottom_joint" gain="0.1" cmd_interface="position" init_pos="0.0"/>
+            <xacro:add_joint name="left_finger_tip_joint" gain="0.1" cmd_interface="position" init_pos="0.0"/>
         </xacro:if>
         <xacro:if value="${gripper == 'robotiq_2f_85'}">
             <joint name ="left_outer_knuckle_joint">
                 <command_interface name="position"/>
-                <state_interface name="position"/>
+                <state_interface name="position" >
+                    <param name="initial_value">0.0</param>
+                </state_interface>
                 <state_interface name="velocity"/>
                 <param name="position_proportional_gain">0.1</param>
@@ -45,5 +49,7 @@
                 <param name="mimic">left_outer_knuckle_joint</param>
                 <param name="multiplier">-1.0</param>
-                <state_interface name="position"/>
+                <state_interface name="position">
+                    <param name="initial_value">0.0</param>
+                </state_interface>
                 <state_interface name="velocity"/>
             </joint>
@@ -51,5 +57,7 @@
                 <param name="mimic">left_outer_knuckle_joint</param>
                 <param name="multiplier">1.0</param>
-                <state_interface name="position"/>
+                <state_interface name="position">
+                    <param name="initial_value">0.0</param>
+                </state_interface>
                 <state_interface name="velocity"/>
             </joint>
@@ -57,5 +65,7 @@
                 <param name="mimic">left_outer_knuckle_joint</param>
                 <param name="multiplier">1.0</param>
-                <state_interface name="position"/>
+                <state_interface name="position">
+                    <param name="initial_value">0.0</param>
+                </state_interface>
                 <state_interface name="velocity"/>
             </joint>
@@ -63,5 +73,7 @@
                 <param name="mimic">left_outer_knuckle_joint</param>
                 <param name="multiplier">-1.0</param>
-                <state_interface name="position"/>
+                <state_interface name="position">
+                    <param name="initial_value">0.0</param>
+                </state_interface>
                 <state_interface name="velocity"/>
             </joint>
@@ -69,5 +81,7 @@
                 <param name="mimic">left_outer_knuckle_joint</param>
                 <param name="multiplier">1.0</param>
-                <state_interface name="position"/>
+                <state_interface name="position">
+                    <param name="initial_value">0.0</param>
+                </state_interface>
                 <state_interface name="velocity"/>
             </joint>

Commit message: update joystick base control

File: src/tidybot_description/urdf/tidybot.ros2_control.xacro (robot description, xacro)
@@ -1,5 +1,5 @@
 <?xml version="1.0"?>
 <robot name="ros2_control" xmlns:xacro="http://ros.org/wiki/xacro">
-    <xacro:macro name="load_ros2_control" params="hardware_plugin arm gripper">
+    <xacro:macro name="load_ros2_control" params="hardware_plugin arm gripper base_mode">
         <xacro:macro name="add_joint" params="name gain cmd_interface init_pos">
             <joint name="${name}">
@@ -16,10 +16,7 @@
             <plugin>${hardware_plugin}</plugin>
         </hardware>
-        <xacro:add_joint name="joint_x" gain="0.1" cmd_interface="velocity" init_pos="0.0"/>
-        <xacro:add_joint name="joint_x" gain="0.1" cmd_interface="position" init_pos="0.0"/>
-        <xacro:add_joint name="joint_y" gain="0.1" cmd_interface="velocity" init_pos="0.0"/>
-        <xacro:add_joint name="joint_y" gain="0.1" cmd_interface="position" init_pos="0.0"/>
-        <xacro:add_joint name="joint_th" gain="0.1" cmd_interface="velocity" init_pos="0.0"/>
-        <xacro:add_joint name="joint_th" gain="0.1" cmd_interface="position" init_pos="0.0"/>
+        <xacro:add_joint name="joint_x" gain="0.1" cmd_interface="${base_mode}" init_pos="0.0"/>
+        <xacro:add_joint name="joint_y" gain="0.1" cmd_interface="${base_mode}" init_pos="0.0"/>
+        <xacro:add_joint name="joint_th" gain="0.1" cmd_interface="${base_mode}" init_pos="0.0"/>
         <xacro:add_joint name="joint_1" gain="0.1" cmd_interface="position" init_pos="0.0"/>
         <xacro:add_joint name="joint_2" gain="0.1" cmd_interface="position" init_pos="-0.348927"/>

File: src/tidybot_description/urdf/tidybot.urdf (robot description, URDF)
Before this commit: robot tidybot, 31 links, 30 joints
Links:
- removed link finger_link
Joints:
- removed joint finger_joint
- joint camera_module: origin xyz=0 0.05639 -0.00305 rpy=3.14159265358979 3.14159265358979 0 -> xyz=0 0.05639 -0.00405 rpy=3.14159265358979 3.14159265358979 0

File: src/tidybot_description/urdf/tidybot.xacro (robot description, xacro)
@@ -5,4 +5,5 @@
     <xacro:arg name="arm" default="gen3_7dof" />
     <xacro:arg name="gripper" default="robotiq_2f_85" />
+    <xacro:arg name="base_mode" default="position" />
     <xacro:arg name="vision" default="true" />
     <xacro:arg name="prefix" default="" />
@@ -13,5 +14,5 @@
     <!-- configure ros2_control joints -->
     <xacro:include filename="$(find tidybot_description)/urdf/tidybot.ros2_control.xacro" />
-    <xacro:load_ros2_control hardware_plugin="$(arg hardware_plugin)" arm="$(arg arm)" gripper="$(arg gripper)" />
+    <xacro:load_ros2_control hardware_plugin="$(arg hardware_plugin)" arm="$(arg arm)" gripper="$(arg gripper)" base_mode="$(arg base_mode)" />
     <!-- load gazebo plugins -->
     <xacro:include filename="$(find tidybot_description)/urdf/tidybot.gazebo.xacro" />
