Commit message: merge gen3_dof

File: src/tidybot_description/urdf/bot.xacro (robot description, xacro)
@@ -5,7 +5,7 @@
     <xacro:include filename="$(find tidybot_description)/urdf/arms/${arm}/${arm}_macro.xacro" />
     <xacro:include filename="$(find tidybot_description)/urdf/grippers/${gripper}/${gripper}_macro.xacro" />
-    <xacro:include filename="$(find tidybot_description)/urdf/base/base.xacro" />
+    <xacro:include filename="$(find tidybot_description)/urdf/base/tidybot++/base_kinova_macro.xacro" />
     <!-- load the base -->
-    <xacro:load_base parent="" prefix="${prefix}" />
+    <xacro:load_base parent="" prefix="${prefix}" vision="${vision}" />
     <!-- load the arm -->
     <xacro:load_arm parent="${last_base_link}" vision="${vision}" prefix="${prefix}">

File: src/tidybot_description/urdf/grippers/robotiq_2f_85/robotiq_2f_85_macro.xacro (robot description, xacro)
@@ -2,6 +2,19 @@
 <robot name="robotiq_arg2f_85_model" xmlns:xacro="http://ros.org/wiki/xacro">
   <xacro:macro name="load_gripper" params="parent prefix">
-    <xacro:include filename="$(find simulation)/urdf/grippers/robotiq_2f_85/robotiq_arg2f_85_model_macro.xacro" />
-    <xacro:robotiq_arg2f_85 parent="${parent}" prefix="${prefix}"/>
+    <xacro:include filename="$(find tidybot_description)/urdf/grippers/robotiq_2f_85/robotiq_arg2f.xacro" />
+    <xacro:include filename="$(find tidybot_description)/urdf/grippers/robotiq_2f_85/robotiq_arg2f_85_model_macro.xacro" />
+    <link name="${prefix}tool_frame"/>
+    <joint name="${prefix}tool_frame_joint" type="fixed">
+        <origin xyz="0 0 0.120" rpy="0 0 0" />
+        <parent link="${parent}" />
+        <child link="${prefix}tool_frame" />
+        <axis xyz="0 0 0" />
+    </joint>
+    <!-- Gripper description -->
+    <xacro:robotiq_arg2f_base_link prefix="${prefix}" parent="${parent}"/>
+    <xacro:finger_links prefix="${prefix}" fingerprefix="left" stroke="85"/>
+    <xacro:finger_links prefix="${prefix}" fingerprefix="right" stroke="85"/>
+    <xacro:left_outer_knuckle_joint prefix="${prefix}"/>
+    <xacro:right_outer_knuckle_joint prefix="${prefix}"/>
   </xacro:macro>
 </robot>

File: src/tidybot_description/urdf/grippers/robotiq_2f_85/robotiq_arg2f.xacro (robot description, xacro)
@@ -2,4 +2,5 @@
 <robot xmlns:xacro="http://ros.org/wiki/xacro">
   <xacro:macro name="robotiq_arg2f_base_link" params="parent prefix">
+    <xacro:include filename="$(find tidybot_description)/urdf/grippers/robotiq_2f_85/robotiq_arg2f_85_model_macro.xacro" />
     <!-- This joint was added by Kinova -->
     <joint name="${prefix}gripper_base_joint" type="fixed">
@@ -19,5 +20,5 @@
           <!-- The DAE file doesn't show well in Gazebo so we're using the STL instead -->
           <!-- <mesh filename="file://$(find simulation)/meshes/grippers/robotiq_2f_85/meshes/visual/robotiq_arg2f_85_base_link.dae" scale="0.001 0.001 0.001"/> -->
-          <mesh filename="file://$(find simulation)/meshes/grippers/robotiq_2f_85/collision/robotiq_arg2f_base_link.stl" />
+          <mesh filename="file://$(find tidybot_description)/meshes/grippers/robotiq_2f_85/collision/robotiq_arg2f_base_link.stl" />
         </geometry>
         <material name="">
@@ -28,5 +29,5 @@
         <origin xyz="0 0 0" rpy="0 0 0" />
         <geometry>
-           <mesh filename="file://$(find simulation)/meshes/grippers/robotiq_2f_85/collision/robotiq_arg2f_base_link.stl" />
+          <mesh filename="file://$(find tidybot_description)/meshes/grippers/robotiq_2f_85/collision/robotiq_arg2f_base_link.stl" />
         </geometry>
       </collision>

File: src/tidybot_description/urdf/grippers/robotiq_2f_85/robotiq_arg2f_85_model_macro.xacro (robot description, xacro)
@@ -13,5 +13,5 @@
         <origin xyz="0 0 0" rpy="0 0 0" />
         <geometry>
-          <mesh filename="file://$(find simulation)/meshes/grippers/robotiq_2f_85/visual/robotiq_arg2f_85_outer_knuckle.dae" scale="0.001 0.001 0.001"/>
+          <mesh filename="file://$(find tidybot_description)/meshes/grippers/robotiq_2f_85/visual/robotiq_arg2f_85_outer_knuckle.dae" scale="0.001 0.001 0.001"/>
         </geometry>
         <material name="">
@@ -22,5 +22,5 @@
         <origin xyz="0 0 0" rpy="0 0 0" />
         <geometry>
-          <mesh filename="file://$(find simulation)/meshes/grippers/robotiq_2f_85/collision/robotiq_arg2f_85_outer_knuckle.dae" scale="0.001 0.001 0.001"/>
+          <mesh filename="file://$(find tidybot_description)/meshes/grippers/robotiq_2f_85/collision/robotiq_arg2f_85_outer_knuckle.dae" scale="0.001 0.001 0.001"/>
         </geometry>
       </collision>
@@ -37,5 +37,5 @@
         <origin xyz="0 0 0" rpy="0 0 0" />
         <geometry>
-          <mesh filename="file://$(find simulation)/meshes/grippers/robotiq_2f_85/visual/robotiq_arg2f_85_outer_finger.dae" scale="0.001 0.001 0.001"/>
+          <mesh filename="file://$(find tidybot_description)/meshes/grippers/robotiq_2f_85/visual/robotiq_arg2f_85_outer_finger.dae" scale="0.001 0.001 0.001"/>
         </geometry>
         <material name="">
@@ -46,5 +46,5 @@
         <origin xyz="0 0 0" rpy="0 0 0" />
         <geometry>
-          <mesh filename="file://$(find simulation)/meshes/grippers/robotiq_2f_85/collision/robotiq_arg2f_85_outer_finger.dae" scale="0.001 0.001 0.001"/>
+          <mesh filename="file://$(find tidybot_description)/meshes/grippers/robotiq_2f_85/collision/robotiq_arg2f_85_outer_finger.dae" scale="0.001 0.001 0.001"/>
         </geometry>
       </collision>
@@ -55,5 +55,5 @@
       <inertial>
         <origin xyz="0.000123011831763771 0.0507850843201817 0.00103968640075166" rpy="0 0 0" />
-       <mass value="0.0271177346495152" />
+      <mass value="0.0271177346495152" />
         <inertia ixx="2.61910379223783E-05" ixy="-2.43616858946494E-07" ixz="-6.37789906117123E-09" iyy="2.8270243746167E-06" iyz="-5.37200748039765E-07" izz="2.83695868220296E-05" />
       </inertial>
@@ -61,5 +61,5 @@
         <origin xyz="0 0 0" rpy="0 0 0" />
         <geometry>
-          <mesh filename="file://$(find simulation)/meshes/grippers/robotiq_2f_85/visual/robotiq_arg2f_85_inner_knuckle.dae" scale="0.001 0.001 0.001"/>
+          <mesh filename="file://$(find tidybot_description)/meshes/grippers/robotiq_2f_85/visual/robotiq_arg2f_85_inner_knuckle.dae" scale="0.001 0.001 0.001"/>
         </geometry>
         <material name="">
@@ -70,5 +70,5 @@
         <origin xyz="0 0 0" rpy="0 0 0" />
         <geometry>
-          <mesh filename="file://$(find simulation)/meshes/grippers/robotiq_2f_85/collision/robotiq_arg2f_85_inner_knuckle.dae" scale="0.001 0.001 0.001"/>
+          <mesh filename="file://$(find tidybot_description)/meshes/grippers/robotiq_2f_85/collision/robotiq_arg2f_85_inner_knuckle.dae" scale="0.001 0.001 0.001"/>
         </geometry>
       </collision>
@@ -85,5 +85,5 @@
         <origin xyz="0 0 0" rpy="0 0 0" />
         <geometry>
-          <mesh filename="file://$(find simulation)/meshes/grippers/robotiq_2f_85/visual/robotiq_arg2f_85_inner_finger.dae" scale="0.001 0.001 0.001"/>
+          <mesh filename="file://$(find tidybot_description)/meshes/grippers/robotiq_2f_85/visual/robotiq_arg2f_85_inner_finger.dae" scale="0.001 0.001 0.001"/>
         </geometry>
         <material name="">
@@ -94,10 +94,10 @@
         <origin xyz="0 0 0" rpy="0 0 0" />
         <geometry>
-          <mesh filename="file://$(find simulation)/meshes/grippers/robotiq_2f_85/collision/robotiq_arg2f_85_inner_finger.dae" scale="0.001 0.001 0.001" />
+          <mesh filename="file://$(find tidybot_description)/meshes/grippers/robotiq_2f_85/collision/robotiq_arg2f_85_inner_finger.dae" scale="0.001 0.001 0.001" />
         </geometry>
       </collision>
     </link>
   </xacro:macro>
-   <!-- Finger pad link, the default are the "big pads" with rubber-->
+  <!-- Finger pad link, the default are the "big pads" with rubber-->
   <xacro:macro name="inner_finger_pad" params="prefix fingerprefix">
     <link name="${prefix}${fingerprefix}_inner_finger_pad">
@@ -108,5 +108,5 @@
         </geometry>
         <material name="">
-          <color rgba="0.9 0.9 0.9 1" />
+          <color rgba="0.0 0.0 0.0 1" />
         </material>
       </visual>
@@ -114,8 +114,8 @@
         <origin xyz="0 0 0" rpy="0 0 0" />
         <geometry>
-           <box size="0.022 0.00635 0.0375"/>
+          <box size="0.022 0.00635 0.0375"/>
         </geometry>
         <material name="">
-          <color rgba="0.9 0.0 0.0 1" />
+          <color rgba="0.0 0.0 0.0 1" />
         </material>
       </collision>
@@ -137,14 +137,7 @@
       <child link="${prefix}${fingerprefix}_inner_knuckle" />
       <axis xyz="1 0 0" />
-      <limit lower="0" upper="0.8757" velocity="2.0" effort="1000" />
-      <mimic joint="${prefix}finger_joint" multiplier="1" offset="0" />
+      <limit lower="-1.0" upper="1.0" velocity="1.0" effort="1000" />
+      <mimic joint="${prefix}left_outer_knuckle_joint" multiplier="1" offset="0" />
     </joint>
-    <transmission name="{prefix}${fingerprefix}_inner_knuckle_joint_trans">
-      <type>transmission_interface/SimpleTransmission</type>
-      <joint name="${prefix}${fingerprefix}_inner_knuckle_joint" />
-      <actuator name="${prefix}${fingerprefix}_inner_knuckle_joint_motor">
-          <mechanicalReduction>1</mechanicalReduction>
-      </actuator>
-    </transmission>
   </xacro:macro>
   <xacro:macro name="inner_finger_joint" params="prefix fingerprefix">
@@ -154,14 +147,7 @@
       <child link="${prefix}${fingerprefix}_inner_finger" />
       <axis xyz="1 0 0" />
-      <limit lower="-0.8757" upper="0.8757" velocity="2.0" effort="1000" />
-      <mimic joint="${prefix}finger_joint" multiplier="-1" offset="0" />
+      <limit lower="-1.0" upper="1.0" velocity="1.0" effort="1000" />
+      <mimic joint="${prefix}left_outer_knuckle_joint" multiplier="-1" offset="0" />
     </joint>
-    <transmission name="${prefix}${fingerprefix}_inner_finger_joint_trans">
-      <type>transmission_interface/SimpleTransmission</type>
-      <joint name="${prefix}${fingerprefix}_inner_finger_joint" />
-      <actuator name="${prefix}${fingerprefix}_inner_finger_joint_motor">
-          <mechanicalReduction>1</mechanicalReduction>
-      </actuator>
-    </transmission>
   </xacro:macro>
   <xacro:macro name="inner_finger_pad_joint" params="prefix fingerprefix">
@@ -173,20 +159,12 @@
     </joint>
   </xacro:macro>
-  <xacro:include filename="$(find kortex_description)/grippers/robotiq_2f_85/urdf/robotiq_arg2f.xacro" />
-  <xacro:macro name="finger_joint" params="prefix">
-    <joint name="${prefix}finger_joint" type="revolute">
+  <xacro:macro name="left_outer_knuckle_joint" params="prefix">
+    <joint name="${prefix}left_outer_knuckle_joint" type="revolute">
       <origin xyz="0 -0.0306011 0.054904" rpy="0 0 ${pi}"/>
       <parent link="${prefix}robotiq_arg2f_base_link" />
       <child link="${prefix}left_outer_knuckle" />
       <axis xyz="1 0 0" />
-      <limit lower="0" upper="0.8" velocity="2.0" effort="1000" />
+      <limit lower="-1.0" upper="1.0" velocity="1.0" effort="1000" />
     </joint>
-    <transmission name="${prefix}finger_joint_trans">
-      <type>transmission_interface/SimpleTransmission</type>
-      <joint name="${prefix}finger_joint" />
-      <actuator name="${prefix}finger_joint_motor">
-          <mechanicalReduction>1</mechanicalReduction>
-      </actuator>
-    </transmission>
     <xacro:finger_joints prefix="${prefix}" fingerprefix="left" reflect="1.0"/>
   </xacro:macro>
@@ -197,34 +175,8 @@
       <child link="${prefix}right_outer_knuckle" />
       <axis xyz="1 0 0" />
-      <limit lower="0" upper="0.81" velocity="2.0" effort="1000" />
-      <mimic joint="${prefix}finger_joint" multiplier="1" offset="0" />
+      <limit lower="-1.0" upper="1.0" velocity="1.0" effort="1000" />
+      <mimic joint="${prefix}left_outer_knuckle_joint" multiplier="1" offset="0" />
     </joint>
-    <transmission name="$${prefix}right_outer_knuckle_joint_trans">
-      <type>transmission_interface/SimpleTransmission</type>
-      <joint name="${prefix}right_outer_knuckle_joint" />
-      <actuator name="${prefix}right_outer_knuckle_joint_motor">
-          <mechanicalReduction>1</mechanicalReduction>
-      </actuator>
-    </transmission>
     <xacro:finger_joints prefix="${prefix}" fingerprefix="right" reflect="-1.0"/>
   </xacro:macro>
-  <!-- Initialization of all joints and links -->
-  <xacro:macro name="robotiq_arg2f_85" params="prefix parent">
-    <!-- Tool frame used by the arm -->
-    <link name="${prefix}tool_frame"/>
-    <joint name="${prefix}tool_frame_joint" type="fixed">
-        <origin xyz="0 0 0.120" rpy="0 0 0" />
-        <parent link="${parent}" />
-        <child link="${prefix}tool_frame" />
-        <axis xyz="0 0 0" />
-    </joint>
-    <!-- Gripper description -->
-    <xacro:robotiq_arg2f_base_link prefix="${prefix}" parent="${parent}"/>
-    <xacro:finger_links prefix="${prefix}" fingerprefix="left" stroke="85"/>
-    <xacro:finger_links prefix="${prefix}" fingerprefix="right" stroke="85"/>
-    <xacro:finger_joint prefix="${prefix}"/>
-    <xacro:right_outer_knuckle_joint prefix="${prefix}"/>
-    <!-- Transmissions are loaded in the generic kortex xacro when simulation is enabled -->
-    <!-- <xacro:robotiq_arg2f_transmission prefix="${prefix}"/> -->
-  </xacro:macro>
 </robot>

File: src/tidybot_description/urdf/tidybot.gazebo.xacro (robot description, xacro)
@@ -1,5 +1,5 @@
 <?xml version="1.0"?>
 <robot xmlns:xacro="http://ros.org/wiki/xacro">
-<xacro:macro name="load_gazebo_plugins" params="config_path">
+<xacro:macro name="load_gazebo_plugins" params="config_path prefix arm vision">
   <gazebo>
       <plugin name="gz_ros2_control::GazeboSimROS2ControlPlugin" filename="gz_ros2_control-system">
@@ -7,7 +7,7 @@
           <robot_description_param>robot_description</robot_description_param>
       </plugin>
-      <self_collide>true</self_collide>
+      <plugin name="ignition::gazebo::systems::Sensors" filename="libignition-gazebo-sensors-system.so"/>
   </gazebo>
-  <gazebo>
+  <!-- <gazebo>
     <plugin filename="ignition-gazebo-joint-state-publisher-system" name="ignition::gazebo::systems::JointStatePublisher"/>
     <plugin
@@ -17,5 +17,67 @@
         <use_pose_vector_msg>true</use_pose_vector_msg>
     </plugin>
-  </gazebo>
+  </gazebo> -->
+  <xacro:if value="${vision}">
+    <gazebo reference="${prefix}arm_camera_link">
+      <sensor name="${prefix}arm_camera" type="rgbd_camera">
+        <always_on>1</always_on>
+        <update_rate>30</update_rate>
+        <visualize>true</visualize>
+        <pose>0 -0.01 0.03 0 4.7124 1.5708</pose>
+				<topic>/arm_camera</topic>
+        <gz_frame_id>${prefix}arm_camera_link</gz_frame_id>
+        <camera>
+          <horizontal_fov>1.247</horizontal_fov>
+          <image>
+            <width>640</width>
+            <height>480</height>
+            <format>R8G8B8</format>
+          </image>
+          <clip>
+            <near>0.03</near>
+            <far>3.0</far>
+          </clip>
+          <noise>
+            <type>gaussian</type>
+            <mean>0.0</mean>
+            <stddev>0.007</stddev>
+          </noise>
+        </camera>
+      </sensor>
+    </gazebo>
+    <gazebo reference="${prefix}base_camera_link">
+      <sensor name="${prefix}base_camera" type="rgbd_camera">
+        <always_on>1</always_on>
+        <update_rate>30</update_rate>
+        <visualize>true</visualize>
+        <pose>0 0 0 0 0 0</pose>
+				<topic>/base_camera</topic>
+        <gz_frame_id>${prefix}base_camera_link</gz_frame_id>
+        <camera>
+          <horizontal_fov>1.434</horizontal_fov>
+          <image>
+            <width>640</width>
+            <height>360</height>
+            <format>R8G8B8</format>
+          </image>
+          <clip>
+            <near>0.03</near>
+            <far>3.0</far>
+          </clip>
+          <noise>
+            <type>gaussian</type>
+            <mean>0.0</mean>
+            <stddev>0.007</stddev>
+          </noise>
+        </camera>
+      </sensor>
+    </gazebo>
+  </xacro:if>
+  <xacro:include filename="$(find tidybot_description)/urdf/arms/${arm}/${arm}_transmission.xacro" />
+  <xacro:load_arm_transmission prefix="${prefix}" />
+  <xacro:include filename="$(find tidybot_description)/urdf/base/tidybot++/base_kinova_transmission.xacro" />
+  <xacro:load_base_transmission prefix="${prefix}" />
+  <xacro:include filename="$(find tidybot_description)/urdf/grippers/robotiq_2f_85/robotiq_2f_85_transmission.xacro" />
+  <xacro:load_gripper_transmission prefix="${prefix}" />
 </xacro:macro>
 </robot>
