Commit message: merge gen3_dof

File: src/tidybot_description/urdf/tidybot.ros2_control.xacro (robot description, xacro)
@@ -1,33 +1,90 @@
 <?xml version="1.0"?>
 <robot name="ros2_control" xmlns:xacro="http://ros.org/wiki/xacro">
-    <xacro:macro name="load_ros2_control" params="hardware_plugin">
-        <xacro:macro name="add_joint" params="name gain cmd_interface">
+    <xacro:macro name="load_ros2_control" params="hardware_plugin arm gripper">
+        <xacro:macro name="add_joint" params="name gain cmd_interface init_pos">
             <joint name="${name}">
                 <command_interface name="${cmd_interface}"/>
-                <state_interface name="position"/>
+                <state_interface name="position">
+                    <param name="initial_value">${init_pos}</param>
+                </state_interface>
                 <state_interface name="velocity"/>
                 <param name="position_proportional_gain">${gain}</param>
             </joint>
         </xacro:macro>
-        <ros2_control name="GazeboSystem" type="system">
+        <ros2_control name="TidybotSystem" type="system">
         <hardware>
             <plugin>${hardware_plugin}</plugin>
         </hardware>
-        <xacro:add_joint name="joint_x" gain="0.1" cmd_interface="velocity"/>
-        <xacro:add_joint name="joint_x" gain="0.1" cmd_interface="position"/>
-        <xacro:add_joint name="joint_y" gain="0.1" cmd_interface="velocity"/>
-        <xacro:add_joint name="joint_y" gain="0.1" cmd_interface="position"/>
-        <xacro:add_joint name="joint_th" gain="0.1" cmd_interface="velocity"/>
-        <xacro:add_joint name="joint_th" gain="0.1" cmd_interface="position"/>
-        <xacro:add_joint name="joint_1" gain="0.1" cmd_interface="position"/>
-        <xacro:add_joint name="joint_2" gain="0.1" cmd_interface="position"/>
-        <xacro:add_joint name="joint_3" gain="0.1" cmd_interface="position"/>
-        <xacro:add_joint name="joint_4" gain="0.1" cmd_interface="position"/>
-        <xacro:add_joint name="joint_5" gain="0.1" cmd_interface="position"/>
-        <xacro:add_joint name="joint_6" gain="0.1" cmd_interface="position"/>
-        <xacro:add_joint name="right_finger_bottom_joint" gain="0.1" cmd_interface="position"/>
-        <xacro:add_joint name="right_finger_tip_joint" gain="0.1" cmd_interface="position"/>
-        <xacro:add_joint name="left_finger_bottom_joint" gain="0.1" cmd_interface="position"/>
-        <xacro:add_joint name="left_finger_tip_joint" gain="0.1" cmd_interface="position"/>
+        <xacro:add_joint name="joint_x" gain="0.1" cmd_interface="velocity" init_pos="0.0"/>
+        <xacro:add_joint name="joint_x" gain="0.1" cmd_interface="position" init_pos="0.0"/>
+        <xacro:add_joint name="joint_y" gain="0.1" cmd_interface="velocity" init_pos="0.0"/>
+        <xacro:add_joint name="joint_y" gain="0.1" cmd_interface="position" init_pos="0.0"/>
+        <xacro:add_joint name="joint_th" gain="0.1" cmd_interface="velocity" init_pos="0.0"/>
+        <xacro:add_joint name="joint_th" gain="0.1" cmd_interface="position" init_pos="0.0"/>
+        <xacro:add_joint name="joint_1" gain="0.1" cmd_interface="position" init_pos="0.0"/>
+        <xacro:add_joint name="joint_2" gain="0.1" cmd_interface="position" init_pos="-0.348927"/>
+        <xacro:add_joint name="joint_3" gain="0.1" cmd_interface="position" init_pos="3.141522"/>
+        <xacro:add_joint name="joint_4" gain="0.1" cmd_interface="position" init_pos="-2.548368"/>
+        <xacro:add_joint name="joint_5" gain="0.1" cmd_interface="position" init_pos="-3.195793"/>
+        <xacro:add_joint name="joint_6" gain="0.1" cmd_interface="position" init_pos="0.872947"/>
+        <xacro:if value="${arm == 'gen3_7dof'}">
+            <xacro:add_joint name="joint_7" gain="0.1" cmd_interface="position" init_pos="-1.574186"/>
+        </xacro:if>
+        <xacro:if value="${gripper == 'gen3_lite_2f'}">
+            <xacro:add_joint name="right_finger_bottom_joint" gain="0.1" cmd_interface="position" init_pos="0.0"/>
+            <xacro:add_joint name="right_finger_tip_joint" gain="0.1" cmd_interface="position" init_pos="0.0"/>
+            <xacro:add_joint name="left_finger_bottom_joint" gain="0.1" cmd_interface="position" init_pos="0.0"/>
+            <xacro:add_joint name="left_finger_tip_joint" gain="0.1" cmd_interface="position" init_pos="0.0"/>
+        </xacro:if>
+        <xacro:if value="${gripper == 'robotiq_2f_85'}">
+            <joint name ="left_outer_knuckle_joint">
+                <command_interface name="position"/>
+                <state_interface name="position" >
+                    <param name="initial_value">0.0</param>
+                </state_interface>
+                <state_interface name="velocity"/>
+                <param name="position_proportional_gain">0.1</param>
+            </joint>
+            <joint name ="right_inner_finger_joint">
+                <param name="mimic">left_outer_knuckle_joint</param>
+                <param name="multiplier">-1.0</param>
+                <state_interface name="position">
+                    <param name="initial_value">0.0</param>
+                </state_interface>
+                <state_interface name="velocity"/>
+            </joint>
+            <joint name ="right_outer_knuckle_joint">
+                <param name="mimic">left_outer_knuckle_joint</param>
+                <param name="multiplier">1.0</param>
+                <state_interface name="position">
+                    <param name="initial_value">0.0</param>
+                </state_interface>
+                <state_interface name="velocity"/>
+            </joint>
+            <joint name ="right_inner_knuckle_joint">
+                <param name="mimic">left_outer_knuckle_joint</param>
+                <param name="multiplier">1.0</param>
+                <state_interface name="position">
+                    <param name="initial_value">0.0</param>
+                </state_interface>
+                <state_interface name="velocity"/>
+            </joint>
+            <joint name ="left_inner_finger_joint">
+                <param name="mimic">left_outer_knuckle_joint</param>
+                <param name="multiplier">-1.0</param>
+                <state_interface name="position">
+                    <param name="initial_value">0.0</param>
+                </state_interface>
+                <state_interface name="velocity"/>
+            </joint>
+            <joint name ="left_inner_knuckle_joint">
+                <param name="mimic">left_outer_knuckle_joint</param>
+                <param name="multiplier">1.0</param>
+                <state_interface name="position">
+                    <param name="initial_value">0.0</param>
+                </state_interface>
+                <state_interface name="velocity"/>
+            </joint>
+        </xacro:if>
         </ros2_control>
     </xacro:macro>

File: src/tidybot_description/urdf/tidybot.urdf (robot description, URDF)
Before this commit: robot tidybot, 18 links, 17 joints
Links:
- removed link arm_link
- removed link gripper_base_link
- removed link left_finger_dist_link
- removed link left_finger_prox_link
- removed link lower_wrist_link
- removed link right_finger_dist_link
- removed link right_finger_prox_link
- removed link upper_wrist_link
- added link arm_camera_link
- added link base_camera_link
- added link bracelet_link, mass 0.5; collision mesh filename=file:///home/janchen/Documents/tidybot_platform/install/tid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; visual mesh filename=file:///home/janchen/Documents/tidybot_platform/install/tid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
- added link camera_color_frame
- added link camera_depth_frame
- added link finger_link
- added link half_arm_1_link, mass 1.1636; collision mesh filename=file:///home/janchen/Documents/tidybot_platform/install/tid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; visual mesh filename=file:///home/janchen/Documents/tidybot_platform/install/tid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
- added link half_arm_2_link, mass 1.1636; collision mesh filename=file:///home/janchen/Documents/tidybot_platform/install/tid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; visual mesh filename=file:///home/janchen/Documents/tidybot_platform/install/tid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
- added link left_inner_finger, mass 0.0104003125914103; collision mesh filename=file:///home/janchen/Documents/tidybot_platform/install/tid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 scale=0.001 0.001 0.001; visual mesh filename=file:///home/janchen/Documents/tidybot_platform/install/tid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 scale=0.001 0.001 0.001
- added link left_inner_finger_pad; collision box size=0.022 0.00635 0.0375; visual box size=0.022 0.00635 0.0375
- added link left_inner_knuckle, mass 0.0271177346495152; collision mesh filename=file:///home/janchen/Documents/tidybot_platform/install/tid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 scale=0.001 0.001 0.001; visual mesh filename=file:///home/janchen/Documents/tidybot_platform/install/tid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 scale=0.001 0.001 0.001
- added link left_outer_finger, mass 0.022614240507152; collision mesh filename=file:///home/janchen/Documents/tidybot_platform/install/tid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 scale=0.001 0.001 0.001; visual mesh filename=file:///home/janchen/Documents/tidybot_platform/install/tid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 scale=0.001 0.001 0.001
- added link left_outer_knuckle, mass 0.00853198276973456; collision mesh filename=file:///home/janchen/Documents/tidybot_platform/install/tid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 scale=0.001 0.001 0.001; visual mesh filename=file:///home/janchen/Documents/tidybot_platform/install/tid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 scale=0.001 0.001 0.001
- added link right_inner_finger, mass 0.0104003125914103; collision mesh filename=file:///home/janchen/Documents/tidybot_platform/install/tid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 scale=0.001 0.001 0.001; visual mesh filename=file:///home/janchen/Documents/tidybot_platform/install/tid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 scale=0.001 0.001 0.001
- added link right_inner_finger_pad; collision box size=0.022 0.00635 0.0375; visual box size=0.022 0.00635 0.0375
- added link right_inner_knuckle, mass 0.0271177346495152; collision mesh filename=file:///home/janchen/Documents/tidybot_platform/install/tid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 scale=0.001 0.001 0.001; visual mesh filename=file:///home/janchen/Documents/tidybot_platform/install/tid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 scale=0.001 0.001 0.001
- added link right_outer_finger, mass 0.022614240507152; collision mesh filename=file:///home/janchen/Documents/tidybot_platform/install/tid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 scale=0.001 0.001 0.001; visual mesh filename=file:///home/janchen/Documents/tidybot_platform/install/tid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 scale=0.001 0.001 0.001
- added link right_outer_knuckle, mass 0.00853198276973456; collision mesh filename=file:///home/janchen/Documents/tidybot_platform/install/tid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 scale=0.001 0.001 0.001; visual mesh filename=file:///home/janchen/Documents/tidybot_platform/install/tid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 scale=0.001 0.001 0.001
- added link robotiq_arg2f_base_link, mass 0.22652; collision mesh filename=file:///home/janchen/Documents/tidybot_platform/install/tid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; visual mesh filename=file:///home/janchen/Documents/tidybot_platform/install/tid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
- added link spherical_wrist_1_link, mass 0.6781; collision mesh filename=file:///home/janchen/Documents/tidybot_platform/install/tid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; visual mesh filename=file:///home/janchen/Documents/tidybot_platform/install/tid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
- added link spherical_wrist_2_link, mass 0.6781; collision mesh filename=file:///home/janchen/Documents/tidybot_platform/install/tid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; visual mesh filename=file:///home/janchen/Documents/tidybot_platform/install/tid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
- link arm_base_link: mass 1.14608471 -> 1.697; geometry collision mesh filename=file:///home/janchen/Documents/tidybot_platform/install/tid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; visual mesh filename=file:///home/janchen/Documents/tidybot_platform/install/tid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
- link base: mass 60.0 -> 34; geometry collision mesh filename=file:///home/janchen/Documents/tidybot_platform/install/tid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; visual mesh filename=file:///home/janchen/Documents/tidybot_platform/install/tid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
- link forearm_link: mass 0.59767669 -> 0.9302; geometry collision mesh filename=file:///home/janchen/Documents/tidybot_platform/install/tid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; visual mesh filename=file:///home/janchen/Documents/tidybot_platform/install/tid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
- link shoulder_link: mass 0.95974404 -> 1.3773; geometry collision mesh filename=file:///home/janchen/Documents/tidybot_platform/install/tid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; visual mesh filename=file:///home/janchen/Documents/tidybot_platform/install/tid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
Joints:
- removed joint left_finger_bottom_joint
- removed joint left_finger_tip_joint
- removed joint right_finger_bottom_joint
- removed joint right_finger_tip_joint
- added joint base_camera_joint: type fixed, parent base, child base_camera_link, origin xyz=0.2525 0.0 0.315 rpy=0 0.7853981634 0
- added joint camera_module: type fixed, parent end_effector_link, child arm_camera_link, origin xyz=0 0.05639 -0.00305 rpy=3.14159265358979 3.14159265358979 0
- added joint color_module: type fixed, parent end_effector_link, child camera_color_frame, origin xyz=0 0.05639 -0.00305 rpy=3.14159265358979 3.14159265358979 0
- added joint depth_module: type fixed, parent end_effector_link, child camera_depth_frame, origin xyz=0.0275 0.066 -0.00305 rpy=3.14159265358979 3.14159265358979 0
- added joint end_effector: type fixed, parent bracelet_link, child end_effector_link, origin xyz=0 0 -0.0615250000000001 rpy=3.14159265358979 1.09937075168372E-32 0, axis 0 0 0
- added joint finger_joint: type revolute, parent end_effector_link, child finger_link, origin xyz=0 0 0 rpy=0 0 0, axis 1 0 0, limit lower=0 upper=0.81 effort=1000 velocity=1.0
- added joint joint_7: type continuous, parent spherical_wrist_2_link, child bracelet_link, origin xyz=0 -0.10593 -0.00017505 rpy=-1.5708 -5.5511E-17 9.6396E-17, axis 0 0 1, limit effort=9 velocity=1.2218
- added joint left_inner_finger_joint: type revolute, parent left_outer_finger, child left_inner_finger, origin xyz=0 0.0061 0.0471 rpy=0 0 0, axis 1 0 0, limit lower=-1.0 upper=1.0 effort=1000 velocity=1.0, mimic joint=left_outer_knuckle_joint multiplier=-1 offset=0
- added joint left_inner_finger_pad_joint: type fixed, parent left_inner_finger, child left_inner_finger_pad, origin xyz=0 -0.0220203446692936 0.03242 rpy=0 0 0, axis 0 0 1
- added joint left_inner_knuckle_joint: type revolute, parent robotiq_arg2f_base_link, child left_inner_knuckle, origin xyz=0 -0.0127 0.06142 rpy=0 0 3.141592653589793, axis 1 0 0, limit lower=-1.0 upper=1.0 effort=1000 velocity=1.0, mimic joint=left_outer_knuckle_joint multiplier=1 offset=0
- added joint left_outer_finger_joint: type fixed, parent left_outer_knuckle, child left_outer_finger, origin xyz=0 0.0315 -0.0041 rpy=0 0 0, axis 1 0 0
- added joint left_outer_knuckle_joint: type revolute, parent robotiq_arg2f_base_link, child left_outer_knuckle, origin xyz=0 -0.0306011 0.054904 rpy=0 0 3.141592653589793, axis 1 0 0, limit lower=-1.0 upper=1.0 effort=1000 velocity=1.0
- added joint right_inner_finger_joint: type revolute, parent right_outer_finger, child right_inner_finger, origin xyz=0 0.0061 0.0471 rpy=0 0 0, axis 1 0 0, limit lower=-1.0 upper=1.0 effort=1000 velocity=1.0, mimic joint=left_outer_knuckle_joint multiplier=-1 offset=0
- added joint right_inner_finger_pad_joint: type fixed, parent right_inner_finger, child right_inner_finger_pad, origin xyz=0 -0.0220203446692936 0.03242 rpy=0 0 0, axis 0 0 1
- added joint right_inner_knuckle_joint: type revolute, parent robotiq_arg2f_base_link, child right_inner_knuckle, origin xyz=0 0.0127 0.06142 rpy=0 0 0.0, axis 1 0 0, limit lower=-1.0 upper=1.0 effort=1000 velocity=1.0, mimic joint=left_outer_knuckle_joint multiplier=1 offset=0
- added joint right_outer_finger_joint: type fixed, parent right_outer_knuckle, child right_outer_finger, origin xyz=0 0.0315 -0.0041 rpy=0 0 0, axis 1 0 0
- added joint right_outer_knuckle_joint: type revolute, parent robotiq_arg2f_base_link, child right_outer_knuckle, origin xyz=0 0.0306011 0.054904 rpy=0 0 0, axis 1 0 0, limit lower=-1.0 upper=1.0 effort=1000 velocity=1.0, mimic joint=left_outer_knuckle_joint multiplier=1 offset=0
- joint arm_base_joint: origin xyz=0 0 0.33 rpy=0 0 0 -> xyz=0.12 3.76986e-15 0.374775 rpy=0 0 0
- joint gripper_base_joint: axis 0 0 0 -> (none); child gripper_base_link -> robotiq_arg2f_base_link; origin xyz=0 0 0 rpy=0 0 0 -> xyz=0.0 0.0 0.0 rpy=0.0 0.0 1.57
- joint joint_1: limit lower=-2.69 upper=2.69 effort=10 velocity=1.6 -> effort=39 velocity=1.3963; origin xyz=0 0 0.12825 rpy=0 0 0 -> xyz=0 0 0.15643 rpy=3.1416 2.7629E-18 -4.9305E-36; type revolute -> continuous
- joint joint_2: child arm_link -> half_arm_1_link; limit lower=-2.69 upper=2.69 effort=14 velocity=1.6 -> lower=-2.24 upper=2.24 effort=39 velocity=1.3963; origin xyz=0 -0.03 0.115 rpy=1.5708 0 0 -> xyz=0 0.005375 -0.12838 rpy=1.5708 2.1343E-17 -1.1102E-16
- joint joint_3: child forearm_link -> half_arm_2_link; limit lower=-2.69 upper=2.69 effort=10 velocity=1.6 -> effort=39 velocity=1.3963; origin xyz=0 0.28 0 rpy=-3.1416 0 0 -> xyz=0 -0.21038 -0.006375 rpy=-1.5708 1.2326E-32 -2.9122E-16; parent arm_link -> half_arm_1_link; type revolute -> continuous
- joint joint_4: child lower_wrist_link -> forearm_link; limit lower=-2.59 upper=2.59 effort=7 velocity=1.6 -> lower=-2.57 upper=2.57 effort=39 velocity=1.3963; origin xyz=0 -0.14 0.02 rpy=1.5708 0 0 -> xyz=0 0.006375 -0.21038 rpy=1.5708 -6.6954E-17 -1.6653E-16; parent forearm_link -> half_arm_2_link
- joint joint_5: child upper_wrist_link -> spherical_wrist_1_link; limit lower=-2.57 upper=2.57 effort=7 velocity=1.6 -> effort=9 velocity=1.2218; origin xyz=0.0285 0 0.105 rpy=0 1.5708 0 -> xyz=0 -0.20843 -0.006375 rpy=-1.5708 2.2204E-16 -6.373E-17; parent lower_wrist_link -> forearm_link; type revolute -> continuous
- joint joint_6: child end_effector_link -> spherical_wrist_2_link; limit lower=-2.59 upper=2.59 effort=7 velocity=3.2 -> lower=-2.09 upper=2.09 effort=9 velocity=1.2218; origin xyz=-0.105 0 0.0285 rpy=0 -1.5708 0 -> xyz=0 0.00017505 -0.10593 rpy=1.5708 9.2076E-28 -8.2157E-15; parent upper_wrist_link -> spherical_wrist_1_link
- joint tool_frame_joint: origin xyz=0 0 0.130 rpy=0 0 1.57079632679 -> xyz=0 0 0.120 rpy=0 0 0

File: src/tidybot_description/urdf/tidybot.xacro (robot description, xacro)
@@ -1,8 +1,9 @@
 <?xml version="1.0"?>
 <robot name="tidybot" xmlns:xacro="http://ros.org/wiki/xacro">
-    <xacro:arg name="hardware_plugin" default="mock_components/GenericSystem" />
-    <xacro:arg name="arm" default="gen3_lite" />
-    <xacro:arg name="gripper" default="gen3_lite_2f" />
-    <xacro:arg name="vision" default="false" />
+    <!-- <xacro:arg name="hardware_plugin" default="mock_components/GenericSystem" />     -->
+    <xacro:arg name="hardware_plugin" default="gz_ros2_control/GazeboSimSystem" />
+    <xacro:arg name="arm" default="gen3_7dof" />
+    <xacro:arg name="gripper" default="robotiq_2f_85" />
+    <xacro:arg name="vision" default="true" />
     <xacro:arg name="prefix" default="" />
     <xacro:arg name="ros2_control_config_path" default="$(find tidybot_description)/config/tidybot_controllers.yaml"/>
@@ -12,7 +13,7 @@
     <!-- configure ros2_control joints -->
     <xacro:include filename="$(find tidybot_description)/urdf/tidybot.ros2_control.xacro" />
-    <xacro:load_ros2_control hardware_plugin="$(arg hardware_plugin)" />
+    <xacro:load_ros2_control hardware_plugin="$(arg hardware_plugin)" arm="$(arg arm)" gripper="$(arg gripper)" />
     <!-- load gazebo plugins -->
     <xacro:include filename="$(find tidybot_description)/urdf/tidybot.gazebo.xacro" />
-    <xacro:load_gazebo_plugins config_path="$(arg ros2_control_config_path)" />
+    <xacro:load_gazebo_plugins config_path="$(arg ros2_control_config_path)" prefix="$(arg prefix)" arm="$(arg arm)" vision="$(arg vision)" />
 </robot>

File: src/tidybot_moveit_config/config/tidybot.ros2_control.xacro (robot description, xacro)
@@ -50,8 +50,8 @@
                 <state_interface name="velocity"/>
             </joint>
-            <joint name="right_finger_bottom_joint">
+            <joint name="joint_7">
                 <command_interface name="position"/>
                 <state_interface name="position">
-                  <param name="initial_value">${initial_positions['right_finger_bottom_joint']}</param>
+                  <param name="initial_value">${initial_positions['joint_7']}</param>
                 </state_interface>
                 <state_interface name="velocity"/>
