Commit message: change the style and the base controller to velocity controller

File: src/tidybot_description/urdf/tidybot.urdf (robot description, URDF)
Before this commit: robot tidybot, 18 links, 17 joints
Links:
- link arm_base_link: geometry collision mesh filename=file:///home/janchen/Documents/ros2/tidybot_ws/install/tidy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; visual mesh filename=file:///home/janchen/Documents/ros2/tidybot_ws/install/tidy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
- link arm_link: geometry collision mesh filename=file:///home/janchen/Documents/ros2/tidybot_ws/install/tidy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; visual mesh filename=file:///home/janchen/Documents/ros2/tidybot_ws/install/tidy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
- link base_link: geometry collision mesh filename=file:///home/janchen/Documents/ros2/tidybot_ws/install/tidy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; collision mesh filename=file:///home/janchen/Documents/ros2/tidybot_ws/install/tidy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
- link forearm_link: geometry collision mesh filename=file:///home/janchen/Documents/ros2/tidybot_ws/install/tidy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; visual mesh filename=file:///home/janchen/Documents/ros2/tidybot_ws/install/tidy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
- link gripper_base_link: geometry collision mesh filename=file:///home/janchen/Documents/ros2/tidybot_ws/install/tidy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; visual mesh filename=file:///home/janchen/Documents/ros2/tidybot_ws/install/tidy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
- link left_finger_dist_link: geometry collision mesh filename=file:///home/janchen/Documents/ros2/tidybot_ws/install/tidy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; visual mesh filename=file:///home/janchen/Documents/ros2/tidybot_ws/install/tidy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
- link left_finger_prox_link: geometry collision mesh filename=file:///home/janchen/Documents/ros2/tidybot_ws/install/tidy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; visual mesh filename=file:///home/janchen/Documents/ros2/tidybot_ws/install/tidy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
- link lower_wrist_link: geometry collision mesh filename=file:///home/janchen/Documents/ros2/tidybot_ws/install/tidy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; visual mesh filename=file:///home/janchen/Documents/ros2/tidybot_ws/install/tidy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
- link right_finger_dist_link: geometry collision mesh filename=file:///home/janchen/Documents/ros2/tidybot_ws/install/tidy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; visual mesh filename=file:///home/janchen/Documents/ros2/tidybot_ws/install/tidy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
- link right_finger_prox_link: geometry collision mesh filename=file:///home/janchen/Documents/ros2/tidybot_ws/install/tidy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; visual mesh filename=file:///home/janchen/Documents/ros2/tidybot_ws/install/tidy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
- link shoulder_link: geometry collision mesh filename=file:///home/janchen/Documents/ros2/tidybot_ws/install/tidy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; visual mesh filename=file:///home/janchen/Documents/ros2/tidybot_ws/install/tidy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
- link upper_wrist_link: geometry collision mesh filename=file:///home/janchen/Documents/ros2/tidybot_ws/install/tidy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; visual mesh filename=file:///home/janchen/Documents/ros2/tidybot_ws/install/tidy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
Joints:
- joint joint_th: limit lower=0.0 upper=0.0 effort=100 velocity=100 -> lower=-3.14 upper=3.14 effort=100 velocity=1
- joint joint_th_offset: axis (none) -> 0.0 0.0 1.0; limit (none) -> lower=0.0 upper=0.0 effort=100 velocity=100
- joint joint_x: axis (none) -> 1 0 0; limit (none) -> lower=-10.0 upper=10.0 effort=100 velocity=1; type fixed -> prismatic
- joint joint_y: axis (none) -> 0 1 0; limit (none) -> lower=-10.0 upper=10.0 effort=100 velocity=1; type fixed -> prismatic
- joint left_finger_bottom_joint: mimic joint=right_finger_bottom_joint multiplier=-1.0 offset=0.0 -> (none)
- joint left_finger_tip_joint: mimic joint=right_finger_bottom_joint multiplier=-0.676 offset=0.149 -> (none)
- joint right_finger_tip_joint: mimic joint=right_finger_bottom_joint multiplier=-0.676 offset=0.149 -> (none)

File: src/tidybot_description/urdf/tidybot.xacro (robot description, xacro)
@@ -5,41 +5,10 @@
     <xacro:arg name="vision" default="false" />
     <xacro:arg name="prefix" default="" />
-    <xacro:arg name="ros2_control_config_path" default="UNSET"/>
+    <xacro:arg name="ros2_control_config_path" default="$(find tidybot_description)/config/tidybot_controllers.yaml"/>
     <xacro:include filename="$(find tidybot_description)/urdf/bot.xacro" />
     <!-- load the robot -->
     <xacro:load_bot arm="$(arg arm)" gripper="$(arg gripper)" vision="$(arg vision)" prefix="$(arg prefix)" />
     <!-- configure ros2_control joints -->
-    <xacro:macro name="add_joint" params="name gain">
-        <joint name="${name}">
-            <command_interface name="position"/>
-            <state_interface name="position"/>
-            <state_interface name="velocity"/>
-            <param name="position_proportional_gain">${gain}</param>
-        </joint>
-    </xacro:macro>
-    <ros2_control name="GazeboSystem" type="system">
-    <hardware>
-        <plugin>gz_ros2_control/GazeboSimSystem</plugin>
-    </hardware>
-    <xacro:add_joint name="joint_x" gain="0.1"/>
-    <xacro:add_joint name="joint_y" gain="0.1"/>
-    <xacro:add_joint name="joint_th" gain="0.1"/>
-    <xacro:add_joint name="joint_1" gain="0.1"/>
-    <xacro:add_joint name="joint_2" gain="0.1"/>
-    <xacro:add_joint name="joint_3" gain="0.1"/>
-    <xacro:add_joint name="joint_4" gain="0.1"/>
-    <xacro:add_joint name="joint_5" gain="0.1"/>
-    <xacro:add_joint name="joint_6" gain="0.1"/>
-    <xacro:add_joint name="right_finger_bottom_joint" gain="0.1"/>
-    <xacro:add_joint name="right_finger_tip_joint" gain="0.1"/>
-    <xacro:add_joint name="left_finger_bottom_joint" gain="0.1"/>
-    <xacro:add_joint name="left_finger_tip_joint" gain="0.1"/>
-    </ros2_control>
-    <gazebo>
-        <plugin name="gz_ros2_control::GazeboSimROS2ControlPlugin" filename="gz_ros2_control-system">
-            <parameters>$(find tidybot_description)/urdf/ros2_control.yaml</parameters>
-            <robot_description_param>robot_description</robot_description_param>
-        </plugin>
-        <self_collide>true</self_collide>
-    </gazebo>
+    <xacro:include filename="$(find tidybot_description)/urdf/ros2_control.xacro" />
+    <xacro:load_ros2_control config_path="$(arg ros2_control_config_path)"/>
 </robot>

Commit message: add moveit_config for gen3_7dof arm

File: src/tidybot_description/urdf/tidybot.urdf (robot description, URDF)
Before this commit: robot tidybot, 18 links, 17 joints
Links:
- removed link arm_link
- removed link lower_wrist_link
- removed link upper_wrist_link
- added link bracelet_link, mass 0.364; collision mesh filename=file:///home/janchen/Documents/ros2/tidybot_ws/install/tidy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; visual mesh filename=file:///home/janchen/Documents/ros2/tidybot_ws/install/tidy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
- added link half_arm_1_link, mass 1.1636; collision mesh filename=file:///home/janchen/Documents/ros2/tidybot_ws/install/tidy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; visual mesh filename=file:///home/janchen/Documents/ros2/tidybot_ws/install/tidy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
- added link half_arm_2_link, mass 1.1636; collision mesh filename=file:///home/janchen/Documents/ros2/tidybot_ws/install/tidy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; visual mesh filename=file:///home/janchen/Documents/ros2/tidybot_ws/install/tidy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
- added link spherical_wrist_1_link, mass 0.6781; collision mesh filename=file:///home/janchen/Documents/ros2/tidybot_ws/install/tidy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; visual mesh filename=file:///home/janchen/Documents/ros2/tidybot_ws/install/tidy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
- added link spherical_wrist_2_link, mass 0.6781; collision mesh filename=file:///home/janchen/Documents/ros2/tidybot_ws/install/tidy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; visual mesh filename=file:///home/janchen/Documents/ros2/tidybot_ws/install/tidy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
- link arm_base_link: mass 1.14608471 -> 1.697
- link forearm_link: mass 0.59767669 -> 0.9302
- link shoulder_link: mass 0.95974404 -> 1.3773
Joints:
- added joint end_effector: type fixed, parent bracelet_link, child end_effector_link, origin xyz=0 0 -0.0615250000000001 rpy=3.14159265358979 1.09937075168372E-32 0, axis 0 0 0
- added joint joint_7: type continuous, parent spherical_wrist_2_link, child bracelet_link, origin xyz=0 -0.10593 -0.00017505 rpy=-1.5708 -5.5511E-17 9.6396E-17, axis 0 0 1, limit effort=9 velocity=1.2218
- joint joint_1: limit lower=-2.69 upper=2.69 effort=10 velocity=1.6 -> effort=39 velocity=1.3963; origin xyz=0 0 0.12825 rpy=0 0 0 -> xyz=0 0 0.15643 rpy=3.1416 2.7629E-18 -4.9305E-36; type revolute -> continuous
- joint joint_2: child arm_link -> half_arm_1_link; limit lower=-2.69 upper=2.69 effort=14 velocity=1.6 -> lower=-2.24 upper=2.24 effort=39 velocity=1.3963; origin xyz=0 -0.03 0.115 rpy=1.5708 0 0 -> xyz=0 0.005375 -0.12838 rpy=1.5708 2.1343E-17 -1.1102E-16
- joint joint_3: child forearm_link -> half_arm_2_link; limit lower=-2.69 upper=2.69 effort=10 velocity=1.6 -> effort=39 velocity=1.3963; origin xyz=0 0.28 0 rpy=-3.1416 0 0 -> xyz=0 -0.21038 -0.006375 rpy=-1.5708 1.2326E-32 -2.9122E-16; parent arm_link -> half_arm_1_link; type revolute -> continuous
- joint joint_4: child lower_wrist_link -> forearm_link; limit lower=-2.59 upper=2.59 effort=7 velocity=1.6 -> lower=-2.57 upper=2.57 effort=39 velocity=1.3963; origin xyz=0 -0.14 0.02 rpy=1.5708 0 0 -> xyz=0 0.006375 -0.21038 rpy=1.5708 -6.6954E-17 -1.6653E-16; parent forearm_link -> half_arm_2_link
- joint joint_5: child upper_wrist_link -> spherical_wrist_1_link; limit lower=-2.57 upper=2.57 effort=7 velocity=1.6 -> effort=9 velocity=1.2218; origin xyz=0.0285 0 0.105 rpy=0 1.5708 0 -> xyz=0 -0.20843 -0.006375 rpy=-1.5708 2.2204E-16 -6.373E-17; parent lower_wrist_link -> forearm_link; type revolute -> continuous
- joint joint_6: child end_effector_link -> spherical_wrist_2_link; limit lower=-2.59 upper=2.59 effort=7 velocity=3.2 -> lower=-2.09 upper=2.09 effort=9 velocity=1.2218; origin xyz=-0.105 0 0.0285 rpy=0 -1.5708 0 -> xyz=0 0.00017505 -0.10593 rpy=1.5708 9.2076E-28 -8.2157E-15; parent upper_wrist_link -> spherical_wrist_1_link

File: src/tidybot_moveit_config/config/tidybot.ros2_control.xacro (robot description, xacro)
@@ -50,4 +50,25 @@
                 <state_interface name="velocity"/>
             </joint>
+            <joint name="joint_7">
+                <command_interface name="position"/>
+                <state_interface name="position">
+                  <param name="initial_value">${initial_positions['joint_7']}</param>
+                </state_interface>
+                <state_interface name="velocity"/>
+            </joint>
+            <joint name="left_finger_bottom_joint">
+                <command_interface name="position"/>
+                <state_interface name="position">
+                  <param name="initial_value">${initial_positions['left_finger_bottom_joint']}</param>
+                </state_interface>
+                <state_interface name="velocity"/>
+            </joint>
+            <joint name="left_finger_tip_joint">
+                <command_interface name="position"/>
+                <state_interface name="position">
+                  <param name="initial_value">${initial_positions['left_finger_tip_joint']}</param>
+                </state_interface>
+                <state_interface name="velocity"/>
+            </joint>
             <joint name="right_finger_bottom_joint">
                 <command_interface name="position"/>
@@ -57,4 +78,11 @@
                 <state_interface name="velocity"/>
             </joint>
+            <joint name="right_finger_tip_joint">
+                <command_interface name="position"/>
+                <state_interface name="position">
+                  <param name="initial_value">${initial_positions['right_finger_tip_joint']}</param>
+                </state_interface>
+                <state_interface name="velocity"/>
+            </joint>
         </ros2_control>
     </xacro:macro>

File: src/tidybot_moveit_config/config/tidybot.urdf.xacro (robot description, xacro)
@@ -2,6 +2,8 @@
 <robot xmlns:xacro="http://www.ros.org/wiki/xacro" name="tidybot">
     <xacro:arg name="initial_positions_file" default="initial_positions.yaml" />
-    <xacro:arg name="ros2_control_config_path" default="$(find tidybot_description)/config/tidybot_controllers.yaml"/>
     <!-- Import tidybot urdf file -->
-    <xacro:include filename="$(find tidybot_description)/urdf/tidybot.xacro" />
+    <xacro:include filename="$(find tidybot_description)/urdf/tidybot.urdf" />
+    <!-- Import control_xacro -->
+    <xacro:include filename="tidybot.ros2_control.xacro" />
+    <xacro:tidybot_ros2_control name="FakeSystem" initial_positions_file="$(arg initial_positions_file)"/>
 </robot>

Commit message: add joint state publisher

File: src/tidybot_description/urdf/tidybot.urdf (robot description, URDF)
Before this commit: robot tidybot, 20 links, 19 joints
Links:
- link arm_base_link: geometry collision mesh filename=file:///home/yuandi/tidybot_platform/install/tidybot_descri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; visual mesh filename=file:///home/yuandi/tidybot_platform/install/tidybot_descri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
- link base: geometry collision mesh filename=file:///home/yuandi/tidybot_platform/install/tidybot_descri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; collision mesh filename=file:///home/yuandi/tidybot_platform/install/tidybot_descri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
- link bracelet_link: geometry collision mesh filename=file:///home/yuandi/tidybot_platform/install/tidybot_descri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; visual mesh filename=file:///home/yuandi/tidybot_platform/install/tidybot_descri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
- link forearm_link: geometry collision mesh filename=file:///home/yuandi/tidybot_platform/install/tidybot_descri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; visual mesh filename=file:///home/yuandi/tidybot_platform/install/tidybot_descri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
- link gripper_base_link: geometry visual mesh filename=file:///home/yuandi/tidybot_platform/install/tidybot_descri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
- link half_arm_1_link: geometry collision mesh filename=file:///home/yuandi/tidybot_platform/install/tidybot_descri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; visual mesh filename=file:///home/yuandi/tidybot_platform/install/tidybot_descri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
- link half_arm_2_link: geometry collision mesh filename=file:///home/yuandi/tidybot_platform/install/tidybot_descri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; visual mesh filename=file:///home/yuandi/tidybot_platform/install/tidybot_descri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
- link left_finger_dist_link: geometry visual mesh filename=file:///home/yuandi/tidybot_platform/install/tidybot_descri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
- link left_finger_prox_link: geometry visual mesh filename=file:///home/yuandi/tidybot_platform/install/tidybot_descri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
- link right_finger_dist_link: geometry visual mesh filename=file:///home/yuandi/tidybot_platform/install/tidybot_descri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
- link right_finger_prox_link: geometry visual mesh filename=file:///home/yuandi/tidybot_platform/install/tidybot_descri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
- link shoulder_link: geometry collision mesh filename=file:///home/yuandi/tidybot_platform/install/tidybot_descri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; visual mesh filename=file:///home/yuandi/tidybot_platform/install/tidybot_descri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
- link spherical_wrist_1_link: geometry collision mesh filename=file:///home/yuandi/tidybot_platform/install/tidybot_descri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; visual mesh filename=file:///home/yuandi/tidybot_platform/install/tidybot_descri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
- link spherical_wrist_2_link: geometry collision mesh filename=file:///home/yuandi/tidybot_platform/install/tidybot_descri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; visual mesh filename=file:///home/yuandi/tidybot_platform/install/tidybot_descri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

Commit message: add episode recorder

File: src/tidybot_description/urdf/tidybot.urdf (robot description, URDF)
Before this commit: robot tidybot, 23 links, 22 joints
Links:
- link arm_base_link: geometry collision mesh filename=file:///home/janchen/Documents/tidybot_platform/install/tid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; visual mesh filename=file:///home/janchen/Documents/tidybot_platform/install/tid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
- link base: geometry collision mesh filename=file:///home/janchen/Documents/tidybot_platform/install/tid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; collision mesh filename=file:///home/janchen/Documents/tidybot_platform/install/tid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
- link bracelet_link: geometry collision mesh filename=file:///home/janchen/Documents/tidybot_platform/install/tid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; visual mesh filename=file:///home/janchen/Documents/tidybot_platform/install/tid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
- link forearm_link: geometry collision mesh filename=file:///home/janchen/Documents/tidybot_platform/install/tid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; visual mesh filename=file:///home/janchen/Documents/tidybot_platform/install/tid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
- link gripper_base_link: geometry visual mesh filename=file:///home/janchen/Documents/tidybot_platform/install/tid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
- link half_arm_1_link: geometry collision mesh filename=file:///home/janchen/Documents/tidybot_platform/install/tid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; visual mesh filename=file:///home/janchen/Documents/tidybot_platform/install/tid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
- link half_arm_2_link: geometry collision mesh filename=file:///home/janchen/Documents/tidybot_platform/install/tid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; visual mesh filename=file:///home/janchen/Documents/tidybot_platform/install/tid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
- link left_finger_dist_link: geometry visual mesh filename=file:///home/janchen/Documents/tidybot_platform/install/tid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
- link left_finger_prox_link: geometry visual mesh filename=file:///home/janchen/Documents/tidybot_platform/install/tid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
- link right_finger_dist_link: geometry visual mesh filename=file:///home/janchen/Documents/tidybot_platform/install/tid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
- link right_finger_prox_link: geometry visual mesh filename=file:///home/janchen/Documents/tidybot_platform/install/tid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
- link shoulder_link: geometry collision mesh filename=file:///home/janchen/Documents/tidybot_platform/install/tid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; visual mesh filename=file:///home/janchen/Documents/tidybot_platform/install/tid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
- link spherical_wrist_1_link: geometry collision mesh filename=file:///home/janchen/Documents/tidybot_platform/install/tid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; visual mesh filename=file:///home/janchen/Documents/tidybot_platform/install/tid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
- link spherical_wrist_2_link: geometry collision mesh filename=file:///home/janchen/Documents/tidybot_platform/install/tid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; visual mesh filename=file:///home/janchen/Documents/tidybot_platform/install/tid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

Commit message: add joint trajectory publisher

File: src/tidybot_description/urdf/tidybot.urdf (robot description, URDF)
Before this commit: robot tidybot, 29 links, 28 joints
Links:
- link arm_base_link: geometry collision mesh filename=file:///home/yuandi/tidybot_platform/install/tidybot_descri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; visual mesh filename=file:///home/yuandi/tidybot_platform/install/tidybot_descri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
- link base: geometry collision mesh filename=file:///home/yuandi/tidybot_platform/install/tidybot_descri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; collision mesh filename=file:///home/yuandi/tidybot_platform/install/tidybot_descri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
- link bracelet_link: geometry collision mesh filename=file:///home/yuandi/tidybot_platform/install/tidybot_descri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; visual mesh filename=file:///home/yuandi/tidybot_platform/install/tidybot_descri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
- link forearm_link: geometry collision mesh filename=file:///home/yuandi/tidybot_platform/install/tidybot_descri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; visual mesh filename=file:///home/yuandi/tidybot_platform/install/tidybot_descri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
- link half_arm_1_link: geometry collision mesh filename=file:///home/yuandi/tidybot_platform/install/tidybot_descri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; visual mesh filename=file:///home/yuandi/tidybot_platform/install/tidybot_descri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
- link half_arm_2_link: geometry collision mesh filename=file:///home/yuandi/tidybot_platform/install/tidybot_descri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; visual mesh filename=file:///home/yuandi/tidybot_platform/install/tidybot_descri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
- link left_inner_finger: geometry collision mesh filename=file:///home/yuandi/tidybot_platform/install/tidybot_descri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 scale=0.001 0.001 0.001; visual mesh filename=file:///home/yuandi/tidybot_platform/install/tidybot_descri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 scale=0.001 0.001 0.001
- link left_inner_knuckle: geometry collision mesh filename=file:///home/yuandi/tidybot_platform/install/tidybot_descri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 scale=0.001 0.001 0.001; visual mesh filename=file:///home/yuandi/tidybot_platform/install/tidybot_descri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 scale=0.001 0.001 0.001
- link left_outer_finger: geometry collision mesh filename=file:///home/yuandi/tidybot_platform/install/tidybot_descri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 scale=0.001 0.001 0.001; visual mesh filename=file:///home/yuandi/tidybot_platform/install/tidybot_descri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 scale=0.001 0.001 0.001
- link left_outer_knuckle: geometry collision mesh filename=file:///home/yuandi/tidybot_platform/install/tidybot_descri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 scale=0.001 0.001 0.001; visual mesh filename=file:///home/yuandi/tidybot_platform/install/tidybot_descri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 scale=0.001 0.001 0.001
- link right_inner_finger: geometry collision mesh filename=file:///home/yuandi/tidybot_platform/install/tidybot_descri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 scale=0.001 0.001 0.001; visual mesh filename=file:///home/yuandi/tidybot_platform/install/tidybot_descri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 scale=0.001 0.001 0.001
- link right_inner_knuckle: geometry collision mesh filename=file:///home/yuandi/tidybot_platform/install/tidybot_descri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 scale=0.001 0.001 0.001; visual mesh filename=file:///home/yuandi/tidybot_platform/install/tidybot_descri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 scale=0.001 0.001 0.001
- link right_outer_finger: geometry collision mesh filename=file:///home/yuandi/tidybot_platform/install/tidybot_descri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 scale=0.001 0.001 0.001; visual mesh filename=file:///home/yuandi/tidybot_platform/install/tidybot_descri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 scale=0.001 0.001 0.001
- link right_outer_knuckle: geometry collision mesh filename=file:///home/yuandi/tidybot_platform/install/tidybot_descri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 scale=0.001 0.001 0.001; visual mesh filename=file:///home/yuandi/tidybot_platform/install/tidybot_descri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 scale=0.001 0.001 0.001
- link robotiq_arg2f_base_link: geometry collision mesh filename=file:///home/yuandi/tidybot_platform/install/tidybot_descri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; visual mesh filename=file:///home/yuandi/tidybot_platform/install/tidybot_descri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
- link shoulder_link: geometry collision mesh filename=file:///home/yuandi/tidybot_platform/install/tidybot_descri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; visual mesh filename=file:///home/yuandi/tidybot_platform/install/tidybot_descri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
- link spherical_wrist_1_link: geometry collision mesh filename=file:///home/yuandi/tidybot_platform/install/tidybot_descri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; visual mesh filename=file:///home/yuandi/tidybot_platform/install/tidybot_descri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
- link spherical_wrist_2_link: geometry collision mesh filename=file:///home/yuandi/tidybot_platform/install/tidybot_descri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; visual mesh filename=file:///home/yuandi/tidybot_platform/install/tidybot_descri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

File: src/tidybot_description/urdf/tidybot.xacro (robot description, xacro)
@@ -4,6 +4,6 @@
     <xacro:arg name="hardware_plugin" default="gz_ros2_control/GazeboSimSystem" />
     <xacro:arg name="arm" default="gen3_7dof" />
-    <xacro:arg name="gripper" default="gen3_lite_2f" />
-    <xacro:arg name="vision" default="false" />
+    <xacro:arg name="gripper" default="robotiq_2f_85" />
+    <xacro:arg name="vision" default="true" />
     <xacro:arg name="prefix" default="" />
     <xacro:arg name="ros2_control_config_path" default="$(find tidybot_description)/config/tidybot_controllers.yaml"/>
@@ -13,7 +13,7 @@
     <!-- configure ros2_control joints -->
     <xacro:include filename="$(find tidybot_description)/urdf/tidybot.ros2_control.xacro" />
-    <xacro:load_ros2_control hardware_plugin="$(arg hardware_plugin)" arm="$(arg arm)" />
+    <xacro:load_ros2_control hardware_plugin="$(arg hardware_plugin)" arm="$(arg arm)" gripper="$(arg gripper)" />
     <!-- load gazebo plugins -->
     <xacro:include filename="$(find tidybot_description)/urdf/tidybot.gazebo.xacro" />
-    <xacro:load_gazebo_plugins config_path="$(arg ros2_control_config_path)" prefix="$(arg prefix) " arm="$(arg arm)" />
+    <xacro:load_gazebo_plugins config_path="$(arg ros2_control_config_path)" prefix="$(arg prefix) " arm="$(arg arm)" vision="$(arg vision)" />
 </robot>
