Commit message: move vla code to src/external

File: src/tidybot_description/urdf/tidybot.urdf (robot description, URDF)
Before this commit: robot tidybot, 30 links, 29 joints
Links:
- link arm_base_link: geometry collision mesh filename=file:///home/yuandi/Documents/tidybot_platform/install/tidy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; visual mesh filename=file:///home/yuandi/Documents/tidybot_platform/install/tidy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
- link base: geometry collision mesh filename=file:///home/yuandi/Documents/tidybot_platform/install/tidy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; visual mesh filename=file:///home/yuandi/Documents/tidybot_platform/install/tidy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
- link bracelet_link: geometry collision mesh filename=file:///home/yuandi/Documents/tidybot_platform/install/tidy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; visual mesh filename=file:///home/yuandi/Documents/tidybot_platform/install/tidy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
- link forearm_link: geometry collision mesh filename=file:///home/yuandi/Documents/tidybot_platform/install/tidy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; visual mesh filename=file:///home/yuandi/Documents/tidybot_platform/install/tidy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
- link half_arm_1_link: geometry collision mesh filename=file:///home/yuandi/Documents/tidybot_platform/install/tidy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; visual mesh filename=file:///home/yuandi/Documents/tidybot_platform/install/tidy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
- link half_arm_2_link: geometry collision mesh filename=file:///home/yuandi/Documents/tidybot_platform/install/tidy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; visual mesh filename=file:///home/yuandi/Documents/tidybot_platform/install/tidy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
- link left_inner_finger: geometry collision mesh filename=file:///home/yuandi/Documents/tidybot_platform/install/tidy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 scale=0.001 0.001 0.001; visual mesh filename=file:///home/yuandi/Documents/tidybot_platform/install/tidy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 scale=0.001 0.001 0.001
- link left_inner_knuckle: geometry collision mesh filename=file:///home/yuandi/Documents/tidybot_platform/install/tidy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 scale=0.001 0.001 0.001; visual mesh filename=file:///home/yuandi/Documents/tidybot_platform/install/tidy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 scale=0.001 0.001 0.001
- link left_outer_finger: geometry collision mesh filename=file:///home/yuandi/Documents/tidybot_platform/install/tidy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 scale=0.001 0.001 0.001; visual mesh filename=file:///home/yuandi/Documents/tidybot_platform/install/tidy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 scale=0.001 0.001 0.001
- link left_outer_knuckle: geometry collision mesh filename=file:///home/yuandi/Documents/tidybot_platform/install/tidy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 scale=0.001 0.001 0.001; visual mesh filename=file:///home/yuandi/Documents/tidybot_platform/install/tidy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 scale=0.001 0.001 0.001
- link right_inner_finger: geometry collision mesh filename=file:///home/yuandi/Documents/tidybot_platform/install/tidy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 scale=0.001 0.001 0.001; visual mesh filename=file:///home/yuandi/Documents/tidybot_platform/install/tidy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 scale=0.001 0.001 0.001
- link right_inner_knuckle: geometry collision mesh filename=file:///home/yuandi/Documents/tidybot_platform/install/tidy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 scale=0.001 0.001 0.001; visual mesh filename=file:///home/yuandi/Documents/tidybot_platform/install/tidy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 scale=0.001 0.001 0.001
- link right_outer_finger: geometry collision mesh filename=file:///home/yuandi/Documents/tidybot_platform/install/tidy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 scale=0.001 0.001 0.001; visual mesh filename=file:///home/yuandi/Documents/tidybot_platform/install/tidy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 scale=0.001 0.001 0.001
- link right_outer_knuckle: geometry collision mesh filename=file:///home/yuandi/Documents/tidybot_platform/install/tidy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 scale=0.001 0.001 0.001; visual mesh filename=file:///home/yuandi/Documents/tidybot_platform/install/tidy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 scale=0.001 0.001 0.001
- link robotiq_arg2f_base_link: geometry collision mesh filename=file:///home/yuandi/Documents/tidybot_platform/install/tidy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; visual mesh filename=file:///home/yuandi/Documents/tidybot_platform/install/tidy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
- link shoulder_link: geometry collision mesh filename=file:///home/yuandi/Documents/tidybot_platform/install/tidy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; visual mesh filename=file:///home/yuandi/Documents/tidybot_platform/install/tidy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
- link spherical_wrist_1_link: geometry collision mesh filename=file:///home/yuandi/Documents/tidybot_platform/install/tidy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; visual mesh filename=file:///home/yuandi/Documents/tidybot_platform/install/tidy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
- link spherical_wrist_2_link: geometry collision mesh filename=file:///home/yuandi/Documents/tidybot_platform/install/tidy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; visual mesh filename=file:///home/yuandi/Documents/tidybot_platform/install/tidy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
