Commit message: update the gripper model to include the out_finger_joints; add instruction to create the inner_knuckle joints in Isaac Sim

File: src/tidybot_description/urdf/arm.xacro (robot description, xacro)
@@ -1,4 +1,5 @@
 <?xml version="1.0"?>
-<robot name="arm_only" xmlns:xacro="http://ros.org/wiki/xacro">
+<robot name="arm_only"
+    xmlns:xacro="http://ros.org/wiki/xacro">
     <link name="world"/>
     <xacro:arg name="hardware_plugin" default="gz_ros2_control/GazeboSimSystem" />
@@ -40,8 +41,8 @@
         </xacro:if>
         <xacro:if value="${'$(arg gripper)' == 'gen3_lite_2f'}">
-                <xacro:add_joint name="right_finger_bottom_joint" gain="0.1" cmd_interface="position" init_pos="0.0"/>
-                <xacro:add_joint name="right_finger_tip_joint" gain="0.1" cmd_interface="position" init_pos="0.0"/>
-                <xacro:add_joint name="left_finger_bottom_joint" gain="0.1" cmd_interface="position" init_pos="0.0"/>
-                <xacro:add_joint name="left_finger_tip_joint" gain="0.1" cmd_interface="position" init_pos="0.0"/>
+            <xacro:add_joint name="right_finger_bottom_joint" gain="0.1" cmd_interface="position" init_pos="0.0"/>
+            <xacro:add_joint name="right_finger_tip_joint" gain="0.1" cmd_interface="position" init_pos="0.0"/>
+            <xacro:add_joint name="left_finger_bottom_joint" gain="0.1" cmd_interface="position" init_pos="0.0"/>
+            <xacro:add_joint name="left_finger_tip_joint" gain="0.1" cmd_interface="position" init_pos="0.0"/>
         </xacro:if>
         <!-- <xacro:add_joint name="joint_1" gain="0.1" cmd_interface="position" init_pos="0.0"/>
@@ -55,7 +56,7 @@
         </xacro:if> -->
         <xacro:if value="${'$(arg gripper)' == 'robotiq_2f_85'}">
-            <joint name ="left_outer_knuckle_joint">
+            <joint name ="finger_joint">
                 <command_interface name="position"/>
-                <state_interface name="position" >
+                <state_interface name="position">
                     <param name="initial_value">0.0</param>
                 </state_interface>
@@ -64,5 +65,5 @@
             </joint>
             <joint name ="right_inner_finger_joint">
-                <param name="mimic">left_outer_knuckle_joint</param>
+                <param name="mimic">finger_joint</param>
                 <param name="multiplier">-1.0</param>
                 <state_interface name="position">
@@ -72,5 +73,5 @@
             </joint>
             <joint name ="right_outer_knuckle_joint">
-                <param name="mimic">left_outer_knuckle_joint</param>
+                <param name="mimic">finger_joint</param>
                 <param name="multiplier">1.0</param>
                 <state_interface name="position">
@@ -79,6 +80,6 @@
                 <state_interface name="velocity"/>
             </joint>
-            <joint name ="right_inner_knuckle_joint">
-                <param name="mimic">left_outer_knuckle_joint</param>
+            <joint name ="right_inner_finger_knuckle_joint">
+                <param name="mimic">finger_joint</param>
                 <param name="multiplier">1.0</param>
                 <state_interface name="position">
@@ -88,5 +89,5 @@
             </joint>
             <joint name ="left_inner_finger_joint">
-                <param name="mimic">left_outer_knuckle_joint</param>
+                <param name="mimic">finger_joint</param>
                 <param name="multiplier">-1.0</param>
                 <state_interface name="position">
@@ -95,7 +96,23 @@
                 <state_interface name="velocity"/>
             </joint>
-            <joint name ="left_inner_knuckle_joint">
-                <param name="mimic">left_outer_knuckle_joint</param>
+            <joint name ="left_inner_finger_knuckle_joint">
+                <param name="mimic">finger_joint</param>
                 <param name="multiplier">1.0</param>
+                <state_interface name="position">
+                    <param name="initial_value">0.0</param>
+                </state_interface>
+                <state_interface name="velocity"/>
+            </joint>
+            <joint name ="left_outer_finger_joint">
+                <param name="mimic">finger_joint</param>
+                <param name="multiplier">0.0</param>
+                <state_interface name="position">
+                    <param name="initial_value">0.0</param>
+                </state_interface>
+                <state_interface name="velocity"/>
+            </joint>
+            <joint name ="right_outer_finger_joint">
+                <param name="mimic">finger_joint</param>
+                <param name="multiplier">0.0</param>
                 <state_interface name="position">
                     <param name="initial_value">0.0</param>
@@ -120,22 +137,22 @@
                 <visualize>true</visualize>
                 <pose>0 -0.01 0.03 0 4.7124 1.5708</pose>
-                        <topic>/arm_camera</topic>
+                <topic>/arm_camera</topic>
                 <gz_frame_id>arm_camera_link</gz_frame_id>
                 <camera>
-                <horizontal_fov>1.247</horizontal_fov>
-                <image>
-                    <width>640</width>
-                    <height>480</height>
-                    <format>R8G8B8</format>
-                </image>
-                <clip>
-                    <near>0.03</near>
-                    <far>3.0</far>
-                </clip>
-                <noise>
-                    <type>gaussian</type>
-                    <mean>0.0</mean>
-                    <stddev>0.007</stddev>
-                </noise>
+                    <horizontal_fov>1.247</horizontal_fov>
+                    <image>
+                        <width>640</width>
+                        <height>480</height>
+                        <format>R8G8B8</format>
+                    </image>
+                    <clip>
+                        <near>0.03</near>
+                        <far>3.0</far>
+                    </clip>
+                    <noise>
+                        <type>gaussian</type>
+                        <mean>0.0</mean>
+                        <stddev>0.007</stddev>
+                    </noise>
                 </camera>
             </sensor>

File: src/tidybot_description/urdf/bot.xacro (robot description, xacro)
@@ -1,17 +1,17 @@
 <?xml version="1.0"?>
 <robot xmlns:xacro="http://ros.org/wiki/xacro">
-<xacro:macro name="load_bot" params="arm gripper vision prefix">
-    <!-- load the corresponding macros -->
-    <xacro:include filename="$(find tidybot_description)/urdf/arms/${arm}/${arm}_macro.xacro" />
-    <xacro:include filename="$(find tidybot_description)/urdf/grippers/${gripper}/${gripper}_macro.xacro" />
-    <xacro:include filename="$(find tidybot_description)/urdf/base/tidybot++/base_kinova_macro.xacro" />
-    <!-- load the base -->
-    <xacro:load_base parent="" prefix="${prefix}" vision="${vision}" />
-    <!-- load the arm -->
-    <xacro:load_arm parent="${last_base_link}" vision="${vision}" prefix="${prefix}">
-        <origin xyz="0.12 3.76986e-15 0.374775" rpy="0 0 0" />
-    </xacro:load_arm>
-    <!-- load the gripper -->
-    <xacro:load_gripper parent="${prefix}${last_arm_link}" prefix="${prefix}" />
+    <xacro:macro name="load_bot" params="arm gripper vision prefix">
+        <!-- load the corresponding macros -->
+        <xacro:include filename="$(find tidybot_description)/urdf/arms/${arm}/${arm}_macro.xacro" />
+        <xacro:include filename="$(find tidybot_description)/urdf/grippers/${gripper}/${gripper}_macro.xacro" />
+        <xacro:include filename="$(find tidybot_description)/urdf/base/tidybot++/base_kinova_macro.xacro" />
+        <!-- load the base -->
+        <xacro:load_base parent="" prefix="${prefix}" vision="${vision}" />
+        <!-- load the arm -->
+        <xacro:load_arm parent="${last_base_link}" vision="${vision}" prefix="${prefix}">
+            <origin xyz="0.12 3.76986e-15 0.374775" rpy="0 0 0" />
+        </xacro:load_arm>
+        <!-- load the gripper -->
+        <xacro:load_gripper parent="${prefix}${last_arm_link}" prefix="${prefix}" />
     </xacro:macro>
 </robot>

File: src/tidybot_description/urdf/grippers/robotiq_2f_85/robotiq_2f_85_macro.xacro (robot description, xacro)
@@ -3,9 +3,11 @@
   Robotiq 2F-85 Gripper Loader
   Unified gripper definition compatible with both Isaac Sim and Gazebo.
-  Uses Isaac Sim kinematic structure with closed-loop kinematics.
+  Uses NVIDIA Isaac Sim coordinate system for consistency across simulators.
+  For Gazebo: outer_finger_joint is fixed (can't simulate closed-loop)
+  For Isaac Sim: Uses physics constraints via setup script
 -->
-<robot name="robotiq_arg2f_85_model" xmlns:xacro="http://ros.org/wiki/xacro">
+<robot name="robotiq_arg2f_85_model"
+  xmlns:xacro="http://ros.org/wiki/xacro">
   <xacro:macro name="load_gripper" params="parent prefix">
-    <xacro:include filename="$(find tidybot_description)/urdf/grippers/robotiq_2f_85/robotiq_arg2f.xacro" />
     <xacro:include filename="$(find tidybot_description)/urdf/grippers/robotiq_2f_85/robotiq_arg2f_85_model_macro.xacro" />
     <!-- Tool frame -->
@@ -17,12 +19,10 @@
       <axis xyz="0 0 0"/>
     </joint>
-    <!-- Gripper base link -->
-    <xacro:robotiq_arg2f_base_link prefix="${prefix}" parent="${parent}"/>
-    <!-- Left finger (reflect=1) -->
-    <xacro:finger_links prefix="${prefix}" fingerprefix="left" reflect="1"/>
-    <xacro:left_outer_knuckle_joint prefix="${prefix}"/>
-    <!-- Right finger (reflect=-1) -->
-    <xacro:finger_links prefix="${prefix}" fingerprefix="right" reflect="-1"/>
-    <xacro:right_outer_knuckle_joint prefix="${prefix}"/>
+    <!-- Gripper assembly (matching Isaac Sim coordinate system) -->
+    <!-- The gripper uses NVIDIA's coordinate frame (X forward, Z up) -->
+    <!-- Rotation aligns gripper with robot's end effector frame -->
+    <xacro:robotiq_gripper prefix="${prefix}" parent="${parent}">
+      <origin xyz="0.0 0.0 0.0" rpy="3.1415927 -1.5707964 1.5707964"/>
+    </xacro:robotiq_gripper>
   </xacro:macro>
 </robot>

File: src/tidybot_description/urdf/grippers/robotiq_2f_85/robotiq_2f_85_transmission.xacro (robot description, xacro)
@@ -2,14 +2,14 @@
 <robot xmlns:xacro="http://ros.org/wiki/xacro">
     <xacro:macro name="load_gripper_transmission" params="prefix">
-        <transmission name="${prefix}left_inner_knuckle_joint_trans">
+        <transmission name="${prefix}left_inner_finger_knuckle_joint_trans">
             <type>transmission_interface/SimpleTransmission</type>
-            <joint name="${prefix}left_inner_knuckle_joint" />
-            <actuator name="${prefix}left_inner_knuckle_joint_motor" />
+            <joint name="${prefix}left_inner_finger_knuckle_joint" />
+            <actuator name="${prefix}left_inner_finger_knuckle_joint_motor" />
             <mechanicalReduction>1</mechanicalReduction>
         </transmission>
-        <transmission name="${prefix}right_inner_knuckle_joint_trans">
+        <transmission name="${prefix}right_inner_finger_knuckle_joint_trans">
             <type>transmission_interface/SimpleTransmission</type>
-            <joint name="${prefix}right_inner_knuckle_joint" />
-            <actuator name="${prefix}right_inner_knuckle_joint_motor" />
+            <joint name="${prefix}right_inner_finger_knuckle_joint" />
+            <actuator name="${prefix}right_inner_finger_knuckle_joint_motor" />
             <mechanicalReduction>1</mechanicalReduction>
         </transmission>
@@ -26,8 +26,8 @@
             <mechanicalReduction>1</mechanicalReduction>
         </transmission>
-        <transmission name="${prefix}left_outer_knuckle_joint_trans">
+        <transmission name="${prefix}finger_joint_trans">
             <type>transmission_interface/SimpleTransmission</type>
-            <joint name="${prefix}left_outer_knuckle_joint" />
-            <actuator name="${prefix}left_outer_knuckle_joint_motor" />
+            <joint name="${prefix}finger_joint" />
+            <actuator name="${prefix}finger_joint_motor" />
             <mechanicalReduction>1</mechanicalReduction>
         </transmission>
@@ -38,4 +38,16 @@
             <mechanicalReduction>1</mechanicalReduction>
         </transmission>
+        <transmission name="${prefix}left_outer_finger_joint_trans">
+            <type>transmission_interface/SimpleTransmission</type>
+            <joint name="${prefix}left_outer_finger_joint" />
+            <actuator name="${prefix}left_outer_finger_joint_motor" />
+            <mechanicalReduction>1</mechanicalReduction>
+        </transmission>
+        <transmission name="${prefix}right_outer_finger_joint_trans">
+            <type>transmission_interface/SimpleTransmission</type>
+            <joint name="${prefix}right_outer_finger_joint" />
+            <actuator name="${prefix}right_outer_finger_joint_motor" />
+            <mechanicalReduction>1</mechanicalReduction>
+        </transmission>
     </xacro:macro>
 </robot>
