Commit message: update the gripper model to include the out_finger_joints; add instruction to create the inner_knuckle joints in Isaac Sim

File: src/tidybot_description/urdf/grippers/robotiq_2f_85/robotiq_arg2f_85_model_macro.xacro (robot description, xacro)
@@ -2,29 +2,51 @@
 <!--
   Robotiq 2F-85 Gripper - Unified model compatible with both Isaac Sim and Gazebo
-  This xacro uses the Isaac Sim kinematic structure with closed-loop kinematics.
-  Joint hierarchy: outer_knuckle -> outer_finger -> inner_finger -> inner_knuckle
-  Uses STL meshes converted from Isaac Sim export for compatibility across simulators.
 -->
 <robot xmlns:xacro="http://ros.org/wiki/xacro">
-  <!-- Mesh directory -->
+  <!-- Mesh directory - uses STL for Gazebo compatibility -->
   <xacro:property name="mesh_dir" value="file://$(find tidybot_description)/meshes/grippers/robotiq_2f_85"/>
   <!-- ============================================ -->
-  <!-- Link Definitions -->
-  <!-- ============================================ -->
-  <!-- Outer Knuckle Link -->
-  <xacro:macro name="outer_knuckle" params="prefix fingerprefix reflect">
-    <link name="${prefix}${fingerprefix}_outer_knuckle">
-      <inertial>
-        <origin xyz="${reflect * 0.0121152} ${reflect * -0.000638} 0." rpy="0. 0. 0."/>
+  <!-- Base Link -->
+  <!-- ============================================ -->
+  <xacro:macro name="robotiq_base_link" params="prefix">
+    <link name="${prefix}robotiq_arg2f_base_link">
+      <inertial>
+        <origin xyz="0.0320809 0.0000006 0.0000228" rpy="0. 0. 0."/>
+        <mass value="0.6098911"/>
+        <inertia ixx="0.0004747" ixy="-0." ixz="0." iyy="0.0003629" iyz="0." izz="0.0005407"/>
+      </inertial>
+      <visual>
+        <origin xyz="-0.000242 0. 0." rpy="0. 0. -1.5707964"/>
+        <geometry>
+          <mesh filename="${mesh_dir}/robotiq_arg2f_85_base_link.stl"/>
+        </geometry>
+        <material name="">
+          <color rgba="0.1 0.1 0.1 1.0"/>
+        </material>
+      </visual>
+      <collision>
+        <origin xyz="-0.000242 0. 0." rpy="0. 0. -1.5707964"/>
+        <geometry>
+          <mesh filename="${mesh_dir}/robotiq_arg2f_85_base_link.stl"/>
+        </geometry>
+      </collision>
+    </link>
+    <gazebo reference="${prefix}robotiq_arg2f_base_link">
+      <material>Gazebo/DarkGrey</material>
+    </gazebo>
+  </xacro:macro>
+  <!-- ============================================ -->
+  <!-- Link Definitions (matching Isaac Sim URDF) -->
+  <!-- ============================================ -->
+  <!-- Left Outer Knuckle -->
+  <xacro:macro name="left_outer_knuckle" params="prefix">
+    <link name="${prefix}left_outer_knuckle">
+      <inertial>
+        <origin xyz="-0.012132 -0.000586 0." rpy="0. 0. 0."/>
         <mass value="0.0127346"/>
         <inertia ixx="0.0000003" ixy="0." ixz="0." iyy="0.0000021" iyz="0." izz="0.0000021"/>
       </inertial>
       <visual>
-        <xacro:if value="${reflect > 0}">
-          <origin xyz="-0.0306 -0.05466 0." rpy="${-pi} 0. ${pi}"/>
-        </xacro:if>
-        <xacro:if value="${reflect &lt; 0}">
-          <origin xyz="0.0306 0.05466 0." rpy="${-pi} 0. 0."/>
-        </xacro:if>
+        <origin xyz="0.0292492 -0.0556365 0." rpy="0. 0. -0.0244589"/>
         <geometry>
           <mesh filename="${mesh_dir}/robotiq_arg2f_85_outer_knuckle.stl"/>
@@ -35,10 +57,5 @@
       </visual>
       <collision>
-        <xacro:if value="${reflect > 0}">
-          <origin xyz="-0.0306 -0.05466 0." rpy="${-pi} 0. ${pi}"/>
-        </xacro:if>
-        <xacro:if value="${reflect &lt; 0}">
-          <origin xyz="0.0306 0.05466 0." rpy="${-pi} 0. 0."/>
-        </xacro:if>
+        <origin xyz="0.0292492 -0.0556365 0." rpy="0. 0. -0.0244589"/>
         <geometry>
           <mesh filename="${mesh_dir}/robotiq_arg2f_85_outer_knuckle.stl"/>
@@ -46,18 +63,46 @@
       </collision>
     </link>
-    <gazebo reference="${prefix}${fingerprefix}_outer_knuckle">
+    <gazebo reference="${prefix}left_outer_knuckle">
       <material>Gazebo/Grey</material>
     </gazebo>
   </xacro:macro>
-  <!-- Outer Finger Link -->
-  <xacro:macro name="outer_finger" params="prefix fingerprefix reflect">
-    <link name="${prefix}${fingerprefix}_outer_finger">
-      <inertial>
-        <origin xyz="${reflect * 0.0000055} ${reflect * -0.0659505} 0.0689531" rpy="0. 0. 0."/>
+  <!-- Right Outer Knuckle -->
+  <xacro:macro name="right_outer_knuckle" params="prefix">
+    <link name="${prefix}right_outer_knuckle">
+      <inertial>
+        <origin xyz="0.012132 0.000586 0." rpy="0. 0. 0."/>
+        <mass value="0.0127346"/>
+        <inertia ixx="0.0000003" ixy="0." ixz="-0." iyy="0.0000021" iyz="0." izz="0.0000021"/>
+      </inertial>
+      <visual>
+        <origin xyz="-0.0292492 0.0556365 0." rpy="0. 0. 3.1171339"/>
+        <geometry>
+          <mesh filename="${mesh_dir}/robotiq_arg2f_85_outer_knuckle.stl"/>
+        </geometry>
+        <material name="">
+          <color rgba="0.792 0.820 0.933 1.0"/>
+        </material>
+      </visual>
+      <collision>
+        <origin xyz="-0.0292492 0.0556365 0." rpy="0. 0. 3.1171339"/>
+        <geometry>
+          <mesh filename="${mesh_dir}/robotiq_arg2f_85_outer_knuckle.stl"/>
+        </geometry>
+      </collision>
+    </link>
+    <gazebo reference="${prefix}right_outer_knuckle">
+      <material>Gazebo/Grey</material>
+    </gazebo>
+  </xacro:macro>
+  <!-- Left Outer Finger -->
+  <xacro:macro name="left_outer_finger" params="prefix">
+    <link name="${prefix}left_outer_finger">
+      <inertial>
+        <origin xyz="-0.0039245 -0.0185808 -0.0000055" rpy="0. 0. 0."/>
         <mass value="0.0391792"/>
-        <inertia ixx="0.0000132" ixy="-0." ixz="-0." iyy="0.0000043" iyz="-0." izz="0.0000109"/>
-      </inertial>
-      <visual>
-        <origin xyz="0. 0. 0." rpy="${pi/2} ${reflect * -0.0000001} ${reflect * pi/2}"/>
+        <inertia ixx="0.0000043" ixy="0." ixz="-0." iyy="0.0000109" iyz="-0." izz="0.0000132"/>
+      </inertial>
+      <visual>
+        <origin xyz="0.062026 0.0503723 0." rpy="-3.1415927 0. 0."/>
         <geometry>
           <mesh filename="${mesh_dir}/robotiq_arg2f_85_outer_finger.stl"/>
@@ -68,5 +113,5 @@
       </visual>
       <collision>
-        <origin xyz="0. 0. 0." rpy="${pi/2} ${reflect * -0.0000001} ${reflect * pi/2}"/>
+        <origin xyz="0.062026 0.0503723 0." rpy="-3.1415927 0. 0."/>
         <geometry>
           <mesh filename="${mesh_dir}/robotiq_arg2f_85_outer_finger.stl"/>
@@ -74,13 +119,41 @@
       </collision>
     </link>
-    <gazebo reference="${prefix}${fingerprefix}_outer_finger">
-      <material>Gazebo/DarkGrey</material>
-    </gazebo>
-  </xacro:macro>
-  <!-- Inner Finger Link (includes pad) -->
-  <xacro:macro name="inner_finger" params="prefix fingerprefix reflect">
-    <link name="${prefix}${fingerprefix}_inner_finger">
-      <inertial>
-        <origin xyz="0.0185829 ${reflect * -0.0274476} 0." rpy="0. 0. 0."/>
+    <gazebo reference="${prefix}left_outer_finger">
+      <material>Gazebo/DarkGrey</material>
+    </gazebo>
+  </xacro:macro>
+  <!-- Right Outer Finger -->
+  <xacro:macro name="right_outer_finger" params="prefix">
+    <link name="${prefix}right_outer_finger">
+      <inertial>
+        <origin xyz="-0.0039245 -0.0185808 -0.0000055" rpy="0. 0. 0."/>
+        <mass value="0.0391792"/>
+        <inertia ixx="0.0000043" ixy="0." ixz="-0." iyy="0.0000109" iyz="-0." izz="0.0000132"/>
+      </inertial>
+      <visual>
+        <origin xyz="0.062026 0.0503723 0." rpy="3.1415927 0. 0."/>
+        <geometry>
+          <mesh filename="${mesh_dir}/robotiq_arg2f_85_outer_finger.stl"/>
+        </geometry>
+        <material name="">
+          <color rgba="0.2 0.2 0.2 1.0"/>
+        </material>
+      </visual>
+      <collision>
+        <origin xyz="0.062026 0.0503723 0." rpy="3.1415927 0. 0."/>
+        <geometry>
+          <mesh filename="${mesh_dir}/robotiq_arg2f_85_outer_finger.stl"/>
+        </geometry>
+      </collision>
+    </link>
+    <gazebo reference="${prefix}right_outer_finger">
+      <material>Gazebo/DarkGrey</material>
+    </gazebo>
+  </xacro:macro>
+  <!-- Left Inner Finger (includes pad) -->
+  <xacro:macro name="left_inner_finger" params="prefix">
+    <link name="${prefix}left_inner_finger">
+      <inertial>
+        <origin xyz="0.0189383 -0.0286037 -0.0133" rpy="0. 0. 0."/>
         <mass value="0.0197616"/>
         <inertia ixx="0.000001" ixy="0." ixz="-0." iyy="0.0000028" iyz="-0." izz="0.0000032"/>
@@ -88,10 +161,5 @@
       <!-- Inner finger body -->
       <visual>
-        <xacro:if value="${reflect > 0}">
-          <origin xyz="0.06776 0.09809 0." rpy="${-pi} 0. 0."/>
-        </xacro:if>
-        <xacro:if value="${reflect &lt; 0}">
-          <origin xyz="0.06776 -0.09809 0." rpy="0. 0. 0."/>
-        </xacro:if>
+        <origin xyz="0.071171 0.0956936 -0.0133" rpy="3.1415927 0. -0.0244594"/>
         <geometry>
           <mesh filename="${mesh_dir}/robotiq_arg2f_85_inner_finger.stl"/>
@@ -103,10 +171,5 @@
       <!-- Inner finger pad -->
       <visual>
-        <xacro:if value="${reflect > 0}">
-          <origin xyz="0.06776 0.09809 0." rpy="${-pi} 0. 0."/>
-        </xacro:if>
-        <xacro:if value="${reflect &lt; 0}">
-          <origin xyz="0.06776 -0.09809 0." rpy="0. 0. 0."/>
-        </xacro:if>
+        <origin xyz="0.071171 0.0956936 -0.0133" rpy="3.1415927 0. -0.0244594"/>
         <geometry>
           <mesh filename="${mesh_dir}/robotiq_arg2f_85_pad.stl"/>
@@ -117,10 +180,5 @@
       </visual>
       <collision>
-        <xacro:if value="${reflect > 0}">
-          <origin xyz="0.06776 0.09809 0." rpy="${-pi} 0. 0."/>
-        </xacro:if>
-        <xacro:if value="${reflect &lt; 0}">
-          <origin xyz="0.06776 -0.09809 0." rpy="0. 0. 0."/>
-        </xacro:if>
+        <origin xyz="0.071171 0.0956936 -0.0133" rpy="3.1415927 0. -0.0244594"/>
         <geometry>
           <mesh filename="${mesh_dir}/robotiq_arg2f_85_inner_finger.stl"/>
@@ -128,10 +186,5 @@
       </collision>
       <collision>
-        <xacro:if value="${reflect > 0}">
-          <origin xyz="0.06776 0.09809 0." rpy="${-pi} 0. 0."/>
-        </xacro:if>
-        <xacro:if value="${reflect &lt; 0}">
-          <origin xyz="0.06776 -0.09809 0." rpy="0. 0. 0."/>
-        </xacro:if>
+        <origin xyz="0.071171 0.0956936 -0.0133" rpy="3.1415927 0. -0.0244594"/>
         <geometry>
           <mesh filename="${mesh_dir}/robotiq_arg2f_85_pad.stl"/>
@@ -139,18 +192,63 @@
       </collision>
     </link>
-    <gazebo reference="${prefix}${fingerprefix}_inner_finger">
-      <material>Gazebo/DarkGrey</material>
-    </gazebo>
-  </xacro:macro>
-  <!-- Inner Knuckle Link -->
-  <xacro:macro name="inner_knuckle" params="prefix fingerprefix reflect">
-    <link name="${prefix}${fingerprefix}_inner_knuckle">
-      <inertial>
-        <origin xyz="0.0176393 -0.0211796 0." rpy="0. 0. 0."/>
+    <gazebo reference="${prefix}left_inner_finger">
+      <material>Gazebo/DarkGrey</material>
+    </gazebo>
+  </xacro:macro>
+  <!-- Right Inner Finger (includes pad) -->
+  <xacro:macro name="right_inner_finger" params="prefix">
+    <link name="${prefix}right_inner_finger">
+      <inertial>
+        <origin xyz="0.0189383 0.0286037 -0.0133" rpy="0. 0. 0."/>
+        <mass value="0.0197616"/>
+        <inertia ixx="0.000001" ixy="-0." ixz="0." iyy="0.0000028" iyz="0." izz="0.0000032"/>
+      </inertial>
+      <!-- Inner finger body -->
+      <visual>
+        <origin xyz="0.071171 -0.0956936 -0.0133" rpy="0. 0. 0.0244594"/>
+        <geometry>
+          <mesh filename="${mesh_dir}/robotiq_arg2f_85_inner_finger.stl"/>
+        </geometry>
+        <material name="">
+          <color rgba="0.2 0.2 0.2 1.0"/>
+        </material>
+      </visual>
+      <!-- Inner finger pad -->
+      <visual>
+        <origin xyz="0.071171 -0.0956936 -0.0133" rpy="0. 0. 0.0244594"/>
+        <geometry>
+          <mesh filename="${mesh_dir}/robotiq_arg2f_85_pad.stl"/>
+        </geometry>
+        <material name="">
+          <color rgba="0.1 0.1 0.1 1.0"/>
+        </material>
+      </visual>
+      <collision>
+        <origin xyz="0.071171 -0.0956936 -0.0133" rpy="0. 0. 0.0244594"/>
+        <geometry>
+          <mesh filename="${mesh_dir}/robotiq_arg2f_85_inner_finger.stl"/>
+        </geometry>
+      </collision>
+      <collision>
+        <origin xyz="0.071171 -0.0956936 -0.0133" rpy="0. 0. 0.0244594"/>
+        <geometry>
+          <mesh filename="${mesh_dir}/robotiq_arg2f_85_pad.stl"/>
+        </geometry>
+      </collision>
+    </link>
+    <gazebo reference="${prefix}right_inner_finger">
+      <material>Gazebo/DarkGrey</material>
+    </gazebo>
+  </xacro:macro>
+  <!-- Left Inner Knuckle -->
+  <xacro:macro name="left_inner_knuckle" params="prefix">
+    <link name="${prefix}left_inner_knuckle">
+      <inertial>
+        <origin xyz="0.0181803 -0.0209509 0." rpy="0. 0. 0."/>
         <mass value="0.0273069"/>
-        <inertia ixx="0.0000045" ixy="0." ixz="0." iyy="0.000008" iyz="-0." izz="0.0000118"/>
-      </inertial>
-      <visual>
-        <origin xyz="0.04986 -0.1046 0." rpy="0. 0. 0."/>
+        <inertia ixx="0.0000045" ixy="0.0000001" ixz="0." iyy="0.000008" iyz="0." izz="0.0000118"/>
+      </inertial>
+      <visual>
+        <origin xyz="0.0483511 -0.1051343 0." rpy="0. 0. -0.0244597"/>
         <geometry>
           <mesh filename="${mesh_dir}/robotiq_arg2f_85_inner_knuckle.stl"/>
@@ -161,5 +259,5 @@
       </visual>
       <collision>
-        <origin xyz="0.04986 -0.1046 0." rpy="0. 0. 0."/>
+        <origin xyz="0.0483511 -0.1051343 0." rpy="0. 0. -0.0244597"/>
         <geometry>
           <mesh filename="${mesh_dir}/robotiq_arg2f_85_inner_knuckle.stl"/>
@@ -167,98 +265,163 @@
       </collision>
     </link>
-    <gazebo reference="${prefix}${fingerprefix}_inner_knuckle">
-      <material>Gazebo/DarkGrey</material>
-    </gazebo>
-  </xacro:macro>
-  <!-- ============================================ -->
-  <!-- Joint Definitions -->
-  <!-- ============================================ -->
-  <!-- Left outer knuckle joint (leader joint - actuated) -->
-  <xacro:macro name="left_outer_knuckle_joint" params="prefix">
-    <joint name="${prefix}left_outer_knuckle_joint" type="revolute">
-      <origin xyz="0. -0.0306 0.05466" rpy="${pi/2} 0. ${-pi/2}"/>
+    <gazebo reference="${prefix}left_inner_knuckle">
+      <material>Gazebo/DarkGrey</material>
+    </gazebo>
+  </xacro:macro>
+  <!-- Right Inner Knuckle -->
+  <xacro:macro name="right_inner_knuckle" params="prefix">
+    <link name="${prefix}right_inner_knuckle">
+      <inertial>
+        <origin xyz="0.0181803 -0.0209509 0." rpy="0. 0. 0."/>
+        <mass value="0.0273069"/>
+        <inertia ixx="0.0000045" ixy="0.0000001" ixz="-0." iyy="0.000008" iyz="-0." izz="0.0000118"/>
+      </inertial>
+      <visual>
+        <origin xyz="0.0483511 -0.1051343 0." rpy="0. 0. -0.0244597"/>
+        <geometry>
+          <mesh filename="${mesh_dir}/robotiq_arg2f_85_inner_knuckle.stl"/>
+        </geometry>
+        <material name="">
+          <color rgba="0.2 0.2 0.2 1.0"/>
+        </material>
+      </visual>
+      <collision>
+        <origin xyz="0.0483511 -0.1051343 0." rpy="0. 0. -0.0244597"/>
+        <geometry>
+          <mesh filename="${mesh_dir}/robotiq_arg2f_85_inner_knuckle.stl"/>
+        </geometry>
+      </collision>
+    </link>
+    <gazebo reference="${prefix}right_inner_knuckle">
+      <material>Gazebo/DarkGrey</material>
+    </gazebo>
+  </xacro:macro>
+  <!-- ============================================ -->
+  <!-- Joint Definitions (matching Isaac Sim URDF) -->
+  <!-- ============================================ -->
+  <!-- Finger joint (leader - actuated) -->
+  <xacro:macro name="finger_joint" params="prefix">
+    <joint name="${prefix}finger_joint" type="revolute">
+      <origin xyz="0.0546625 0.0306011 0." rpy="0. 0. -1.5707964"/>
       <parent link="${prefix}robotiq_arg2f_base_link"/>
       <child link="${prefix}left_outer_knuckle"/>
+      <axis xyz="0. 0. -1."/>
+      <limit lower="0." upper="0.8203047" effort="26." velocity="2.5562093"/>
+      <dynamics damping="1.0" friction="0.5"/>
+    </joint>
+  </xacro:macro>
+  <!-- Left outer finger joint (Revolute for Isaac Sim spring mechanism) -->
+  <xacro:macro name="left_outer_finger_joint" params="prefix">
+    <joint name="${prefix}left_outer_finger_joint" type="revolute">
+      <origin xyz="-0.0315263 -0.0037623 0." rpy="3.1415927 0. -0.0244589"/>
+      <parent link="${prefix}left_outer_knuckle"/>
+      <child link="${prefix}left_outer_finger"/>
+      <axis xyz="0 0 1"/>
+      <limit lower="0.0" upper="0.0" effort="100" velocity="100"/>
+      <mimic joint="${prefix}finger_joint" multiplier="0.0" offset="0"/>
+      <dynamics damping="10.0" friction="10.0"/>
+    </joint>
+  </xacro:macro>
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
File: src/tidybot_description/urdf/tidybot.ros2_control.xacro (robot description, xacro)
@@ -39,8 +39,8 @@
             <!-- - Right outer knuckle: same value as left (mirrored frame, so same numeric value = symmetric motion) -->
             <!-- - Inner fingers: opposite direction to compensate outer knuckle rotation (keeps fingertips parallel) -->
-            <!-- - Inner knuckles: same direction as outer knuckle -->
+            <!-- - Inner finger knuckle joints: connects inner finger to inner knuckle -->
             <xacro:if value="${gripper == 'robotiq_2f_85'}">
                 <!-- Leader joint (actuated) -->
-                <joint name="left_outer_knuckle_joint">
+                <joint name="finger_joint">
                     <command_interface name="position"/>
                     <state_interface name="position">
@@ -51,5 +51,5 @@
                 <!-- Right outer knuckle (mimic, same numeric value for symmetric closing) -->
                 <joint name="right_outer_knuckle_joint">
-                    <param name="mimic">left_outer_knuckle_joint</param>
+                    <param name="mimic">finger_joint</param>
                     <param name="multiplier">1.0</param>
                     <state_interface name="position">
@@ -60,5 +60,5 @@
                 <!-- Left inner finger (mimic, opposite to keep fingertip parallel) -->
                 <joint name="left_inner_finger_joint">
-                    <param name="mimic">left_outer_knuckle_joint</param>
+                    <param name="mimic">finger_joint</param>
                     <param name="multiplier">-1.0</param>
                     <state_interface name="position">
@@ -69,5 +69,5 @@
                 <!-- Right inner finger (mimic) -->
                 <joint name="right_inner_finger_joint">
-                    <param name="mimic">left_outer_knuckle_joint</param>
+                    <param name="mimic">finger_joint</param>
                     <param name="multiplier">1.0</param>
                     <state_interface name="position">
@@ -76,7 +76,7 @@
                     <state_interface name="velocity"/>
                 </joint>
-                <!-- Left inner knuckle (mimic) -->
-                <joint name="left_inner_knuckle_joint">
-                    <param name="mimic">left_outer_knuckle_joint</param>
+                <!-- Left inner finger knuckle (mimic, connects inner finger to inner knuckle) -->
+                <joint name="left_inner_finger_knuckle_joint">
+                    <param name="mimic">finger_joint</param>
                     <param name="multiplier">-1.0</param>
                     <state_interface name="position">
@@ -85,7 +85,7 @@
                     <state_interface name="velocity"/>
                 </joint>
-                <!-- Right inner knuckle (mimic) -->
-                <joint name="right_inner_knuckle_joint">
-                    <param name="mimic">left_outer_knuckle_joint</param>
+                <!-- Right inner finger knuckle (mimic, connects inner finger to inner knuckle) -->
+                <joint name="right_inner_finger_knuckle_joint">
+                    <param name="mimic">finger_joint</param>
                     <param name="multiplier">-1.0</param>
                     <state_interface name="position">

File: src/tidybot_description/urdf/tidybot.xacro (robot description, xacro)
@@ -1,4 +1,5 @@
 <?xml version="1.0"?>
-<robot name="tidybot" xmlns:xacro="http://ros.org/wiki/xacro">
+<robot name="tidybot"
+    xmlns:xacro="http://ros.org/wiki/xacro">
     <!-- <xacro:arg name="hardware_plugin" default="mock_components/GenericSystem" />     -->
     <xacro:arg name="hardware_plugin" default="gz_ros2_control/GazeboSimSystem" />

File: src/tidybot_description/urdf/tidybot_isaac.urdf (robot description, URDF)
Before this commit: robot tidybot, 28 links, 27 joints
Joints:
- removed joint left_inner_knuckle_joint
- removed joint left_outer_knuckle_joint
- removed joint right_inner_knuckle_joint
- added joint finger_joint: type revolute, parent robotiq_arg2f_base_link, child left_outer_knuckle, origin xyz=0.0546625 0.0306011 0. rpy=0. 0. -1.5707964, axis 0. 0. -1., limit lower=0. upper=0.8203047 effort=26. velocity=2.5562093
- added joint left_inner_finger_knuckle_joint: type revolute, parent left_inner_finger, child left_inner_knuckle, origin xyz=0.0177368 -0.0069505 -0.0133 rpy=3.1415927 0. -0.0244594, axis 0. 0. 1., limit lower=-3.1415927 upper=3.1415927 effort=0. velocity=174.5329252
- added joint right_inner_finger_knuckle_joint: type revolute, parent right_inner_finger, child right_inner_knuckle, origin xyz=0.0177368 0.0069505 -0.0133 rpy=0. 0. 0.0244594, axis 0. 0. 1., limit lower=-3.1415927 upper=3.1415927 effort=0. velocity=174.5329252
- joint gripper_base_joint: origin xyz=0.0 0.0 0.0 rpy=0.0 0.0 1.57 -> xyz=0.0 0.0 0.0 rpy=3.1415927 -1.5707964 1.5707964
- joint left_inner_finger_joint: origin xyz=-0. -0.06776 0.09809 rpy=-1.5707963 -0.0000001 1.5707963 -> xyz=-0.0067834 -0.0470334 0.0133 rpy=0. 0. 0.
- joint left_outer_finger_joint: axis (none) -> 0 0 1; limit (none) -> lower=0 upper=3.14 effort=100 velocity=100; origin xyz=-0.0306 -0.05466 -0. rpy=-1.5707965 1.5707963 0. -> xyz=-0.0315263 -0.0037623 0. rpy=3.1415927 0. -0.0244589; type fixed -> revolute
- joint right_inner_finger_joint: origin xyz=-0. 0.06776 0.09809 rpy=1.5707964 0.0000001 -1.5707964 -> xyz=-0.0067834 -0.0470334 -0.0133 rpy=3.1415927 0. 0.
- joint right_outer_finger_joint: axis (none) -> 0 0 1; limit (none) -> lower=0.0 upper=3.14 effort=100 velocity=100; origin xyz=0.0306 0.05466 0. rpy=1.5707963 -1.5707963 0. -> xyz=0.0315263 0.0037623 0. rpy=3.1415927 0. 3.1171336; type fixed -> revolute
- joint right_outer_knuckle_joint: axis 0. 0. 1. -> 0. 0. -1.; limit lower=0. upper=0.8203047 effort=0. velocity=174.5329252 -> lower=-3.14 upper=3.14 effort=0. velocity=174.5329252; origin xyz=0. 0.0306 0.05466 rpy=-1.5707964 0. -1.5707964 -> xyz=0.0546625 -0.0306011 0. rpy=3.1415927 0. -1.5707964
