Commit message: add ros2 isaac sim bridge node and launch file

File: src/tidybot_description/urdf/tidybot_isaac.urdf (robot description, URDF)
Before this commit: robot tidybot, 30 links, 29 joints
Joints:
- joint joint_x: origin xyz=0.0 0.0 0.0 rpy=0.0 0.0 0.0 -> xyz=0.0 0.0 0.085 rpy=0.0 0.0 0.0
- joint left_inner_finger_joint: mimic joint=left_outer_knuckle_joint multiplier=-1 offset=0 -> (none)
- joint left_inner_knuckle_joint: mimic joint=left_outer_knuckle_joint multiplier=1 offset=0 -> (none)
- joint right_inner_finger_joint: mimic joint=left_outer_knuckle_joint multiplier=-1 offset=0 -> (none)
- joint right_inner_knuckle_joint: mimic joint=left_outer_knuckle_joint multiplier=1 offset=0 -> (none)
- joint right_outer_knuckle_joint: mimic joint=left_outer_knuckle_joint multiplier=1 offset=0 -> (none)

Commit message: update the robotiq_2f_85 gripper in isaac sim and add a flattened usd scene

File: src/tidybot_description/urdf/tidybot_isaac.urdf (robot description, URDF)
Before this commit: robot tidybot, 30 links, 29 joints
Links:
- removed link left_inner_finger_pad
- removed link right_inner_finger_pad
- link left_inner_finger: mass 0.0104003125914103 -> 0.0197616; geometry collision mesh filename=file:///tidybot_description/meshes/grippers/robotiq_2f_85_i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; collision mesh filename=file:///tidybot_description/meshes/grippers/robotiq_2f_85_i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
- link left_inner_knuckle: mass 0.0271177346495152 -> 0.0273069; geometry collision mesh filename=file:///tidybot_description/meshes/grippers/robotiq_2f_85_i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; visual mesh filename=file:///tidybot_description/meshes/grippers/robotiq_2f_85_i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
- link left_outer_finger: mass 0.022614240507152 -> 0.0391792; geometry collision mesh filename=file:///tidybot_description/meshes/grippers/robotiq_2f_85_i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; visual mesh filename=file:///tidybot_description/meshes/grippers/robotiq_2f_85_i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
- link left_outer_knuckle: mass 0.00853198276973456 -> 0.0127346; geometry collision mesh filename=file:///tidybot_description/meshes/grippers/robotiq_2f_85_i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; visual mesh filename=file:///tidybot_description/meshes/grippers/robotiq_2f_85_i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
- link right_inner_finger: mass 0.0104003125914103 -> 0.0197616; geometry collision mesh filename=file:///tidybot_description/meshes/grippers/robotiq_2f_85_i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; collision mesh filename=file:///tidybot_description/meshes/grippers/robotiq_2f_85_i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
- link right_inner_knuckle: mass 0.0271177346495152 -> 0.0273069; geometry collision mesh filename=file:///tidybot_description/meshes/grippers/robotiq_2f_85_i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; visual mesh filename=file:///tidybot_description/meshes/grippers/robotiq_2f_85_i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
- link right_outer_finger: mass 0.022614240507152 -> 0.0391792; geometry collision mesh filename=file:///tidybot_description/meshes/grippers/robotiq_2f_85_i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; visual mesh filename=file:///tidybot_description/meshes/grippers/robotiq_2f_85_i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
- link right_outer_knuckle: mass 0.00853198276973456 -> 0.0127346; geometry collision mesh filename=file:///tidybot_description/meshes/grippers/robotiq_2f_85_i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; visual mesh filename=file:///tidybot_description/meshes/grippers/robotiq_2f_85_i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
- link robotiq_arg2f_base_link: mass 0.22652 -> 0.6098911; geometry collision mesh filename=file:///tidybot_description/meshes/grippers/robotiq_2f_85_i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; visual mesh filename=file:///tidybot_description/meshes/grippers/robotiq_2f_85_i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
Joints:
- removed joint left_inner_finger_pad_joint
- removed joint right_inner_finger_pad_joint
- joint left_inner_finger_joint: axis 1 0 0 -> 0. 0. 1.; limit lower=-1.0 upper=1.0 effort=1000 velocity=1.0 -> lower=-3.1415927 upper=3.1415927 effort=0. velocity=174.5329252; origin xyz=0 0.0061 0.0471 rpy=0 0 0 -> xyz=-0. -0.06776 0.09809 rpy=-1.5707963 -0.0000001 1.5707963
- joint left_inner_knuckle_joint: axis 1 0 0 -> 0. 0. 1.; limit lower=-1.0 upper=1.0 effort=1000 velocity=1.0 -> lower=-3.1415927 upper=3.1415927 effort=0. velocity=174.5329252; origin xyz=0 -0.0127 0.06142 rpy=0 0 3.141592653589793 -> xyz=0.0179 -0.00651 0. rpy=3.1415927 0. 0.; parent robotiq_arg2f_base_link -> left_inner_finger
- joint left_outer_finger_joint: axis 1 0 0 -> (none); origin xyz=0 0.0315 -0.0041 rpy=0 0 0 -> xyz=-0.0306 -0.05466 -0. rpy=-1.5707965 1.5707963 0.
- joint left_outer_knuckle_joint: axis 1 0 0 -> 0. 0. 1.; limit lower=-1.0 upper=1.0 effort=1000 velocity=1.0 -> lower=0. upper=0.8203047 effort=26. velocity=2.5562093; origin xyz=0 -0.0306011 0.054904 rpy=0 0 3.141592653589793 -> xyz=0. -0.0306 0.05466 rpy=1.5707964 0. -1.5707964
- joint right_inner_finger_joint: axis 1 0 0 -> 0. 0. 1.; limit lower=-1.0 upper=1.0 effort=1000 velocity=1.0 -> lower=-3.1415927 upper=3.1415927 effort=0. velocity=174.5329252; origin xyz=0 0.0061 0.0471 rpy=0 0 0 -> xyz=-0. 0.06776 0.09809 rpy=1.5707964 0.0000001 -1.5707964
- joint right_inner_knuckle_joint: axis 1 0 0 -> 0. 0. 1.; limit lower=-1.0 upper=1.0 effort=1000 velocity=1.0 -> lower=-3.1415927 upper=3.1415927 effort=0. velocity=174.5329252; origin xyz=0 0.0127 0.06142 rpy=0 0 0.0 -> xyz=0.0179 0.00651 0. rpy=0. 0. 0.; parent robotiq_arg2f_base_link -> right_inner_finger
- joint right_outer_finger_joint: axis 1 0 0 -> (none); origin xyz=0 0.0315 -0.0041 rpy=0 0 0 -> xyz=0.0306 0.05466 0. rpy=1.5707963 -1.5707963 0.
- joint right_outer_knuckle_joint: axis 1 0 0 -> 0. 0. 1.; limit lower=-1.0 upper=1.0 effort=1000 velocity=1.0 -> lower=0. upper=0.8203047 effort=0. velocity=174.5329252; origin xyz=0 0.0306011 0.054904 rpy=0 0 0 -> xyz=0. 0.0306 0.05466 rpy=-1.5707964 0. -1.5707964

Commit message: simplify the gripper in isaac sim to avoid the  simulation to explode

File: src/tidybot_description/urdf/tidybot_isaac.urdf (robot description, URDF)
Before this commit: robot tidybot, 28 links, 27 joints
Links:
- link left_inner_knuckle: geometry visual mesh filename=file:///tidybot_description/meshes/grippers/robotiq_2f_85/r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
- link right_inner_knuckle: geometry visual mesh filename=file:///tidybot_description/meshes/grippers/robotiq_2f_85/r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

Commit message: update gripper params

File: src/tidybot_description/urdf/tidybot_isaac.urdf (robot description, URDF)
Before this commit: robot tidybot, 28 links, 27 joints
Joints:
- joint left_outer_finger_joint: limit lower=0 upper=3.14 effort=100 velocity=100 -> lower=-1.57 upper=0 effort=100 velocity=100
- joint right_outer_finger_joint: limit lower=0.0 upper=3.14 effort=100 velocity=100 -> lower=-1.57 upper=0 effort=100 velocity=100
- joint right_outer_knuckle_joint: limit lower=-3.14 upper=3.14 effort=0. velocity=174.5329252 -> lower=0 upper=0.8203047 effort=26. velocity=2.5562093

Commit message: unified isaac containers

File: src/tidybot_description/urdf/tidybot_isaac.urdf (robot description, URDF)
Before this commit: robot tidybot, 28 links, 27 joints
Links:
- link arm_base_link: geometry collision mesh filename=package://tidybot_description/meshes/arms/gen3_7dof/base_li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; visual mesh filename=package://tidybot_description/meshes/arms/gen3_7dof/base_li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
- link base: geometry collision mesh filename=package://tidybot_description/meshes/base/tidybot++/Kinova.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; visual mesh filename=package://tidybot_description/meshes/base/tidybot++/Kinova.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
- link bracelet_link: geometry collision mesh filename=package://tidybot_description/meshes/arms/gen3_7dof/bracele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; visual mesh filename=package://tidybot_description/meshes/arms/gen3_7dof/bracele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
- link forearm_link: geometry collision mesh filename=package://tidybot_description/meshes/arms/gen3_7dof/forearm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; visual mesh filename=package://tidybot_description/meshes/arms/gen3_7dof/forearm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
- link half_arm_1_link: geometry collision mesh filename=package://tidybot_description/meshes/arms/gen3_7dof/half_ar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; visual mesh filename=package://tidybot_description/meshes/arms/gen3_7dof/half_ar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
- link half_arm_2_link: geometry collision mesh filename=package://tidybot_description/meshes/arms/gen3_7dof/half_ar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; visual mesh filename=package://tidybot_description/meshes/arms/gen3_7dof/half_ar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
- link left_inner_finger: geometry collision mesh filename=package://tidybot_description/meshes/grippers/robotiq_2f_85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; collision mesh filename=package://tidybot_description/meshes/grippers/robotiq_2f_85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
- link left_inner_knuckle: geometry visual mesh filename=package://tidybot_description/meshes/grippers/robotiq_2f_85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
- link left_outer_finger: geometry collision mesh filename=package://tidybot_description/meshes/grippers/robotiq_2f_85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; visual mesh filename=package://tidybot_description/meshes/grippers/robotiq_2f_85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
- link left_outer_knuckle: geometry collision mesh filename=package://tidybot_description/meshes/grippers/robotiq_2f_85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; visual mesh filename=package://tidybot_description/meshes/grippers/robotiq_2f_85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
- link right_inner_finger: geometry collision mesh filename=package://tidybot_description/meshes/grippers/robotiq_2f_85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; collision mesh filename=package://tidybot_description/meshes/grippers/robotiq_2f_85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
- link right_inner_knuckle: geometry visual mesh filename=package://tidybot_description/meshes/grippers/robotiq_2f_85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
- link right_outer_finger: geometry collision mesh filename=package://tidybot_description/meshes/grippers/robotiq_2f_85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; visual mesh filename=package://tidybot_description/meshes/grippers/robotiq_2f_85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
- link right_outer_knuckle: geometry collision mesh filename=package://tidybot_description/meshes/grippers/robotiq_2f_85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; visual mesh filename=package://tidybot_description/meshes/grippers/robotiq_2f_85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
- link robotiq_arg2f_base_link: geometry collision mesh filename=package://tidybot_description/meshes/grippers/robotiq_2f_85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; visual mesh filename=package://tidybot_description/meshes/grippers/robotiq_2f_85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
- link shoulder_link: geometry collision mesh filename=package://tidybot_description/meshes/arms/gen3_7dof/shoulde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; visual mesh filename=package://tidybot_description/meshes/arms/gen3_7dof/shoulde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
- link spherical_wrist_1_link: geometry collision mesh filename=package://tidybot_description/meshes/arms/gen3_7dof/spheric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; visual mesh filename=package://tidybot_description/meshes/arms/gen3_7dof/spheric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
- link spherical_wrist_2_link: geometry collision mesh filename=package://tidybot_description/meshes/arms/gen3_7dof/spheric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; visual mesh filename=package://tidybot_description/meshes/arms/gen3_7dof/spheric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

Commit message: Revert "added hande gripper for tidybot"
This reverts commit 627f805dde5cb1cd2c25c4a8a8fb5f9aa94f07f5.

File: src/tidybot_description/urdf/tidybot_isaac.urdf (robot description, URDF)
Before this commit: robot tidybot, 28 links, 27 joints
Joints:
- joint joint_x: origin xyz=0.0 0.0 0.005 rpy=0.0 0.0 0.0 -> xyz=0.0 0.0 0.085 rpy=0.0 0.0 0.0
