Commit message: add tidybot_base_controller

File: src/tidybot_description/urdf/base/base.xacro (robot description, xacro)
@@ -155,5 +155,5 @@
             <child link="joint_x_jointbody"/>
             <axis xyz="1 0 0" />
-            <limit lower="-2.0" upper="2.0" effort="100" velocity="1" />
+            <limit lower="-10.0" upper="10.0" effort="100" velocity="1" />
         </joint>
         <transmission name="joint_x_trans">
@@ -176,5 +176,5 @@
             <child link="joint_y_jointbody"/>
             <axis xyz="0 1 0" />
-            <limit lower="-2.0" upper="2.0" effort="100" velocity="1" />
+            <limit lower="-10.0" upper="10.0" effort="100" velocity="1" />
         </joint>
         <transmission name="joint_y_trans">

File: src/tidybot_description/urdf/tidybot.xacro (robot description, xacro)
@@ -9,79 +9,37 @@
     <!-- load the robot -->
     <xacro:load_bot arm="$(arg arm)" gripper="$(arg gripper)" vision="$(arg vision)" prefix="$(arg prefix)" />
+    <!-- configure ros2_control joints -->
+    <xacro:macro name="add_joint" params="name gain">
+        <joint name="${name}">
+            <command_interface name="position"/>
+            <state_interface name="position"/>
+            <state_interface name="velocity"/>
+            <param name="position_proportional_gain">${gain}</param>
+        </joint>
+    </xacro:macro>
     <ros2_control name="GazeboSystem" type="system">
     <hardware>
-        <plugin>gz_ros2_control/GazeboSimSystem</plugin>
+        <plugin>mock_components/GenericSystem</plugin>
     </hardware>
-    <joint name="joint_x">
-        <command_interface name="position"/>
-        <state_interface name="position"/>
-        <state_interface name="velocity"/>
-    </joint>
-    <joint name="joint_y">
-        <command_interface name="position"/>
-        <state_interface name="position"/>
-        <state_interface name="velocity"/>
-    </joint>
-    <joint name="joint_th">
-        <command_interface name="position"/>
-        <state_interface name="position"/>
-        <state_interface name="velocity"/>
-    </joint>
-    <joint name="joint_1">
-        <command_interface name="position"/>
-        <state_interface name="position"/>
-        <state_interface name="velocity"/>
-    </joint>
-    <joint name="joint_2">
-        <command_interface name="position"/>
-        <state_interface name="position"/>
-        <state_interface name="velocity"/>
-    </joint>
-    <joint name="joint_3">
-        <command_interface name="position"/>
-        <state_interface name="position"/>
-        <state_interface name="velocity"/>
-    </joint>
-    <joint name="joint_4">
-        <command_interface name="position"/>
-        <state_interface name="position"/>
-        <state_interface name="velocity"/>
-    </joint>
-    <joint name="joint_5">
-        <command_interface name="position"/>
-        <state_interface name="position"/>
-        <state_interface name="velocity"/>
-    </joint>
-    <joint name="joint_6">
-        <command_interface name="position"/>
-        <state_interface name="position"/>
-        <state_interface name="velocity"/>
-    </joint>
-    <joint name="right_finger_bottom_joint">
-        <command_interface name="position"/>
-        <state_interface name="position"/>
-        <state_interface name="velocity"/>
-    </joint>
-    <joint name="right_finger_tip_joint">
-        <command_interface name="position"/>
-        <state_interface name="position"/>
-        <state_interface name="velocity"/>
-    </joint>
-    <joint name="left_finger_bottom_joint">
-        <command_interface name="position"/>
-        <state_interface name="position"/>
-        <state_interface name="velocity"/>
-    </joint>
-    <joint name="left_finger_tip_joint">
-        <command_interface name="position"/>
-        <state_interface name="position"/>
-        <state_interface name="velocity"/>
-    </joint>
+    <xacro:add_joint name="joint_x" gain="0.1"/>
+    <xacro:add_joint name="joint_y" gain="0.1"/>
+    <xacro:add_joint name="joint_th" gain="0.1"/>
+    <xacro:add_joint name="joint_1" gain="0.1"/>
+    <xacro:add_joint name="joint_2" gain="0.1"/>
+    <xacro:add_joint name="joint_3" gain="0.1"/>
+    <xacro:add_joint name="joint_4" gain="0.1"/>
+    <xacro:add_joint name="joint_5" gain="0.1"/>
+    <xacro:add_joint name="joint_6" gain="0.1"/>
+    <xacro:add_joint name="right_finger_bottom_joint" gain="0.1"/>
+    <xacro:add_joint name="right_finger_tip_joint" gain="0.1"/>
+    <xacro:add_joint name="left_finger_bottom_joint" gain="0.1"/>
+    <xacro:add_joint name="left_finger_tip_joint" gain="0.1"/>
     </ros2_control>
     <gazebo>
         <plugin name="gz_ros2_control::GazeboSimROS2ControlPlugin" filename="gz_ros2_control-system">
-        <parameters>$(find tidybot_description)/urdf/ros2_control.yaml</parameters>
-        <robot_description_param>robot_description</robot_description_param>
+            <parameters>$(find tidybot_description)/urdf/ros2_control.yaml</parameters>
+            <robot_description_param>robot_description</robot_description_param>
         </plugin>
+        <self_collide>true</self_collide>
     </gazebo>
 </robot>

File: src/tidybot_moveit_config/config/tidybot.ros2_control.xacro (robot description, xacro)
@@ -3,58 +3,28 @@
     <xacro:macro name="tidybot_ros2_control" params="name initial_positions_file">
         <xacro:property name="initial_positions" value="${xacro.load_yaml(initial_positions_file)['initial_positions']}"/>
-        <ros2_control name="${name}" type="system">
-            <hardware>
-                <!-- By default, set up controllers for simulation. This won't work on real hardware -->
-                <plugin>mock_components/GenericSystem</plugin>
-            </hardware>
-            <joint name="joint_1">
+        <xacro:macro name="add_joint" params="name gain">
+            <joint name="${name}">
                 <command_interface name="position"/>
                 <state_interface name="position">
-                  <param name="initial_value">${initial_positions['joint_1']}</param>
+                  <param name="initial_value">${initial_positions[name]}</param>
                 </state_interface>
                 <state_interface name="velocity"/>
+                <param name="position_proportional_gain">${gain}</param>
             </joint>
-            <joint name="joint_2">
-                <command_interface name="position"/>
-                <state_interface name="position">
-                  <param name="initial_value">${initial_positions['joint_2']}</param>
-                </state_interface>
-                <state_interface name="velocity"/>
-            </joint>
-            <joint name="joint_3">
-                <command_interface name="position"/>
-                <state_interface name="position">
-                  <param name="initial_value">${initial_positions['joint_3']}</param>
-                </state_interface>
-                <state_interface name="velocity"/>
-            </joint>
-            <joint name="joint_4">
-                <command_interface name="position"/>
-                <state_interface name="position">
-                  <param name="initial_value">${initial_positions['joint_4']}</param>
-                </state_interface>
-                <state_interface name="velocity"/>
-            </joint>
-            <joint name="joint_5">
-                <command_interface name="position"/>
-                <state_interface name="position">
-                  <param name="initial_value">${initial_positions['joint_5']}</param>
-                </state_interface>
-                <state_interface name="velocity"/>
-            </joint>
-            <joint name="joint_6">
-                <command_interface name="position"/>
-                <state_interface name="position">
-                  <param name="initial_value">${initial_positions['joint_6']}</param>
-                </state_interface>
-                <state_interface name="velocity"/>
-            </joint>
-            <joint name="right_finger_bottom_joint">
-                <command_interface name="position"/>
-                <state_interface name="position">
-                  <param name="initial_value">${initial_positions['right_finger_bottom_joint']}</param>
-                </state_interface>
-                <state_interface name="velocity"/>
-            </joint>
+        </xacro:macro>
+        <ros2_control name="${name}" type="system">
+        <hardware>
+            <plugin>mock_components/GenericSystem</plugin>
+        </hardware>
+        <xacro:add_joint name="joint_x" gain="0.1"/>
+        <xacro:add_joint name="joint_y" gain="0.1"/>
+        <xacro:add_joint name="joint_th" gain="0.1"/>
+        <xacro:add_joint name="joint_1" gain="0.1"/>
+        <xacro:add_joint name="joint_2" gain="0.1"/>
+        <xacro:add_joint name="joint_3" gain="0.1"/>
+        <xacro:add_joint name="joint_4" gain="0.1"/>
+        <xacro:add_joint name="joint_5" gain="0.1"/>
+        <xacro:add_joint name="joint_6" gain="0.1"/>
+        <xacro:add_joint name="right_finger_bottom_joint" gain="0.1"/>
         </ros2_control>
     </xacro:macro>

Commit message: update the tf calculation in webxr base control

File: src/tidybot_description/urdf/base/base.xacro (robot description, xacro)
@@ -132,5 +132,5 @@
             <child link="joint_th_jointbody"/>
             <axis xyz="0.0 0.0 1.0"/>
-            <limit lower="-3.14" upper="3.14" effort="100" velocity="1"/>
+            <limit lower="-10" upper="10" effort="100" velocity="1"/>
             <dynamics damping="1.0" friction="1.0"/>
         </joint>
