Commit message: update web_server.launch.py and base xacro files

File: src/tidybot_description/urdf/base/base_macro.xacro (robot description, xacro)
@@ -91,11 +91,4 @@
             <dynamics damping="1.0" friction="1.0"/>
         </joint>
-        <transmission name="joint_x_trans">
-            <type>transmission_interface/SimpleTransmission</type>
-            <joint name="${prefix}joint_x" />
-            <actuator name="joint_x_motor">
-                <mechanicalReduction>1</mechanicalReduction>
-            </actuator>
-        </transmission>
         <link name="joint_y_jointbody">
             <inertial>
@@ -113,11 +106,4 @@
             <dynamics damping="1.0" friction="1.0"/>
         </joint>
-        <transmission name="joint_y_trans">
-            <type>transmission_interface/SimpleTransmission</type>
-            <joint name="${prefix}joint_y" />
-            <actuator name="joint_y_motor">
-                <mechanicalReduction>1</mechanicalReduction>
-            </actuator>
-        </transmission>
         <link name="joint_th_jointbody">
             <inertial>
@@ -135,11 +121,4 @@
             <dynamics damping="1.0" friction="1.0"/>
         </joint>
-        <transmission name="joint_th_trans">
-            <type>transmission_interface/SimpleTransmission</type>
-            <joint name="${prefix}joint_th" />
-            <actuator name="joint_th_motor">
-                <mechanicalReduction>1</mechanicalReduction>
-            </actuator>
-        </transmission>
         <joint type="fixed" name="joint_th_offset">
             <origin xyz="-0.0 -0.0 -0.0" rpy="0.0 0.0 0.0"/>

File: src/tidybot_description/urdf/bot.xacro (robot description, xacro)
@@ -5,5 +5,5 @@
     <xacro:include filename="$(find tidybot_description)/urdf/arms/${arm}/${arm}_macro.xacro" />
     <xacro:include filename="$(find tidybot_description)/urdf/grippers/${gripper}/${gripper}_macro.xacro" />
-    <xacro:include filename="$(find tidybot_description)/urdf/base/base.xacro" />
+    <xacro:include filename="$(find tidybot_description)/urdf/base/base_macro.xacro" />
     <!-- load the base -->
     <xacro:load_base parent="" prefix="${prefix}" />

File: src/tidybot_description/urdf/tidybot.gazebo.xacro (robot description, xacro)
@@ -20,4 +20,6 @@
   <xacro:include filename="$(find tidybot_description)/urdf/arms/${arm}/${arm}_transmission.xacro" />
   <xacro:load_arm_transmission prefix="${prefix}" />
+  <xacro:include filename="$(find tidybot_description)/urdf/base/base_transmission.xacro" />
+  <xacro:load_base_transmission prefix="${prefix}" />
 </xacro:macro>
 </robot>
