Commit message: add ros2_control to gazebo (#1)

File: src/tidybot_description/urdf/grippers/gen3_lite_2f/gen3_lite_2f_macro.xacro (robot description, xacro)
@@ -112,5 +112,5 @@
       <axis xyz="0 0 1" />
       <limit lower="-0.50" upper="0.21" effort="1000.0" velocity="1000.0" /> <!--limit lower="-1.03" upper="0.21" effort="1000" velocity="1000" /-->
-      <mimic joint="${prefix}right_finger_bottom_joint" multiplier="-0.676" offset="0.149" />
+      <!-- <mimic joint="${prefix}right_finger_bottom_joint" multiplier="-0.676" offset="0.149" /> -->
     </joint>
     <transmission name="${prefix}right_finger_tip_joint_trans">
@@ -152,5 +152,5 @@
       <axis xyz="0 0 1" />
       <limit lower="-0.96" upper="0.09" effort="1000.0" velocity="1000.0" />
-      <mimic joint="${prefix}right_finger_bottom_joint" multiplier="-1.0" offset="0.0" />
+      <!-- <mimic joint="${prefix}right_finger_bottom_joint" multiplier="-1.0" offset="0.0" /> -->
     </joint>
     <transmission name="${prefix}left_finger_bottom_joint_trans">
@@ -192,5 +192,5 @@
       <axis xyz="0 0 -1" />
       <limit lower="-0.50" upper="0.21" effort="1000.0" velocity="1000.0" /> <!--limit lower="-1.03" upper="0.21" effort="1000" velocity="1000" /-->
-      <mimic joint="${prefix}right_finger_bottom_joint" multiplier="-0.676" offset="0.149" />
+      <!-- <mimic joint="${prefix}right_finger_bottom_joint" multiplier="-0.676" offset="0.149" /> -->
     </joint>
     <transmission name="${prefix}left_finger_tip_joint_trans">

File: src/tidybot_description/urdf/tidybot.xacro (robot description, xacro)
@@ -5,6 +5,83 @@
     <xacro:arg name="vision" default="false" />
     <xacro:arg name="prefix" default="" />
+    <xacro:arg name="ros2_control_config_path" default="UNSET"/>
     <xacro:include filename="$(find tidybot_description)/urdf/bot.xacro" />
     <!-- load the robot -->
     <xacro:load_bot arm="$(arg arm)" gripper="$(arg gripper)" vision="$(arg vision)" prefix="$(arg prefix)" />
+    <ros2_control name="GazeboSystem" type="system">
+    <hardware>
+        <plugin>gz_ros2_control/GazeboSimSystem</plugin>
+    </hardware>
+    <joint name="joint_x">
+        <command_interface name="position"/>
+        <state_interface name="position"/>
+        <state_interface name="velocity"/>
+    </joint>
+    <joint name="joint_y">
+        <command_interface name="position"/>
+        <state_interface name="position"/>
+        <state_interface name="velocity"/>
+    </joint>
+    <joint name="joint_th">
+        <command_interface name="position"/>
+        <state_interface name="position"/>
+        <state_interface name="velocity"/>
+    </joint>
+    <joint name="joint_1">
+        <command_interface name="position"/>
+        <state_interface name="position"/>
+        <state_interface name="velocity"/>
+    </joint>
+    <joint name="joint_2">
+        <command_interface name="position"/>
+        <state_interface name="position"/>
+        <state_interface name="velocity"/>
+    </joint>
+    <joint name="joint_3">
+        <command_interface name="position"/>
+        <state_interface name="position"/>
+        <state_interface name="velocity"/>
+    </joint>
+    <joint name="joint_4">
+        <command_interface name="position"/>
+        <state_interface name="position"/>
+        <state_interface name="velocity"/>
+    </joint>
+    <joint name="joint_5">
+        <command_interface name="position"/>
+        <state_interface name="position"/>
+        <state_interface name="velocity"/>
+    </joint>
+    <joint name="joint_6">
+        <command_interface name="position"/>
+        <state_interface name="position"/>
+        <state_interface name="velocity"/>
+    </joint>
+    <joint name="right_finger_bottom_joint">
+        <command_interface name="position"/>
+        <state_interface name="position"/>
+        <state_interface name="velocity"/>
+    </joint>
+    <joint name="right_finger_tip_joint">
+        <command_interface name="position"/>
+        <state_interface name="position"/>
+        <state_interface name="velocity"/>
+    </joint>
+    <joint name="left_finger_bottom_joint">
+        <command_interface name="position"/>
+        <state_interface name="position"/>
+        <state_interface name="velocity"/>
+    </joint>
+    <joint name="left_finger_tip_joint">
+        <command_interface name="position"/>
+        <state_interface name="position"/>
+        <state_interface name="velocity"/>
+    </joint>
+    </ros2_control>
+    <gazebo>
+        <plugin name="gz_ros2_control::GazeboSimROS2ControlPlugin" filename="gz_ros2_control-system">
+        <parameters>$(find tidybot_description)/urdf/ros2_control.yaml</parameters>
+        <robot_description_param>robot_description</robot_description_param>
+        </plugin>
+    </gazebo>
 </robot>

Commit message: add webxr gripper control

File: src/tidybot_description/urdf/grippers/gen3_lite_2f/gen3_lite_2f_macro.xacro (robot description, xacro)
@@ -73,5 +73,5 @@
       <child link="${prefix}right_finger_prox_link" />
       <axis xyz="0 0 1" />
-      <limit lower="-0.09" upper="0.96" effort="1000" velocity="0.6" />
+      <limit lower="-0.09" upper="0.96" effort="1000" velocity="1000" />
       <dynamics damping="1.0" friction="1.0"/>
     </joint>

File: src/tidybot_description/urdf/tidybot.urdf (robot description, URDF)
Before this commit: robot mogi_bot, 6 links, 5 joints
Links:
- removed link base_footprint
- removed link base_link
- removed link front_left_wheel
- removed link front_right_wheel
- removed link rear_left_wheel
- removed link rear_right_wheel
- added link arm_base_link, mass 1.14608471; collision mesh filename=file:///home/yuandi/yuandi/tidybot_platform/install/tidybot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; visual mesh filename=file:///home/yuandi/yuandi/tidybot_platform/install/tidybot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
- added link arm_link, mass 1.17756164; collision mesh filename=file:///home/yuandi/yuandi/tidybot_platform/install/tidybot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; visual mesh filename=file:///home/yuandi/yuandi/tidybot_platform/install/tidybot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
- added link base, mass 60.0; collision mesh filename=file:///home/yuandi/yuandi/tidybot_platform/install/tidybot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; collision mesh filename=file:///home/yuandi/yuandi/tidybot_platform/install/tidybot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
- added link end_effector_link
- added link forearm_link, mass 0.59767669; collision mesh filename=file:///home/yuandi/yuandi/tidybot_platform/install/tidybot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; visual mesh filename=file:///home/yuandi/yuandi/tidybot_platform/install/tidybot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
- added link gripper_base_link, mass 0.1395; visual mesh filename=file:///home/yuandi/yuandi/tidybot_platform/install/tidybot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
- added link joint_th_jointbody, mass 0.001
- added link joint_x_jointbody, mass 0.001
- added link joint_y_jointbody, mass 0.001
- added link left_finger_dist_link, mass 0.010748; visual mesh filename=file:///home/yuandi/yuandi/tidybot_platform/install/tidybot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
- added link left_finger_prox_link, mass 0.018385; visual mesh filename=file:///home/yuandi/yuandi/tidybot_platform/install/tidybot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
- added link lower_wrist_link, mass 0.52693412; collision mesh filename=file:///home/yuandi/yuandi/tidybot_platform/install/tidybot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; visual mesh filename=file:///home/yuandi/yuandi/tidybot_platform/install/tidybot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
- added link right_finger_dist_link, mass 0.010748; visual mesh filename=file:///home/yuandi/yuandi/tidybot_platform/install/tidybot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
- added link right_finger_prox_link, mass 0.018385; visual mesh filename=file:///home/yuandi/yuandi/tidybot_platform/install/tidybot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
- added link shoulder_link, mass 0.95974404; collision mesh filename=file:///home/yuandi/yuandi/tidybot_platform/install/tidybot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; visual mesh filename=file:///home/yuandi/yuandi/tidybot_platform/install/tidybot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
- added link tool_frame
- added link upper_wrist_link, mass 0.58097325; collision mesh filename=file:///home/yuandi/yuandi/tidybot_platform/install/tidybot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; visual mesh filename=file:///home/yuandi/yuandi/tidybot_platform/install/tidybot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
- added link world
Joints:
- removed joint base_footprint_joint
- removed joint front_left_wheel_joint
- removed joint front_right_wheel_joint
- removed joint rear_left_wheel_joint
- removed joint rear_right_wheel_joint
- added joint arm_base_joint: type fixed, parent base, child arm_base_link, origin xyz=0 0 0.33 rpy=0 0 0
- added joint gripper_base_joint: type fixed, parent end_effector_link, child gripper_base_link, origin xyz=0 0 0 rpy=0 0 0, axis 0 0 0
- added joint joint_1: type revolute, parent arm_base_link, child shoulder_link, origin xyz=0 0 0.12825 rpy=0 0 0, axis 0 0 1, limit lower=-2.69 upper=2.69 effort=10 velocity=1.6
- added joint joint_2: type revolute, parent shoulder_link, child arm_link, origin xyz=0 -0.03 0.115 rpy=1.5708 0 0, axis 0 0 1, limit lower=-2.69 upper=2.69 effort=14 velocity=1.6
- added joint joint_3: type revolute, parent arm_link, child forearm_link, origin xyz=0 0.28 0 rpy=-3.1416 0 0, axis 0 0 1, limit lower=-2.69 upper=2.69 effort=10 velocity=1.6
- added joint joint_4: type revolute, parent forearm_link, child lower_wrist_link, origin xyz=0 -0.14 0.02 rpy=1.5708 0 0, axis 0 0 1, limit lower=-2.59 upper=2.59 effort=7 velocity=1.6
- added joint joint_5: type revolute, parent lower_wrist_link, child upper_wrist_link, origin xyz=0.0285 0 0.105 rpy=0 1.5708 0, axis 0 0 1, limit lower=-2.57 upper=2.57 effort=7 velocity=1.6
- added joint joint_6: type revolute, parent upper_wrist_link, child end_effector_link, origin xyz=-0.105 0 0.0285 rpy=0 -1.5708 0, axis 0 0 1, limit lower=-2.59 upper=2.59 effort=7 velocity=3.2
- added joint joint_th: type revolute, parent joint_y_jointbody, child joint_th_jointbody, origin xyz=0.0 0.0 0.0 rpy=0.0 0.0 0.0, axis 0.0 0.0 1.0, limit lower=-10 upper=10 effort=100 velocity=1
- added joint joint_th_offset: type fixed, parent joint_th_jointbody, child base, origin xyz=-0.0 -0.0 -0.0 rpy=0.0 0.0 0.0, axis 0.0 0.0 1.0, limit lower=0.0 upper=0.0 effort=100 velocity=100
- added joint joint_x: type prismatic, parent world, child joint_x_jointbody, origin xyz=0.0 0.0 0.0 rpy=0.0 0.0 0.0, axis 1 0 0, limit lower=-10.0 upper=10.0 effort=100 velocity=1
- added joint joint_y: type prismatic, parent joint_x_jointbody, child joint_y_jointbody, origin xyz=0.0 0.0 0.0 rpy=0.0 0.0 0.0, axis 0 1 0, limit lower=-10.0 upper=10.0 effort=100 velocity=1
- added joint left_finger_bottom_joint: type revolute, parent gripper_base_link, child left_finger_prox_link, origin xyz=0 0.0305 0.070003 rpy=0 1.5708 0, axis 0 0 1, limit lower=-0.96 upper=0.09 effort=1000.0 velocity=1000.0
- added joint left_finger_tip_joint: type revolute, parent left_finger_prox_link, child left_finger_dist_link, origin xyz=-0.045636 -0.020423 6.9901E-05 rpy=0 0 0, axis 0 0 -1, limit lower=-0.50 upper=0.21 effort=1000.0 velocity=1000.0
- added joint right_finger_bottom_joint: type revolute, parent gripper_base_link, child right_finger_prox_link, origin xyz=0 -0.030501 0.070003 rpy=0 1.5708 0, axis 0 0 1, limit lower=-0.09 upper=0.96 effort=1000 velocity=1000
- added joint right_finger_tip_joint: type revolute, parent right_finger_prox_link, child right_finger_dist_link, origin xyz=-0.045636 0.020423 0 rpy=0 0 0, axis 0 0 1, limit lower=-0.50 upper=0.21 effort=1000.0 velocity=1000.0
- added joint tool_frame_joint: type fixed, parent end_effector_link, child tool_frame, origin xyz=0 0 0.130 rpy=0 0 1.57079632679, axis 0 0 0
