Commit message: Add base joints and transmissions

File: src/tidybot_description/urdf/arms/gen3_lite/gen3_lite_macro.xacro (robot description, xacro)
@@ -66,4 +66,11 @@
       <limit lower="-2.69" upper="2.69" effort="10" velocity="1.6" />
     </joint>
+    <transmission name="joint1_trans">
+      <type>transmission_interface/SimpleTransmission</type>
+      <joint name="${prefix}joint_1" />
+      <actuator name="joint1_motor">
+        <mechanicalReduction>1</mechanicalReduction>
+      </actuator>
+    </transmission>
     <link name="${prefix}arm_link">
       <inertial>
@@ -98,4 +105,11 @@
       <limit lower="-2.69" upper="2.69" effort="14" velocity="1.6" />
     </joint>
+    <transmission name="joint2_trans">
+      <type>transmission_interface/SimpleTransmission</type>
+      <joint name="${prefix}joint_2" />
+      <actuator name="joint2_motor">
+        <mechanicalReduction>1</mechanicalReduction>
+      </actuator>
+    </transmission>
     <link name="${prefix}forearm_link">
       <inertial>
@@ -130,4 +144,11 @@
       <limit lower="-2.69" upper="2.69" effort="10" velocity="1.6" />
     </joint>
+    <transmission name="joint3_trans">
+      <type>transmission_interface/SimpleTransmission</type>
+      <joint name="${prefix}joint_3" />
+      <actuator name="joint3_motor">
+        <mechanicalReduction>1</mechanicalReduction>
+      </actuator>
+    </transmission>
     <link name="${prefix}lower_wrist_link">
       <inertial>
@@ -162,4 +183,11 @@
       <limit lower="-2.59" upper="2.59" effort="7" velocity="1.6" />
     </joint>
+    <transmission name="joint4_trans">
+      <type>transmission_interface/SimpleTransmission</type>
+      <joint name="${prefix}joint_4" />
+      <actuator name="joint4_motor">
+        <mechanicalReduction>1</mechanicalReduction>
+      </actuator>
+    </transmission>
     <link name="${prefix}upper_wrist_link">
       <inertial>
@@ -194,4 +222,11 @@
       <limit lower="-2.57" upper="2.57" effort="7" velocity="1.6" />
     </joint>
+    <transmission name="joint5_trans">
+      <type>transmission_interface/SimpleTransmission</type>
+      <joint name="${prefix}joint_5" />
+      <actuator name="joint5_motor">
+        <mechanicalReduction>1</mechanicalReduction>
+      </actuator>
+    </transmission>
     <link name="${prefix}end_effector_link" />
     <joint name="${prefix}joint_6" type="revolute">
@@ -202,4 +237,11 @@
       <limit lower="-2.59" upper="2.59" effort="7" velocity="3.2" />
     </joint>
+    <transmission name="joint6_trans">
+      <type>transmission_interface/SimpleTransmission</type>
+      <joint name="${prefix}joint_6" />
+      <actuator name="joint6_motor">
+        <mechanicalReduction>1</mechanicalReduction>
+      </actuator>
+    </transmission>
   </xacro:macro>
 </robot>

File: src/tidybot_description/urdf/base/base.xacro (robot description, xacro)
@@ -150,9 +150,18 @@
             </inertial>
         </link>
-        <joint type="fixed" name="joint_x">
+        <joint type="prismatic" name="joint_x">
+            <origin xyz="0.0 0.0 0.0" rpy="0.0 0.0 0.0"/>
             <parent link="world"/>
             <child link="joint_x_jointbody"/>
-            <origin xyz="0.0 0.0 0.0" rpy="0.0 0.0 0.0"/>
-        </joint>
+            <axis xyz="1 0 0" />
+            <limit lower="-2.0" upper="2.0" effort="100" velocity="1" />
+        </joint>
+        <transmission name="joint_x_trans">
+            <type>transmission_interface/SimpleTransmission</type>
+            <joint name="${prefix}joint_x" />
+            <actuator name="joint_x_motor">
+                <mechanicalReduction>1</mechanicalReduction>
+            </actuator>
+        </transmission>
         <link name="joint_y_jointbody">
             <inertial>
@@ -162,9 +171,18 @@
             </inertial>
         </link>
-        <joint type="fixed" name="joint_y">
+        <joint type="prismatic" name="joint_y">
+            <origin xyz="0.0 0.0 0.0" rpy="0.0 0.0 0.0"/>
             <parent link="joint_x_jointbody"/>
             <child link="joint_y_jointbody"/>
-            <origin xyz="0.0 0.0 0.0" rpy="0.0 0.0 0.0"/>
-        </joint>
+            <axis xyz="0 1 0" />
+            <limit lower="-2.0" upper="2.0" effort="100" velocity="1" />
+        </joint>
+        <transmission name="joint_y_trans">
+            <type>transmission_interface/SimpleTransmission</type>
+            <joint name="${prefix}joint_y" />
+            <actuator name="joint_y_motor">
+                <mechanicalReduction>1</mechanicalReduction>
+            </actuator>
+        </transmission>
         <link name="joint_th_jointbody">
             <inertial>
@@ -175,14 +193,23 @@
         </link>
         <joint type="revolute" name="joint_th">
+            <origin xyz="0.0 0.0 0.0" rpy="0.0 0.0 0.0"/>
             <parent link="joint_y_jointbody"/>
             <child link="joint_th_jointbody"/>
-            <origin xyz="0.0 0.0 0.0" rpy="0.0 0.0 0.0"/>
+            <axis xyz="0.0 0.0 1.0"/>
+            <limit lower="-3.14" upper="3.14" effort="100" velocity="1"/>
+        </joint>
+        <transmission name="joint_th_trans">
+            <type>transmission_interface/SimpleTransmission</type>
+            <joint name="${prefix}joint_th" />
+            <actuator name="joint_th_motor">
+                <mechanicalReduction>1</mechanicalReduction>
+            </actuator>
+        </transmission>
+        <joint type="fixed" name="joint_th_offset">
+            <origin xyz="-0.0 -0.0 -0.0" rpy="0.0 0.0 0.0"/>
+            <parent link="joint_th_jointbody"/>
+            <child link="base_link"/>
             <axis xyz="0.0 0.0 1.0"/>
             <limit lower="0.0" upper="0.0" effort="100" velocity="100"/>
-        </joint>
-        <joint type="fixed" name="joint_th_offset">
-            <parent link="joint_th_jointbody"/>
-            <child link="base_link"/>
-            <origin xyz="-0.0 -0.0 -0.0" rpy="0.0 0.0 0.0"/>
         </joint>
         <material name="white">

File: src/tidybot_description/urdf/grippers/gen3_lite_2f/gen3_lite_2f_macro.xacro (robot description, xacro)
@@ -74,4 +74,11 @@
       <limit lower="-0.09" upper="0.96" effort="1000" velocity="0.6" />
     </joint>
+    <transmission name="${prefix}right_finger_bottom_joint_trans">
+      <type>transmission_interface/SimpleTransmission</type>
+      <joint name="${prefix}right_finger_bottom_joint" />
+      <actuator name="${prefix}right_finger_bottom_joint_motor">
+          <mechanicalReduction>1</mechanicalReduction>
+      </actuator>
+    </transmission>
     <link name="${prefix}right_finger_dist_link">
       <inertial>
@@ -107,4 +114,11 @@
       <mimic joint="${prefix}right_finger_bottom_joint" multiplier="-0.676" offset="0.149" />
     </joint>
+    <transmission name="${prefix}right_finger_tip_joint_trans">
+      <type>transmission_interface/SimpleTransmission</type>
+      <joint name="${prefix}right_finger_tip_joint" />
+      <actuator name="${prefix}right_finger_tip_joint_motor">
+          <mechanicalReduction>1</mechanicalReduction>
+      </actuator>
+    </transmission>
     <link name="${prefix}left_finger_prox_link">
       <inertial>
@@ -140,4 +154,11 @@
       <mimic joint="${prefix}right_finger_bottom_joint" multiplier="-1.0" offset="0.0" />
     </joint>
+    <transmission name="${prefix}left_finger_bottom_joint_trans">
+      <type>transmission_interface/SimpleTransmission</type>
+      <joint name="${prefix}left_finger_bottom_joint" />
+      <actuator name="${prefix}left_finger_bottom_joint_motor">
+          <mechanicalReduction>1</mechanicalReduction>
+      </actuator>
+    </transmission>
     <link name="${prefix}left_finger_dist_link">
       <inertial>
@@ -173,4 +194,11 @@
       <mimic joint="${prefix}right_finger_bottom_joint" multiplier="-0.676" offset="0.149" />
     </joint>
+    <transmission name="${prefix}left_finger_tip_joint_trans">
+      <type>transmission_interface/SimpleTransmission</type>
+      <joint name="${prefix}left_finger_tip_joint" />
+      <actuator name="${prefix}left_finger_tip_joint_motor">
+          <mechanicalReduction>1</mechanicalReduction>
+      </actuator>
+    </transmission>
   </xacro:macro>
 </robot>

File: src/tidybot_description/urdf/grippers/robotiq_2f_85/robotiq_arg2f_85_model_macro.xacro (robot description, xacro)
@@ -140,4 +140,11 @@
       <mimic joint="${prefix}finger_joint" multiplier="1" offset="0" />
     </joint>
+    <transmission name="{prefix}${fingerprefix}_inner_knuckle_joint_trans">
+      <type>transmission_interface/SimpleTransmission</type>
+      <joint name="${prefix}${fingerprefix}_inner_knuckle_joint" />
+      <actuator name="${prefix}${fingerprefix}_inner_knuckle_joint_motor">
+          <mechanicalReduction>1</mechanicalReduction>
+      </actuator>
+    </transmission>
   </xacro:macro>
   <xacro:macro name="inner_finger_joint" params="prefix fingerprefix">
@@ -150,4 +157,11 @@
       <mimic joint="${prefix}finger_joint" multiplier="-1" offset="0" />
     </joint>
+    <transmission name="${prefix}${fingerprefix}_inner_finger_joint_trans">
+      <type>transmission_interface/SimpleTransmission</type>
+      <joint name="${prefix}${fingerprefix}_inner_finger_joint" />
+      <actuator name="${prefix}${fingerprefix}_inner_finger_joint_motor">
+          <mechanicalReduction>1</mechanicalReduction>
+      </actuator>
+    </transmission>
   </xacro:macro>
   <xacro:macro name="inner_finger_pad_joint" params="prefix fingerprefix">
@@ -168,4 +182,11 @@
       <limit lower="0" upper="0.8" velocity="2.0" effort="1000" />
     </joint>
+    <transmission name="${prefix}finger_joint_trans">
+      <type>transmission_interface/SimpleTransmission</type>
+      <joint name="${prefix}finger_joint" />
+      <actuator name="${prefix}finger_joint_motor">
+          <mechanicalReduction>1</mechanicalReduction>
+      </actuator>
+    </transmission>
     <xacro:finger_joints prefix="${prefix}" fingerprefix="left" reflect="1.0"/>
   </xacro:macro>
@@ -179,4 +200,11 @@
       <mimic joint="${prefix}finger_joint" multiplier="1" offset="0" />
     </joint>
+    <transmission name="$${prefix}right_outer_knuckle_joint_trans">
+      <type>transmission_interface/SimpleTransmission</type>
+      <joint name="${prefix}right_outer_knuckle_joint" />
+      <actuator name="${prefix}right_outer_knuckle_joint_motor">
+          <mechanicalReduction>1</mechanicalReduction>
+      </actuator>
+    </transmission>
     <xacro:finger_joints prefix="${prefix}" fingerprefix="right" reflect="-1.0"/>
   </xacro:macro>

Commit message: add moveit joint_trajectory_controller

File: src/tidybot_description/urdf/arms/gen3_lite/gen3_lite_macro.xacro (robot description, xacro)
@@ -65,4 +65,5 @@
       <axis xyz="0 0 1" />
       <limit lower="-2.69" upper="2.69" effort="10" velocity="1.6" />
+      <dynamics damping="1.0" friction="1.0"/>
     </joint>
     <transmission name="joint1_trans">
@@ -104,4 +105,5 @@
       <axis xyz="0 0 1" />
       <limit lower="-2.69" upper="2.69" effort="14" velocity="1.6" />
+      <dynamics damping="1.0" friction="1.0"/>
     </joint>
     <transmission name="joint2_trans">
@@ -143,4 +145,5 @@
       <axis xyz="0 0 1" />
       <limit lower="-2.69" upper="2.69" effort="10" velocity="1.6" />
+      <dynamics damping="1.0" friction="1.0"/>
     </joint>
     <transmission name="joint3_trans">
@@ -182,4 +185,5 @@
       <axis xyz="0 0 1" />
       <limit lower="-2.59" upper="2.59" effort="7" velocity="1.6" />
+      <dynamics damping="1.0" friction="1.0"/>
     </joint>
     <transmission name="joint4_trans">
@@ -221,4 +225,5 @@
       <axis xyz="0 0 1" />
       <limit lower="-2.57" upper="2.57" effort="7" velocity="1.6" />
+      <dynamics damping="1.0" friction="1.0"/>
     </joint>
     <transmission name="joint5_trans">
@@ -236,4 +241,5 @@
       <axis xyz="0 0 1" />
       <limit lower="-2.59" upper="2.59" effort="7" velocity="3.2" />
+      <dynamics damping="1.0" friction="1.0"/>
     </joint>
     <transmission name="joint6_trans">

File: src/tidybot_description/urdf/base/base.xacro (robot description, xacro)
@@ -155,5 +155,6 @@
             <child link="joint_x_jointbody"/>
             <axis xyz="1 0 0" />
-            <limit lower="-10.0" upper="10.0" effort="100" velocity="1" />
+            <limit lower="-10.0" upper="10.0" effort="100" velocity="1"/>
+            <dynamics damping="1.0" friction="1.0"/>
         </joint>
         <transmission name="joint_x_trans">
@@ -176,5 +177,6 @@
             <child link="joint_y_jointbody"/>
             <axis xyz="0 1 0" />
-            <limit lower="-10.0" upper="10.0" effort="100" velocity="1" />
+            <limit lower="-10.0" upper="10.0" effort="100" velocity="1"/>
+            <dynamics damping="1.0" friction="1.0"/>
         </joint>
         <transmission name="joint_y_trans">
@@ -198,4 +200,5 @@
             <axis xyz="0.0 0.0 1.0"/>
             <limit lower="-3.14" upper="3.14" effort="100" velocity="1"/>
+            <dynamics damping="1.0" friction="1.0"/>
         </joint>
         <transmission name="joint_th_trans">

File: src/tidybot_description/urdf/grippers/gen3_lite_2f/gen3_lite_2f_macro.xacro (robot description, xacro)
@@ -73,4 +73,5 @@
       <axis xyz="0 0 1" />
       <limit lower="-0.09" upper="0.96" effort="1000" velocity="0.6" />
+      <dynamics damping="1.0" friction="1.0"/>
     </joint>
     <transmission name="${prefix}right_finger_bottom_joint_trans">
@@ -113,4 +114,5 @@
       <limit lower="-0.50" upper="0.21" effort="1000.0" velocity="1000.0" /> <!--limit lower="-1.03" upper="0.21" effort="1000" velocity="1000" /-->
       <!-- <mimic joint="${prefix}right_finger_bottom_joint" multiplier="-0.676" offset="0.149" /> -->
+      <dynamics damping="1.0" friction="1.0"/>
     </joint>
     <transmission name="${prefix}right_finger_tip_joint_trans">
@@ -153,4 +155,5 @@
       <limit lower="-0.96" upper="0.09" effort="1000.0" velocity="1000.0" />
       <!-- <mimic joint="${prefix}right_finger_bottom_joint" multiplier="-1.0" offset="0.0" /> -->
+      <dynamics damping="1.0" friction="1.0"/>
     </joint>
     <transmission name="${prefix}left_finger_bottom_joint_trans">
@@ -193,4 +196,5 @@
       <limit lower="-0.50" upper="0.21" effort="1000.0" velocity="1000.0" /> <!--limit lower="-1.03" upper="0.21" effort="1000" velocity="1000" /-->
       <!-- <mimic joint="${prefix}right_finger_bottom_joint" multiplier="-0.676" offset="0.149" /> -->
+      <dynamics damping="1.0" friction="1.0"/>
     </joint>
     <transmission name="${prefix}left_finger_tip_joint_trans">

File: src/tidybot_description/urdf/tidybot.xacro (robot description, xacro)
@@ -20,5 +20,5 @@
     <ros2_control name="GazeboSystem" type="system">
     <hardware>
-        <plugin>mock_components/GenericSystem</plugin>
+        <plugin>gz_ros2_control/GazeboSimSystem</plugin>
     </hardware>
     <xacro:add_joint name="joint_x" gain="0.1"/>
