Commit message: merge old repo

File: src/tidybot_description/urdf/arms/gen3_lite/gen3_lite_macro.xacro (robot description, xacro)
@@ -65,7 +65,4 @@
       <axis xyz="0 0 1" />
       <limit lower="-2.69" upper="2.69" effort="10" velocity="1.6" />
-<<<<<<< HEAD
-    </joint>
-=======
       <dynamics damping="1.0" friction="1.0"/>
     </joint>
@@ -77,5 +74,4 @@
       </actuator>
     </transmission>
->>>>>>> master
     <link name="${prefix}arm_link">
       <inertial>
@@ -109,7 +105,4 @@
       <axis xyz="0 0 1" />
       <limit lower="-2.69" upper="2.69" effort="14" velocity="1.6" />
-<<<<<<< HEAD
-    </joint>
-=======
       <dynamics damping="1.0" friction="1.0"/>
     </joint>
@@ -121,5 +114,4 @@
       </actuator>
     </transmission>
->>>>>>> master
     <link name="${prefix}forearm_link">
       <inertial>
@@ -153,7 +145,4 @@
       <axis xyz="0 0 1" />
       <limit lower="-2.69" upper="2.69" effort="10" velocity="1.6" />
-<<<<<<< HEAD
-    </joint>
-=======
       <dynamics damping="1.0" friction="1.0"/>
     </joint>
@@ -165,5 +154,4 @@
       </actuator>
     </transmission>
->>>>>>> master
     <link name="${prefix}lower_wrist_link">
       <inertial>
@@ -197,7 +185,4 @@
       <axis xyz="0 0 1" />
       <limit lower="-2.59" upper="2.59" effort="7" velocity="1.6" />
-<<<<<<< HEAD
-    </joint>
-=======
       <dynamics damping="1.0" friction="1.0"/>
     </joint>
@@ -209,5 +194,4 @@
       </actuator>
     </transmission>
->>>>>>> master
     <link name="${prefix}upper_wrist_link">
       <inertial>
@@ -241,7 +225,4 @@
       <axis xyz="0 0 1" />
       <limit lower="-2.57" upper="2.57" effort="7" velocity="1.6" />
-<<<<<<< HEAD
-    </joint>
-=======
       <dynamics damping="1.0" friction="1.0"/>
     </joint>
@@ -253,5 +234,4 @@
       </actuator>
     </transmission>
->>>>>>> master
     <link name="${prefix}end_effector_link" />
     <joint name="${prefix}joint_6" type="revolute">
@@ -261,7 +241,4 @@
       <axis xyz="0 0 1" />
       <limit lower="-2.59" upper="2.59" effort="7" velocity="3.2" />
-<<<<<<< HEAD
-    </joint>
-=======
       <dynamics damping="1.0" friction="1.0"/>
     </joint>
@@ -273,5 +250,4 @@
       </actuator>
     </transmission>
->>>>>>> master
   </xacro:macro>
 </robot>

File: src/tidybot_description/urdf/base/base.xacro (robot description, xacro)
@@ -150,11 +150,4 @@
             </inertial>
         </link>
-<<<<<<< HEAD
-        <joint type="fixed" name="joint_x">
-            <parent link="world"/>
-            <child link="joint_x_jointbody"/>
-            <origin xyz="0.0 0.0 0.0" rpy="0.0 0.0 0.0"/>
-        </joint>
-=======
         <joint type="prismatic" name="joint_x">
             <origin xyz="0.0 0.0 0.0" rpy="0.0 0.0 0.0"/>
@@ -172,5 +165,4 @@
             </actuator>
         </transmission>
->>>>>>> master
         <link name="joint_y_jointbody">
             <inertial>
@@ -180,11 +172,4 @@
             </inertial>
         </link>
-<<<<<<< HEAD
-        <joint type="fixed" name="joint_y">
-            <parent link="joint_x_jointbody"/>
-            <child link="joint_y_jointbody"/>
-            <origin xyz="0.0 0.0 0.0" rpy="0.0 0.0 0.0"/>
-        </joint>
-=======
         <joint type="prismatic" name="joint_y">
             <origin xyz="0.0 0.0 0.0" rpy="0.0 0.0 0.0"/>
@@ -202,5 +187,4 @@
             </actuator>
         </transmission>
->>>>>>> master
         <link name="joint_th_jointbody">
             <inertial>
@@ -211,16 +195,4 @@
         </link>
         <joint type="revolute" name="joint_th">
-<<<<<<< HEAD
-            <parent link="joint_y_jointbody"/>
-            <child link="joint_th_jointbody"/>
-            <origin xyz="0.0 0.0 0.0" rpy="0.0 0.0 0.0"/>
-            <axis xyz="0.0 0.0 1.0"/>
-            <limit lower="0.0" upper="0.0" effort="100" velocity="100"/>
-        </joint>
-        <joint type="fixed" name="joint_th_offset">
-            <parent link="joint_th_jointbody"/>
-            <child link="base_link"/>
-            <origin xyz="-0.0 -0.0 -0.0" rpy="0.0 0.0 0.0"/>
-=======
             <origin xyz="0.0 0.0 0.0" rpy="0.0 0.0 0.0"/>
             <parent link="joint_y_jointbody"/>
@@ -243,5 +215,4 @@
             <axis xyz="0.0 0.0 1.0"/>
             <limit lower="0.0" upper="0.0" effort="100" velocity="100"/>
->>>>>>> master
         </joint>
         <material name="white">
@@ -250,7 +221,3 @@
     </xacro:macro>
     <!-- <xacro:load_base prefix=""/> -->
-<<<<<<< HEAD
 </robot>
-=======
-</robot>
->>>>>>> master

File: src/tidybot_description/urdf/grippers/gen3_lite_2f/gen3_lite_2f_macro.xacro (robot description, xacro)
@@ -73,7 +73,4 @@
       <axis xyz="0 0 1" />
       <limit lower="-0.09" upper="0.96" effort="1000" velocity="0.6" />
-<<<<<<< HEAD
-    </joint>
-=======
       <dynamics damping="1.0" friction="1.0"/>
     </joint>
@@ -85,5 +82,4 @@
       </actuator>
     </transmission>
->>>>>>> master
     <link name="${prefix}right_finger_dist_link">
       <inertial>
@@ -117,8 +113,4 @@
       <axis xyz="0 0 1" />
       <limit lower="-0.50" upper="0.21" effort="1000.0" velocity="1000.0" /> <!--limit lower="-1.03" upper="0.21" effort="1000" velocity="1000" /-->
-<<<<<<< HEAD
-      <mimic joint="${prefix}right_finger_bottom_joint" multiplier="-0.676" offset="0.149" />
-    </joint>
-=======
       <!-- <mimic joint="${prefix}right_finger_bottom_joint" multiplier="-0.676" offset="0.149" /> -->
       <dynamics damping="1.0" friction="1.0"/>
@@ -131,5 +123,4 @@
       </actuator>
     </transmission>
->>>>>>> master
     <link name="${prefix}left_finger_prox_link">
       <inertial>
@@ -163,8 +154,4 @@
       <axis xyz="0 0 1" />
       <limit lower="-0.96" upper="0.09" effort="1000.0" velocity="1000.0" />
-<<<<<<< HEAD
-      <mimic joint="${prefix}right_finger_bottom_joint" multiplier="-1.0" offset="0.0" />
-    </joint>
-=======
       <!-- <mimic joint="${prefix}right_finger_bottom_joint" multiplier="-1.0" offset="0.0" /> -->
       <dynamics damping="1.0" friction="1.0"/>
@@ -177,5 +164,4 @@
       </actuator>
     </transmission>
->>>>>>> master
     <link name="${prefix}left_finger_dist_link">
       <inertial>
@@ -209,8 +195,4 @@
       <axis xyz="0 0 -1" />
       <limit lower="-0.50" upper="0.21" effort="1000.0" velocity="1000.0" /> <!--limit lower="-1.03" upper="0.21" effort="1000" velocity="1000" /-->
-<<<<<<< HEAD
-      <mimic joint="${prefix}right_finger_bottom_joint" multiplier="-0.676" offset="0.149" />
-    </joint>
-=======
       <!-- <mimic joint="${prefix}right_finger_bottom_joint" multiplier="-0.676" offset="0.149" /> -->
       <dynamics damping="1.0" friction="1.0"/>
@@ -223,5 +205,4 @@
       </actuator>
     </transmission>
->>>>>>> master
   </xacro:macro>
 </robot>

File: src/tidybot_description/urdf/grippers/robotiq_2f_85/robotiq_arg2f_85_model_macro.xacro (robot description, xacro)
@@ -140,6 +140,4 @@
       <mimic joint="${prefix}finger_joint" multiplier="1" offset="0" />
     </joint>
-<<<<<<< HEAD
-=======
     <transmission name="{prefix}${fingerprefix}_inner_knuckle_joint_trans">
       <type>transmission_interface/SimpleTransmission</type>
@@ -149,5 +147,4 @@
       </actuator>
     </transmission>
->>>>>>> master
   </xacro:macro>
   <xacro:macro name="inner_finger_joint" params="prefix fingerprefix">
@@ -160,6 +157,4 @@
       <mimic joint="${prefix}finger_joint" multiplier="-1" offset="0" />
     </joint>
-<<<<<<< HEAD
-=======
     <transmission name="${prefix}${fingerprefix}_inner_finger_joint_trans">
       <type>transmission_interface/SimpleTransmission</type>
@@ -169,5 +164,4 @@
       </actuator>
     </transmission>
->>>>>>> master
   </xacro:macro>
   <xacro:macro name="inner_finger_pad_joint" params="prefix fingerprefix">
@@ -188,6 +182,4 @@
       <limit lower="0" upper="0.8" velocity="2.0" effort="1000" />
     </joint>
-<<<<<<< HEAD
-=======
     <transmission name="${prefix}finger_joint_trans">
       <type>transmission_interface/SimpleTransmission</type>
@@ -197,5 +189,4 @@
       </actuator>
     </transmission>
->>>>>>> master
     <xacro:finger_joints prefix="${prefix}" fingerprefix="left" reflect="1.0"/>
   </xacro:macro>
@@ -209,6 +200,4 @@
       <mimic joint="${prefix}finger_joint" multiplier="1" offset="0" />
     </joint>
-<<<<<<< HEAD
-=======
     <transmission name="$${prefix}right_outer_knuckle_joint_trans">
       <type>transmission_interface/SimpleTransmission</type>
@@ -218,5 +207,4 @@
       </actuator>
     </transmission>
->>>>>>> master
     <xacro:finger_joints prefix="${prefix}" fingerprefix="right" reflect="-1.0"/>
   </xacro:macro>

File: src/tidybot_description/urdf/tidybot.xacro (robot description, xacro)
@@ -1,25 +1,15 @@
 <?xml version="1.0"?>
-<<<<<<< HEAD
-<robot name="tidybot" xmlns:xacro="http://ros.org/wiki/xacro">
-=======
 <robot name="tidybot" xmlns:xacro="http://ros.org/wiki/xacro">
     <xacro:arg name="hardware_plugin" default="mock_components/GenericSystem" />
->>>>>>> master
     <xacro:arg name="arm" default="gen3_lite" />
     <xacro:arg name="gripper" default="gen3_lite_2f" />
     <xacro:arg name="vision" default="false" />
     <xacro:arg name="prefix" default="" />
-<<<<<<< HEAD
-=======
     <xacro:arg name="ros2_control_config_path" default="$(find tidybot_description)/config/tidybot_controllers.yaml"/>
->>>>>>> master
     <xacro:include filename="$(find tidybot_description)/urdf/bot.xacro" />
     <!-- load the robot -->
     <xacro:load_bot arm="$(arg arm)" gripper="$(arg gripper)" vision="$(arg vision)" prefix="$(arg prefix)" />
-<<<<<<< HEAD
-=======
     <!-- configure ros2_control joints -->
     <xacro:include filename="$(find tidybot_description)/urdf/ros2_control.xacro" />
     <xacro:load_ros2_control config_path="$(arg ros2_control_config_path)" hardware_plugin="$(arg hardware_plugin)" />
->>>>>>> master
 </robot>

File: src/tidybot_moveit_config/config/tidybot.urdf.xacro (robot description, xacro)
@@ -2,15 +2,6 @@
 <robot xmlns:xacro="http://www.ros.org/wiki/xacro" name="tidybot">
     <xacro:arg name="initial_positions_file" default="initial_positions.yaml" />
-<<<<<<< HEAD
-=======
     <xacro:arg name="ros2_control_config_path" default="$(find tidybot_description)/config/tidybot_controllers.yaml"/>
->>>>>>> master
     <!-- Import tidybot urdf file -->
     <xacro:include filename="$(find tidybot_description)/urdf/tidybot.xacro" />
-<<<<<<< HEAD
-    <!-- Import control_xacro -->
-    <xacro:include filename="tidybot.ros2_control.xacro" />
-    <xacro:tidybot_ros2_control name="FakeSystem" initial_positions_file="$(arg initial_positions_file)"/>
-=======
->>>>>>> master
 </robot>

Commit message: update xacro files and launch files in tidybot_description

File: src/tidybot_description/urdf/arms/gen3_lite/gen3_lite_macro.xacro (robot description, xacro)
@@ -5,5 +5,5 @@
   <xacro:macro name="load_arm" params="parent:='' vision prefix *origin">
     <joint name="${prefix}arm_base_joint" type="fixed">
-      <origin xyz="0 0 0.335" rpy="0 0 0" />
+      <origin xyz="0 0 0.33" rpy="0 0 0" />
       <parent link="${parent}" />
       <child link="${prefix}arm_base_link" />

File: src/tidybot_description/urdf/base/base.xacro (robot description, xacro)
@@ -1,10 +1,8 @@
 <?xml version="1.0"?>
 <robot name="tidybot_base" xmlns:xacro="http://ros.org/wiki/xacro">
-    <xacro:property name="last_base_link" value="base_link"/>
+    <xacro:property name="last_base_link" value="base"/>
     <xacro:macro name="load_base" params="parent:='' prefix">
-        <link name="world">
-            <origin xyz="0.0 0.0 0.0" rpy="0.0 0.0 0.0"/>
-        </link>
-        <link name="${prefix}base_link">
+        <link name="world"></link>
+        <link name="${prefix}base">
             <inertial>
                 <origin xyz="0.0 0.0 0.035" rpy="0.0 0.0 0.0"/>
@@ -12,69 +10,4 @@
                 <inertia ixx="0.001" iyy="0.001" izz="0.001" ixy="0" ixz="0" iyz="0"/>
             </inertial>
-            <visual name="bumper">
-                <origin xyz="-1.3915598211675165e-07 -2.058962502098711e-07 0.05386474576457055" rpy="-2.442021632452952 -1.5707963267948966 0.0"/>
-                <geometry>
-                    <mesh filename="file://$(find tidybot_description)/meshes/base/bumper.stl"/>
-                </geometry>
-                <material name="white"/>
-            </visual>
-            <collision name="bumper">
-                <origin xyz="-1.3915598211675165e-07 -2.058962502098711e-07 0.05386474576457055" rpy="-2.442021632452952 -1.5707963267948966 0.0"/>
-                <geometry>
-                    <mesh filename="file://$(find tidybot_description)/meshes/base/bumper.stl"/>
-                </geometry>
-            </collision>
-            <visual name="bottom_plate">
-                <origin xyz="4.155854111430312e-11 1.8201972332496634e-11 0.08495000004768373" rpy="1.6659662035857206 -1.5707963267948966 0.0"/>
-                <geometry>
-                    <mesh filename="file://$(find tidybot_description)/meshes/base/bottom_plate.stl"/>
-                </geometry>
-                <material name="white"/>
-            </visual>
-            <collision name="bottom_plate">
-                <origin xyz="4.155854111430312e-11 1.8201972332496634e-11 0.08495000004768373" rpy="1.6659662035857206 -1.5707963267948966 0.0"/>
-                <geometry>
-                    <mesh filename="file://$(find tidybot_description)/meshes/base/bottom_plate.stl"/>
-                </geometry>
-            </collision>
-            <visual name="body">
-                <origin xyz="7.590768644441668e-06 -6.000635064190085e-10 0.20330222068596052" rpy="-1.5707963267948966 -1.570779305272103 3.141592653589793"/>
-                <geometry>
-                    <mesh filename="file://$(find tidybot_description)/meshes/base/body.stl"/>
-                </geometry>
-                <material name="white"/>
-            </visual>
-            <collision name="body">
-                <origin xyz="7.590768644441668e-06 -6.000635064190085e-10 0.20330222068596052" rpy="-1.5707963267948966 -1.570779305272103 3.141592653589793"/>
-                <geometry>
-                    <mesh filename="file://$(find tidybot_description)/meshes/base/body.stl"/>
-                </geometry>
-            </collision>
-            <visual name="top_plate">
-                <origin xyz="-2.9658670629084936e-11 -3.476524862019053e-11 0.3216499984264373" rpy="1.6906681075416252 -1.5707963267948966 0.0"/>
-                <geometry>
-                    <mesh filename="file://$(find tidybot_description)/meshes/base/top_plate.stl"/>
-                </geometry>
-                <material name="white"/>
-            </visual>
-            <collision name="top_plate">
-                <origin xyz="-2.9658670629084936e-11 -3.476524862019053e-11 0.3216499984264373" rpy="1.6906681075416252 -1.5707963267948966 0.0"/>
-                <geometry>
-                    <mesh filename="file://$(find tidybot_description)/meshes/base/top_plate.stl"/>
-                </geometry>
-            </collision>
-            <visual name="arm_plate">
-                <origin xyz="-2.7580994002430455e-12 -3.3382504263355704e-12 0.32999999883475684" rpy="1.5707963267948966 -1.5707963267948966 0.0"/>
-                <geometry>
-                    <mesh filename="file://$(find tidybot_description)/meshes/base/arm_plate.stl"/>
-                </geometry>
-                <material name="white"/>
-            </visual>
-            <collision name="arm_plate">
-                <origin xyz="-2.7580994002430455e-12 -3.3382504263355704e-12 0.32999999883475684" rpy="1.5707963267948966 -1.5707963267948966 0.0"/>
-                <geometry>
-                    <mesh filename="file://$(find tidybot_description)/meshes/base/arm_plate.stl"/>
-                </geometry>
-            </collision>
             <visual name="bumper">
                 <origin xyz="-1.3915598211675165e-07 -2.058962502098711e-07 0.05386474576457055" rpy="-2.442021632452952 -1.5707963267948966 0.0"/>
@@ -212,5 +145,5 @@
             <origin xyz="-0.0 -0.0 -0.0" rpy="0.0 0.0 0.0"/>
             <parent link="joint_th_jointbody"/>
-            <child link="base_link"/>
+            <child link="base"/>
             <axis xyz="0.0 0.0 1.0"/>
             <limit lower="0.0" upper="0.0" effort="100" velocity="100"/>

File: src/tidybot_description/urdf/grippers/gen3_lite_2f/gen3_lite_2f_macro.xacro (robot description, xacro)
@@ -32,10 +32,11 @@
         </material>
       </visual>
-      <collision>
+      <!-- TODO: replace with simplified mesh -->
+      <!-- <collision>
         <origin xyz="0 0 0" rpy="0 0 0" />
         <geometry>
           <mesh filename="file://$(find tidybot_description)/meshes/grippers/gen3_lite_2f/gripper_base_link.STL" />
         </geometry>
-      </collision>
+      </collision> -->
     </link>
     <gazebo reference="${prefix}gripper_base_link">
@@ -57,10 +58,10 @@
       </material>
     </visual>
-    <collision>
+    <!-- <collision>
       <origin xyz="0 0 0" rpy="0 0 0" />
       <geometry>
         <mesh filename="file://$(find tidybot_description)/meshes/grippers/gen3_lite_2f/right_finger_prox_link.STL" />
       </geometry>
-    </collision>
+    </collision> -->
     </link>
     <gazebo reference="${prefix}right_finger_prox_link">
@@ -97,10 +98,10 @@
         </material>
       </visual>
-      <collision>
+      <!-- <collision>
         <origin xyz="0 0 0" rpy="0 0 0" />
         <geometry>
           <mesh filename="file://$(find tidybot_description)/meshes/grippers/gen3_lite_2f/right_finger_dist_link.STL" />
         </geometry>
-      </collision>
+      </collision> -->
     </link>
     <gazebo reference="${prefix}right_finger_dist_link">
@@ -138,10 +139,10 @@
         </material>
       </visual>
-      <collision>
+      <!-- <collision>
         <origin xyz="0 0 0" rpy="0 0 0" />
         <geometry>
           <mesh filename="file://$(find tidybot_description)/meshes/grippers/gen3_lite_2f/left_finger_prox_link.STL" />
         </geometry>
-      </collision>
+      </collision> -->
     </link>
     <gazebo reference="${prefix}left_finger_prox_link">
@@ -179,10 +180,10 @@
         </material>
       </visual>
-      <collision>
+      <!-- <collision>
         <origin xyz="0 0 0" rpy="0 0 0" />
         <geometry>
           <mesh filename="file://$(find tidybot_description)/meshes/grippers/gen3_lite_2f/left_finger_dist_link.STL" />
         </geometry>
-      </collision>
+      </collision> -->
     </link>
     <gazebo reference="${prefix}left_finger_dist_link">

File: src/tidybot_description/urdf/tidybot.ros2_control.xacro (robot description, xacro)
@@ -1,5 +1,5 @@
 <?xml version="1.0"?>
 <robot name="ros2_control" xmlns:xacro="http://ros.org/wiki/xacro">
-    <xacro:macro name="load_ros2_control" params="config_path hardware_plugin">
+    <xacro:macro name="load_ros2_control" params="hardware_plugin">
         <xacro:macro name="add_joint" params="name gain cmd_interface">
             <joint name="${name}">
@@ -31,11 +31,4 @@
         <xacro:add_joint name="left_finger_tip_joint" gain="0.1" cmd_interface="position"/>
         </ros2_control>
-        <gazebo>
-            <plugin name="gz_ros2_control::GazeboSimROS2ControlPlugin" filename="gz_ros2_control-system">
-                <parameters>${config_path}</parameters>
-                <robot_description_param>robot_description</robot_description_param>
-            </plugin>
-            <self_collide>true</self_collide>
-        </gazebo>
     </xacro:macro>
 </robot>

File: src/tidybot_description/urdf/tidybot.urdf (robot description, URDF)
Before this commit: robot tidybot, 18 links, 17 joints
Links:
- removed link arm_base_link
- removed link arm_link
- removed link end_effector_link
- removed link forearm_link
- removed link gripper_base_link
- removed link joint_th_jointbody
- removed link joint_x_jointbody
- removed link joint_y_jointbody
- removed link left_finger_dist_link
- removed link left_finger_prox_link
- removed link lower_wrist_link
- removed link right_finger_dist_link
- removed link right_finger_prox_link
- removed link shoulder_link
- removed link tool_frame
- removed link upper_wrist_link
- removed link world
- added link base_footprint
- added link front_left_wheel, mass 5.0; collision cylinder length=.05 radius=.1; visual mesh filename=package://bme_gazebo_basics/meshes/wheel.dae
- added link front_right_wheel, mass 5.0; collision cylinder length=.05 radius=.1; visual mesh filename=package://bme_gazebo_basics/meshes/wheel.dae
- added link rear_left_wheel, mass 5.0; collision cylinder length=.05 radius=.1; visual mesh filename=package://bme_gazebo_basics/meshes/wheel.dae
- added link rear_right_wheel, mass 5.0; collision cylinder length=.05 radius=.1; visual mesh filename=package://bme_gazebo_basics/meshes/wheel.dae
- link base_link: mass 60.0 -> 15.0; geometry collision box size=.4 .2 .1; visual mesh filename=package://bme_gazebo_basics/meshes/mogi_bot.dae
Joints:
- removed joint arm_base_joint
- removed joint gripper_base_joint
- removed joint joint_1
- removed joint joint_2
- removed joint joint_3
- removed joint joint_4
- removed joint joint_5
- removed joint joint_6
- removed joint joint_th
- removed joint joint_th_offset
- removed joint joint_x
- removed joint joint_y
- removed joint left_finger_bottom_joint
- removed joint left_finger_tip_joint
- removed joint right_finger_bottom_joint
- removed joint right_finger_tip_joint
- removed joint tool_frame_joint
- added joint base_footprint_joint: type fixed, parent base_footprint, child base_link, origin xyz=0 0 0 rpy=0 0 0
- added joint front_left_wheel_joint: type continuous, parent base_link, child front_left_wheel, origin xyz=0.15 0.15 0 rpy=0 0 0, axis 0 1 0, limit effort=100 velocity=10
- added joint front_right_wheel_joint: type continuous, parent base_link, child front_right_wheel, origin xyz=0.15 -0.15 0 rpy=0 0 0, axis 0 1 0, limit effort=100 velocity=10
- added joint rear_left_wheel_joint: type continuous, parent base_link, child rear_left_wheel, origin xyz=-0.15 0.15 0 rpy=0 0 0, axis 0 1 0, limit effort=100 velocity=10
- added joint rear_right_wheel_joint: type continuous, parent base_link, child rear_right_wheel, origin xyz=-0.15 -0.15 0 rpy=0 0 0, axis 0 1 0, limit effort=100 velocity=10

File: src/tidybot_description/urdf/tidybot.xacro (robot description, xacro)
@@ -11,5 +11,8 @@
     <xacro:load_bot arm="$(arg arm)" gripper="$(arg gripper)" vision="$(arg vision)" prefix="$(arg prefix)" />
     <!-- configure ros2_control joints -->
-    <xacro:include filename="$(find tidybot_description)/urdf/ros2_control.xacro" />
-    <xacro:load_ros2_control config_path="$(arg ros2_control_config_path)" hardware_plugin="$(arg hardware_plugin)" />
+    <xacro:include filename="$(find tidybot_description)/urdf/tidybot.ros2_control.xacro" />
+    <xacro:load_ros2_control hardware_plugin="$(arg hardware_plugin)" />
+    <!-- load gazebo plugins -->
+    <xacro:include filename="$(find tidybot_description)/urdf/tidybot.gazebo.xacro" />
+    <xacro:load_gazebo_plugins config_path="$(arg ros2_control_config_path)" />
 </robot>
