Commit message: add gen3_7dof arm xacro

File: src/tidybot_description/urdf/arms/gen3_lite/gen3_lite_macro.xacro (robot description, xacro)
@@ -67,11 +67,4 @@
       <dynamics damping="1.0" friction="1.0"/>
     </joint>
-    <transmission name="joint1_trans">
-      <type>transmission_interface/SimpleTransmission</type>
-      <joint name="${prefix}joint_1" />
-      <actuator name="joint1_motor">
-        <mechanicalReduction>1</mechanicalReduction>
-      </actuator>
-    </transmission>
     <link name="${prefix}arm_link">
       <inertial>
@@ -107,11 +100,4 @@
       <dynamics damping="1.0" friction="1.0"/>
     </joint>
-    <transmission name="joint2_trans">
-      <type>transmission_interface/SimpleTransmission</type>
-      <joint name="${prefix}joint_2" />
-      <actuator name="joint2_motor">
-        <mechanicalReduction>1</mechanicalReduction>
-      </actuator>
-    </transmission>
     <link name="${prefix}forearm_link">
       <inertial>
@@ -147,11 +133,4 @@
       <dynamics damping="1.0" friction="1.0"/>
     </joint>
-    <transmission name="joint3_trans">
-      <type>transmission_interface/SimpleTransmission</type>
-      <joint name="${prefix}joint_3" />
-      <actuator name="joint3_motor">
-        <mechanicalReduction>1</mechanicalReduction>
-      </actuator>
-    </transmission>
     <link name="${prefix}lower_wrist_link">
       <inertial>
@@ -187,11 +166,4 @@
       <dynamics damping="1.0" friction="1.0"/>
     </joint>
-    <transmission name="joint4_trans">
-      <type>transmission_interface/SimpleTransmission</type>
-      <joint name="${prefix}joint_4" />
-      <actuator name="joint4_motor">
-        <mechanicalReduction>1</mechanicalReduction>
-      </actuator>
-    </transmission>
     <link name="${prefix}upper_wrist_link">
       <inertial>
@@ -227,11 +199,4 @@
       <dynamics damping="1.0" friction="1.0"/>
     </joint>
-    <transmission name="joint5_trans">
-      <type>transmission_interface/SimpleTransmission</type>
-      <joint name="${prefix}joint_5" />
-      <actuator name="joint5_motor">
-        <mechanicalReduction>1</mechanicalReduction>
-      </actuator>
-    </transmission>
     <link name="${prefix}end_effector_link" />
     <joint name="${prefix}joint_6" type="revolute">
@@ -243,11 +208,4 @@
       <dynamics damping="1.0" friction="1.0"/>
     </joint>
-    <transmission name="joint6_trans">
-      <type>transmission_interface/SimpleTransmission</type>
-      <joint name="${prefix}joint_6" />
-      <actuator name="joint6_motor">
-        <mechanicalReduction>1</mechanicalReduction>
-      </actuator>
-    </transmission>
   </xacro:macro>
 </robot>

File: src/tidybot_description/urdf/tidybot.gazebo.xacro (robot description, xacro)
@@ -1,5 +1,5 @@
 <?xml version="1.0"?>
 <robot xmlns:xacro="http://ros.org/wiki/xacro">
-<xacro:macro name="load_gazebo_plugins" params="config_path">
+<xacro:macro name="load_gazebo_plugins" params="config_path prefix arm">
   <gazebo>
       <plugin name="gz_ros2_control::GazeboSimROS2ControlPlugin" filename="gz_ros2_control-system">
@@ -18,4 +18,6 @@
     </plugin>
   </gazebo>
+  <xacro:include filename="$(find tidybot_description)/urdf/arms/${arm}/${arm}_transmission.xacro" />
+  <xacro:load_arm_transmission prefix="${prefix}" />
 </xacro:macro>
 </robot>

File: src/tidybot_description/urdf/tidybot.ros2_control.xacro (robot description, xacro)
@@ -1,5 +1,5 @@
 <?xml version="1.0"?>
 <robot name="ros2_control" xmlns:xacro="http://ros.org/wiki/xacro">
-    <xacro:macro name="load_ros2_control" params="hardware_plugin">
+    <xacro:macro name="load_ros2_control" params="hardware_plugin arm">
         <xacro:macro name="add_joint" params="name gain cmd_interface">
             <joint name="${name}">
@@ -26,4 +26,7 @@
         <xacro:add_joint name="joint_5" gain="0.1" cmd_interface="position"/>
         <xacro:add_joint name="joint_6" gain="0.1" cmd_interface="position"/>
+        <xacro:if value="${arm == 'gen3_7dof'}">
+            <xacro:add_joint name="joint_7" gain="0.1" cmd_interface="position"/>
+        </xacro:if>
         <xacro:add_joint name="right_finger_bottom_joint" gain="0.1" cmd_interface="position"/>
         <xacro:add_joint name="right_finger_tip_joint" gain="0.1" cmd_interface="position"/>

File: src/tidybot_description/urdf/tidybot.xacro (robot description, xacro)
@@ -3,5 +3,5 @@
     <!-- <xacro:arg name="hardware_plugin" default="mock_components/GenericSystem" />     -->
     <xacro:arg name="hardware_plugin" default="gz_ros2_control/GazeboSimSystem" />
-    <xacro:arg name="arm" default="gen3_lite" />
+    <xacro:arg name="arm" default="gen3_7dof" />
     <xacro:arg name="gripper" default="gen3_lite_2f" />
     <xacro:arg name="vision" default="false" />
@@ -13,7 +13,7 @@
     <!-- configure ros2_control joints -->
     <xacro:include filename="$(find tidybot_description)/urdf/tidybot.ros2_control.xacro" />
-    <xacro:load_ros2_control hardware_plugin="$(arg hardware_plugin)" />
+    <xacro:load_ros2_control hardware_plugin="$(arg hardware_plugin)" arm="$(arg arm)" />
     <!-- load gazebo plugins -->
     <xacro:include filename="$(find tidybot_description)/urdf/tidybot.gazebo.xacro" />
-    <xacro:load_gazebo_plugins config_path="$(arg ros2_control_config_path)" />
+    <xacro:load_gazebo_plugins config_path="$(arg ros2_control_config_path)" prefix="$(arg prefix) " arm="$(arg arm)" />
 </robot>
