Commit message: update episode recorder

File: src/tidybot_description/urdf/base/tidybot++/base_kinova_macro.xacro (robot description, xacro)
@@ -21,5 +21,5 @@
             </visual>
             <collision>
-                <origin xyz="-0.3066 0.064 0.0.085" rpy="0 -0 0"/>
+                <origin xyz="-0.3066 0.064 0.085" rpy="0 -0 0"/>
                 <geometry>
                     <mesh filename="file://$(find tidybot_description)/meshes/base/tidybot++/Kinova.stl"/>

Commit message: update the base camera

File: src/tidybot_description/urdf/base/tidybot++/base_kinova_macro.xacro (robot description, xacro)
@@ -30,9 +30,9 @@
             <link name="${prefix}base_camera_link" />
             <joint type="fixed" name="${prefix}base_camera_joint">
-                <origin xyz="0.2285 0.0 0.315" rpy="0.0 1.57079632679 0.0"/>
+                <origin xyz="0.2525 0.0 0.315" rpy="0 0.7853981634 0"/>
                 <parent link="${prefix}base"/>
                 <child link="${prefix}base_camera_link"/>
                 <visual>
-                    <origin xyz="0.2285 0.0 0.315" rpy="0.0 0.0 0.0"/>
+                    <origin xyz="0.2285 0.0 0.315" rpy="0 0 0"/>
                     <geometry>
                         <box size="0.1 0.1 0.1"/>

File: src/tidybot_description/urdf/tidybot.gazebo.xacro (robot description, xacro)
@@ -52,9 +52,9 @@
         <update_rate>30</update_rate>
         <visualize>true</visualize>
-        <pose>0 0 0 0 4.7124 0</pose>
+        <pose>0 0 0 0 0 0</pose>
 				<topic>/base_camera</topic>
         <gz_frame_id>${prefix}base_camera_link</gz_frame_id>
         <camera>
-          <horizontal_fov>1.047</horizontal_fov>
+          <horizontal_fov>1.434</horizontal_fov>
           <image>
             <width>640</width>

Commit message: update diffusion policy control

File: src/tidybot_description/urdf/base/tidybot++/base_kinova_macro.xacro (robot description, xacro)
@@ -16,6 +16,6 @@
                     <mesh filename="file://$(find tidybot_description)/meshes/base/tidybot++/Kinova.stl"/>
                 </geometry>
-                <material name="kinova_material">
-                    <color rgba="0.917647 0.917647 0.917647 1"/>
+                <material name="grey">
+                    <color rgba="0.5 0.5 0.5 1"/>
                 </material>
             </visual>
@@ -96,6 +96,6 @@
             <limit lower="0.0" upper="0.0" effort="100" velocity="100"/>
         </joint>
-        <material name="white">
-            <color rgba="1 1 1 1"/>
+        <material name="grey">
+            <color rgba="0.5 0.5 0.5 1"/>
         </material>
     </xacro:macro>

File: src/tidybot_description/urdf/grippers/robotiq_2f_85/robotiq_arg2f_85_model_macro.xacro (robot description, xacro)
@@ -108,5 +108,5 @@
         </geometry>
         <material name="">
-          <color rgba="0.9 0.9 0.9 1" />
+          <color rgba="0.0 0.0 0.0 1" />
         </material>
       </visual>
@@ -117,5 +117,5 @@
         </geometry>
         <material name="">
-          <color rgba="0.9 0.0 0.0 1" />
+          <color rgba="0.0 0.0 0.0 1" />
         </material>
       </collision>

File: src/tidybot_description/urdf/tidybot.gazebo.xacro (robot description, xacro)
@@ -28,5 +28,5 @@
         <gz_frame_id>${prefix}arm_camera_link</gz_frame_id>
         <camera>
-          <horizontal_fov>1.147</horizontal_fov>
+          <horizontal_fov>1.247</horizontal_fov>
           <image>
             <width>640</width>
