Commit message: add rgbd_camera

File: src/tidybot_description/urdf/grippers/robotiq_2f_85/robotiq_2f_85_macro.xacro (robot description, xacro)
@@ -2,5 +2,5 @@
 <robot name="robotiq_arg2f_85_model" xmlns:xacro="http://ros.org/wiki/xacro">
   <xacro:macro name="load_gripper" params="parent prefix">
-    <xacro:include filename="$(find simulation)/urdf/grippers/robotiq_2f_85/robotiq_arg2f_85_model_macro.xacro" />
+    <xacro:include filename="$(find tidybot_description)/urdf/grippers/robotiq_2f_85/robotiq_arg2f_85_model_macro.xacro" />
     <xacro:robotiq_arg2f_85 parent="${parent}" prefix="${prefix}"/>
   </xacro:macro>

File: src/tidybot_description/urdf/grippers/robotiq_2f_85/robotiq_arg2f.xacro (robot description, xacro)
@@ -19,5 +19,5 @@
           <!-- The DAE file doesn't show well in Gazebo so we're using the STL instead -->
           <!-- <mesh filename="file://$(find simulation)/meshes/grippers/robotiq_2f_85/meshes/visual/robotiq_arg2f_85_base_link.dae" scale="0.001 0.001 0.001"/> -->
-          <mesh filename="file://$(find simulation)/meshes/grippers/robotiq_2f_85/collision/robotiq_arg2f_base_link.stl" />
+          <mesh filename="file://$(find tidybot_description)/meshes/grippers/robotiq_2f_85/collision/robotiq_arg2f_base_link.stl" />
         </geometry>
         <material name="">
@@ -28,5 +28,5 @@
         <origin xyz="0 0 0" rpy="0 0 0" />
         <geometry>
-           <mesh filename="file://$(find simulation)/meshes/grippers/robotiq_2f_85/collision/robotiq_arg2f_base_link.stl" />
+           <mesh filename="file://$(find tidybot_description)/meshes/grippers/robotiq_2f_85/collision/robotiq_arg2f_base_link.stl" />
         </geometry>
       </collision>

File: src/tidybot_description/urdf/grippers/robotiq_2f_85/robotiq_arg2f_85_model_macro.xacro (robot description, xacro)
@@ -13,5 +13,5 @@
         <origin xyz="0 0 0" rpy="0 0 0" />
         <geometry>
-          <mesh filename="file://$(find simulation)/meshes/grippers/robotiq_2f_85/visual/robotiq_arg2f_85_outer_knuckle.dae" scale="0.001 0.001 0.001"/>
+          <mesh filename="file://$(find tidybot_description)/meshes/grippers/robotiq_2f_85/visual/robotiq_arg2f_85_outer_knuckle.dae" scale="0.001 0.001 0.001"/>
         </geometry>
         <material name="">
@@ -22,5 +22,5 @@
         <origin xyz="0 0 0" rpy="0 0 0" />
         <geometry>
-          <mesh filename="file://$(find simulation)/meshes/grippers/robotiq_2f_85/collision/robotiq_arg2f_85_outer_knuckle.dae" scale="0.001 0.001 0.001"/>
+          <mesh filename="file://$(find tidybot_description)/meshes/grippers/robotiq_2f_85/collision/robotiq_arg2f_85_outer_knuckle.dae" scale="0.001 0.001 0.001"/>
         </geometry>
       </collision>
@@ -37,5 +37,5 @@
         <origin xyz="0 0 0" rpy="0 0 0" />
         <geometry>
-          <mesh filename="file://$(find simulation)/meshes/grippers/robotiq_2f_85/visual/robotiq_arg2f_85_outer_finger.dae" scale="0.001 0.001 0.001"/>
+          <mesh filename="file://$(find tidybot_description)/meshes/grippers/robotiq_2f_85/visual/robotiq_arg2f_85_outer_finger.dae" scale="0.001 0.001 0.001"/>
         </geometry>
         <material name="">
@@ -46,5 +46,5 @@
         <origin xyz="0 0 0" rpy="0 0 0" />
         <geometry>
-          <mesh filename="file://$(find simulation)/meshes/grippers/robotiq_2f_85/collision/robotiq_arg2f_85_outer_finger.dae" scale="0.001 0.001 0.001"/>
+          <mesh filename="file://$(find tidybot_description)/meshes/grippers/robotiq_2f_85/collision/robotiq_arg2f_85_outer_finger.dae" scale="0.001 0.001 0.001"/>
         </geometry>
       </collision>
@@ -61,5 +61,5 @@
         <origin xyz="0 0 0" rpy="0 0 0" />
         <geometry>
-          <mesh filename="file://$(find simulation)/meshes/grippers/robotiq_2f_85/visual/robotiq_arg2f_85_inner_knuckle.dae" scale="0.001 0.001 0.001"/>
+          <mesh filename="file://$(find tidybot_description)/meshes/grippers/robotiq_2f_85/visual/robotiq_arg2f_85_inner_knuckle.dae" scale="0.001 0.001 0.001"/>
         </geometry>
         <material name="">
@@ -70,5 +70,5 @@
         <origin xyz="0 0 0" rpy="0 0 0" />
         <geometry>
-          <mesh filename="file://$(find simulation)/meshes/grippers/robotiq_2f_85/collision/robotiq_arg2f_85_inner_knuckle.dae" scale="0.001 0.001 0.001"/>
+          <mesh filename="file://$(find tidybot_description)/meshes/grippers/robotiq_2f_85/collision/robotiq_arg2f_85_inner_knuckle.dae" scale="0.001 0.001 0.001"/>
         </geometry>
       </collision>
@@ -85,5 +85,5 @@
         <origin xyz="0 0 0" rpy="0 0 0" />
         <geometry>
-          <mesh filename="file://$(find simulation)/meshes/grippers/robotiq_2f_85/visual/robotiq_arg2f_85_inner_finger.dae" scale="0.001 0.001 0.001"/>
+          <mesh filename="file://$(find tidybot_description)/meshes/grippers/robotiq_2f_85/visual/robotiq_arg2f_85_inner_finger.dae" scale="0.001 0.001 0.001"/>
         </geometry>
         <material name="">
@@ -94,5 +94,5 @@
         <origin xyz="0 0 0" rpy="0 0 0" />
         <geometry>
-          <mesh filename="file://$(find simulation)/meshes/grippers/robotiq_2f_85/collision/robotiq_arg2f_85_inner_finger.dae" scale="0.001 0.001 0.001" />
+          <mesh filename="file://$(find tidybot_description)/meshes/grippers/robotiq_2f_85/collision/robotiq_arg2f_85_inner_finger.dae" scale="0.001 0.001 0.001" />
         </geometry>
       </collision>
@@ -138,5 +138,5 @@
       <axis xyz="1 0 0" />
       <limit lower="0" upper="0.8757" velocity="2.0" effort="1000" />
-      <mimic joint="${prefix}finger_joint" multiplier="1" offset="0" />
+      <!-- <mimic joint="${prefix}finger_joint" multiplier="1" offset="0" /> -->
     </joint>
     <transmission name="{prefix}${fingerprefix}_inner_knuckle_joint_trans">
@@ -155,5 +155,5 @@
       <axis xyz="1 0 0" />
       <limit lower="-0.8757" upper="0.8757" velocity="2.0" effort="1000" />
-      <mimic joint="${prefix}finger_joint" multiplier="-1" offset="0" />
+      <!-- <mimic joint="${prefix}finger_joint" multiplier="-1" offset="0" /> -->
     </joint>
     <transmission name="${prefix}${fingerprefix}_inner_finger_joint_trans">
@@ -173,5 +173,5 @@
     </joint>
   </xacro:macro>
-  <xacro:include filename="$(find kortex_description)/grippers/robotiq_2f_85/urdf/robotiq_arg2f.xacro" />
+  <xacro:include filename="$(find tidybot_description)/urdf/grippers/robotiq_2f_85/robotiq_arg2f.xacro" />
   <xacro:macro name="finger_joint" params="prefix">
     <joint name="${prefix}finger_joint" type="revolute">
@@ -198,5 +198,5 @@
       <axis xyz="1 0 0" />
       <limit lower="0" upper="0.81" velocity="2.0" effort="1000" />
-      <mimic joint="${prefix}finger_joint" multiplier="1" offset="0" />
+      <!-- <mimic joint="${prefix}finger_joint" multiplier="1" offset="0" /> -->
     </joint>
     <transmission name="$${prefix}right_outer_knuckle_joint_trans">

File: src/tidybot_description/urdf/tidybot.gazebo.xacro (robot description, xacro)
@@ -1,10 +1,11 @@
 <?xml version="1.0"?>
 <robot xmlns:xacro="http://ros.org/wiki/xacro">
-<xacro:macro name="load_gazebo_plugins" params="config_path prefix arm">
+<xacro:macro name="load_gazebo_plugins" params="config_path prefix arm vision">
   <gazebo>
       <plugin name="gz_ros2_control::GazeboSimROS2ControlPlugin" filename="gz_ros2_control-system">
           <parameters>${config_path}</parameters>
-          <!-- <robot_description_param>robot_description</robot_description_param> -->
+          <robot_description_param>robot_description</robot_description_param>
       </plugin>
+      <plugin name="ignition::gazebo::systems::Sensors" filename="libignition-gazebo-sensors-system.so"/>
       <!-- <self_collide>true</self_collide> -->
   </gazebo>
@@ -18,4 +19,33 @@
     </plugin>
   </gazebo> -->
+  <xacro:if value="${vision}">
+    <gazebo reference="${prefix}camera_link">
+      <sensor name="${prefix}camera" type="rgbd_camera">
+        <always_on>1</always_on>
+        <update_rate>30</update_rate>
+        <visualize>true</visualize>
+        <pose>0 -0.01 0.03 0 4.7124 1.5708</pose>
+				<topic>/camera</topic>
+        <gz_frame_id>${prefix}camera_link</gz_frame_id>
+        <camera>
+          <horizontal_fov>1.047</horizontal_fov>
+          <image>
+            <width>640</width>
+            <height>480</height>
+            <format>R8G8B8</format>
+          </image>
+          <clip>
+            <near>0.03</near>
+            <far>3.0</far>
+          </clip>
+          <noise>
+            <type>gaussian</type>
+            <mean>0.0</mean>
+            <stddev>0.007</stddev>
+          </noise>
+        </camera>
+      </sensor>
+    </gazebo>
+  </xacro:if>
   <xacro:include filename="$(find tidybot_description)/urdf/arms/${arm}/${arm}_transmission.xacro" />
   <xacro:load_arm_transmission prefix="${prefix}" />

File: src/tidybot_description/urdf/tidybot.ros2_control.xacro (robot description, xacro)
@@ -1,5 +1,5 @@
 <?xml version="1.0"?>
 <robot name="ros2_control" xmlns:xacro="http://ros.org/wiki/xacro">
-    <xacro:macro name="load_ros2_control" params="hardware_plugin arm">
+    <xacro:macro name="load_ros2_control" params="hardware_plugin arm gripper">
         <xacro:macro name="add_joint" params="name gain cmd_interface">
             <joint name="${name}">
@@ -29,8 +29,18 @@
             <xacro:add_joint name="joint_7" gain="0.1" cmd_interface="position"/>
         </xacro:if>
-        <xacro:add_joint name="right_finger_bottom_joint" gain="0.1" cmd_interface="position"/>
-        <xacro:add_joint name="right_finger_tip_joint" gain="0.1" cmd_interface="position"/>
-        <xacro:add_joint name="left_finger_bottom_joint" gain="0.1" cmd_interface="position"/>
-        <xacro:add_joint name="left_finger_tip_joint" gain="0.1" cmd_interface="position"/>
+        <xacro:if value="${gripper == 'gen3_lite_2f'}">
+            <xacro:add_joint name="right_finger_bottom_joint" gain="0.1" cmd_interface="position"/>
+            <xacro:add_joint name="right_finger_tip_joint" gain="0.1" cmd_interface="position"/>
+            <xacro:add_joint name="left_finger_bottom_joint" gain="0.1" cmd_interface="position"/>
+            <xacro:add_joint name="left_finger_tip_joint" gain="0.1" cmd_interface="position"/>
+        </xacro:if>
+        <xacro:if value="${gripper == 'robotiq_2f_85'}">
+            <xacro:add_joint name="right_inner_finger_joint" gain="0.1" cmd_interface="position"/>
+            <xacro:add_joint name="right_outer_knuckle_joint" gain="0.1" cmd_interface="position"/>
+            <xacro:add_joint name="right_inner_knuckle_joint" gain="0.1" cmd_interface="position"/>
+            <xacro:add_joint name="left_inner_finger_joint" gain="0.1" cmd_interface="position"/>
+            <xacro:add_joint name="left_outer_knuckle_joint" gain="0.1" cmd_interface="position"/>
+            <xacro:add_joint name="left_inner_knuckle_joint" gain="0.1" cmd_interface="position"/>
+        </xacro:if>
         </ros2_control>
     </xacro:macro>

File: src/tidybot_description/urdf/tidybot.urdf (robot description, URDF)
Before this commit: robot tidybot, 20 links, 19 joints
Links:
- added link camera_color_frame
- added link camera_depth_frame
- added link camera_link
- link arm_base_link: geometry collision mesh filename=file:///home/yuandi/tidybot_platform/install/tidybot_descri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; visual mesh filename=file:///home/yuandi/tidybot_platform/install/tidybot_descri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
- link base: geometry collision mesh filename=file:///home/yuandi/tidybot_platform/install/tidybot_descri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; collision mesh filename=file:///home/yuandi/tidybot_platform/install/tidybot_descri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
- link bracelet_link: mass 0.364 -> 0.5; geometry collision mesh filename=file:///home/yuandi/tidybot_platform/install/tidybot_descri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; visual mesh filename=file:///home/yuandi/tidybot_platform/install/tidybot_descri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
- link forearm_link: geometry collision mesh filename=file:///home/yuandi/tidybot_platform/install/tidybot_descri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; visual mesh filename=file:///home/yuandi/tidybot_platform/install/tidybot_descri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
- link gripper_base_link: geometry visual mesh filename=file:///home/yuandi/tidybot_platform/install/tidybot_descri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
- link half_arm_1_link: geometry collision mesh filename=file:///home/yuandi/tidybot_platform/install/tidybot_descri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; visual mesh filename=file:///home/yuandi/tidybot_platform/install/tidybot_descri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
- link half_arm_2_link: geometry collision mesh filename=file:///home/yuandi/tidybot_platform/install/tidybot_descri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; visual mesh filename=file:///home/yuandi/tidybot_platform/install/tidybot_descri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
- link left_finger_dist_link: geometry visual mesh filename=file:///home/yuandi/tidybot_platform/install/tidybot_descri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
- link left_finger_prox_link: geometry visual mesh filename=file:///home/yuandi/tidybot_platform/install/tidybot_descri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
- link right_finger_dist_link: geometry visual mesh filename=file:///home/yuandi/tidybot_platform/install/tidybot_descri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
- link right_finger_prox_link: geometry visual mesh filename=file:///home/yuandi/tidybot_platform/install/tidybot_descri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
- link shoulder_link: geometry collision mesh filename=file:///home/yuandi/tidybot_platform/install/tidybot_descri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; visual mesh filename=file:///home/yuandi/tidybot_platform/install/tidybot_descri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
- link spherical_wrist_1_link: geometry collision mesh filename=file:///home/yuandi/tidybot_platform/install/tidybot_descri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; visual mesh filename=file:///home/yuandi/tidybot_platform/install/tidybot_descri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
- link spherical_wrist_2_link: geometry collision mesh filename=file:///home/yuandi/tidybot_platform/install/tidybot_descri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; visual mesh filename=file:///home/yuandi/tidybot_platform/install/tidybot_descri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
Joints:
- added joint camera_module: type fixed, parent end_effector_link, child camera_link, origin xyz=0 0.05639 -0.00305 rpy=3.14159265358979 3.14159265358979 0
- added joint color_module: type fixed, parent end_effector_link, child camera_color_frame, origin xyz=0 0.05639 -0.00305 rpy=3.14159265358979 3.14159265358979 0
- added joint depth_module: type fixed, parent end_effector_link, child camera_depth_frame, origin xyz=0.0275 0.066 -0.00305 rpy=3.14159265358979 3.14159265358979 0

File: src/tidybot_description/urdf/tidybot.xacro (robot description, xacro)
@@ -5,5 +5,5 @@
     <xacro:arg name="arm" default="gen3_7dof" />
     <xacro:arg name="gripper" default="gen3_lite_2f" />
-    <xacro:arg name="vision" default="false" />
+    <xacro:arg name="vision" default="true" />
     <xacro:arg name="prefix" default="" />
     <xacro:arg name="ros2_control_config_path" default="$(find tidybot_description)/config/tidybot_controllers.yaml"/>
@@ -13,7 +13,7 @@
     <!-- configure ros2_control joints -->
     <xacro:include filename="$(find tidybot_description)/urdf/tidybot.ros2_control.xacro" />
-    <xacro:load_ros2_control hardware_plugin="$(arg hardware_plugin)" arm="$(arg arm)" />
+    <xacro:load_ros2_control hardware_plugin="$(arg hardware_plugin)" arm="$(arg arm)" gripper="$(arg gripper)"/>
     <!-- load gazebo plugins -->
     <xacro:include filename="$(find tidybot_description)/urdf/tidybot.gazebo.xacro" />
-    <xacro:load_gazebo_plugins config_path="$(arg ros2_control_config_path)" prefix="$(arg prefix) " arm="$(arg arm)" />
+    <xacro:load_gazebo_plugins config_path="$(arg ros2_control_config_path)" prefix="$(arg prefix)" arm="$(arg arm)" vision="$(arg vision)" />
 </robot>
