Commit message: update simulated gripper control

File: src/tidybot_description/urdf/grippers/robotiq_2f_85/robotiq_2f_85_macro.xacro (robot description, xacro)
@@ -2,6 +2,19 @@
 <robot name="robotiq_arg2f_85_model" xmlns:xacro="http://ros.org/wiki/xacro">
   <xacro:macro name="load_gripper" params="parent prefix">
+    <xacro:include filename="$(find tidybot_description)/urdf/grippers/robotiq_2f_85/robotiq_arg2f.xacro" />
     <xacro:include filename="$(find tidybot_description)/urdf/grippers/robotiq_2f_85/robotiq_arg2f_85_model_macro.xacro" />
-    <xacro:robotiq_arg2f_85 parent="${parent}" prefix="${prefix}"/>
+    <link name="${prefix}tool_frame"/>
+    <joint name="${prefix}tool_frame_joint" type="fixed">
+        <origin xyz="0 0 0.120" rpy="0 0 0" />
+        <parent link="${parent}" />
+        <child link="${prefix}tool_frame" />
+        <axis xyz="0 0 0" />
+    </joint>
+    <!-- Gripper description -->
+    <xacro:robotiq_arg2f_base_link prefix="${prefix}" parent="${parent}"/>
+    <xacro:finger_links prefix="${prefix}" fingerprefix="left" stroke="85"/>
+    <xacro:finger_links prefix="${prefix}" fingerprefix="right" stroke="85"/>
+    <xacro:left_outer_knuckle_joint prefix="${prefix}"/>
+    <xacro:right_outer_knuckle_joint prefix="${prefix}"/>
   </xacro:macro>
 </robot>

File: src/tidybot_description/urdf/grippers/robotiq_2f_85/robotiq_2f_85_transmission.xacro (robot description, xacro)
@@ -20,5 +20,5 @@
             <mechanicalReduction>1</mechanicalReduction>
         </transmission>
-       <transmission name="${prefix}right_inner_finger_joint_trans">
+        <transmission name="${prefix}right_inner_finger_joint_trans">
             <type>transmission_interface/SimpleTransmission</type>
             <joint name="${prefix}right_inner_finger_joint" />

File: src/tidybot_description/urdf/grippers/robotiq_2f_85/robotiq_arg2f.xacro (robot description, xacro)
@@ -2,4 +2,5 @@
 <robot xmlns:xacro="http://ros.org/wiki/xacro">
   <xacro:macro name="robotiq_arg2f_base_link" params="parent prefix">
+    <xacro:include filename="$(find tidybot_description)/urdf/grippers/robotiq_2f_85/robotiq_arg2f_85_model_macro.xacro" />
     <!-- This joint was added by Kinova -->
     <joint name="${prefix}gripper_base_joint" type="fixed">
@@ -28,5 +29,5 @@
         <origin xyz="0 0 0" rpy="0 0 0" />
         <geometry>
-           <mesh filename="file://$(find tidybot_description)/meshes/grippers/robotiq_2f_85/collision/robotiq_arg2f_base_link.stl" />
+          <mesh filename="file://$(find tidybot_description)/meshes/grippers/robotiq_2f_85/collision/robotiq_arg2f_base_link.stl" />
         </geometry>
       </collision>

File: src/tidybot_description/urdf/grippers/robotiq_2f_85/robotiq_arg2f_85_model_macro.xacro (robot description, xacro)
@@ -55,5 +55,5 @@
       <inertial>
         <origin xyz="0.000123011831763771 0.0507850843201817 0.00103968640075166" rpy="0 0 0" />
-       <mass value="0.0271177346495152" />
+      <mass value="0.0271177346495152" />
         <inertia ixx="2.61910379223783E-05" ixy="-2.43616858946494E-07" ixz="-6.37789906117123E-09" iyy="2.8270243746167E-06" iyz="-5.37200748039765E-07" izz="2.83695868220296E-05" />
       </inertial>
@@ -99,5 +99,5 @@
     </link>
   </xacro:macro>
-   <!-- Finger pad link, the default are the "big pads" with rubber-->
+  <!-- Finger pad link, the default are the "big pads" with rubber-->
   <xacro:macro name="inner_finger_pad" params="prefix fingerprefix">
     <link name="${prefix}${fingerprefix}_inner_finger_pad">
@@ -114,5 +114,5 @@
         <origin xyz="0 0 0" rpy="0 0 0" />
         <geometry>
-           <box size="0.022 0.00635 0.0375"/>
+          <box size="0.022 0.00635 0.0375"/>
         </geometry>
         <material name="">
@@ -138,5 +138,5 @@
       <axis xyz="1 0 0" />
       <limit lower="-1.0" upper="1.0" velocity="1.0" effort="1000" />
-      <!-- <mimic joint="${prefix}finger_joint" multiplier="1" offset="0" /> -->
+      <mimic joint="${prefix}left_outer_knuckle_joint" multiplier="1" offset="0" />
     </joint>
   </xacro:macro>
@@ -148,5 +148,5 @@
       <axis xyz="1 0 0" />
       <limit lower="-1.0" upper="1.0" velocity="1.0" effort="1000" />
-      <!-- <mimic joint="${prefix}finger_joint" multiplier="-1" offset="0" /> -->
+      <mimic joint="${prefix}left_outer_knuckle_joint" multiplier="-1" offset="0" />
     </joint>
   </xacro:macro>
@@ -159,5 +159,4 @@
     </joint>
   </xacro:macro>
-  <xacro:include filename="$(find tidybot_description)/urdf/grippers/robotiq_2f_85/robotiq_arg2f.xacro" />
   <xacro:macro name="left_outer_knuckle_joint" params="prefix">
     <joint name="${prefix}left_outer_knuckle_joint" type="revolute">
@@ -177,26 +176,7 @@
       <axis xyz="1 0 0" />
       <limit lower="-1.0" upper="1.0" velocity="1.0" effort="1000" />
-      <!-- <mimic joint="${prefix}finger_joint" multiplier="1" offset="0" /> -->
+      <mimic joint="${prefix}left_outer_knuckle_joint" multiplier="1" offset="0" />
     </joint>
     <xacro:finger_joints prefix="${prefix}" fingerprefix="right" reflect="-1.0"/>
   </xacro:macro>
-  <!-- Initialization of all joints and links -->
-  <xacro:macro name="robotiq_arg2f_85" params="prefix parent">
-    <!-- Tool frame used by the arm -->
-    <link name="${prefix}tool_frame"/>
-    <joint name="${prefix}tool_frame_joint" type="fixed">
-        <origin xyz="0 0 0.120" rpy="0 0 0" />
-        <parent link="${parent}" />
-        <child link="${prefix}tool_frame" />
-        <axis xyz="0 0 0" />
-    </joint>
-    <!-- Gripper description -->
-    <xacro:robotiq_arg2f_base_link prefix="${prefix}" parent="${parent}"/>
-    <xacro:finger_links prefix="${prefix}" fingerprefix="left" stroke="85"/>
-    <xacro:finger_links prefix="${prefix}" fingerprefix="right" stroke="85"/>
-    <xacro:left_outer_knuckle_joint prefix="${prefix}"/>
-    <xacro:right_outer_knuckle_joint prefix="${prefix}"/>
-    <!-- Transmissions are loaded in the generic kortex xacro when simulation is enabled -->
-    <!-- <xacro:robotiq_arg2f_transmission prefix="${prefix}"/> -->
-  </xacro:macro>
 </robot>

File: src/tidybot_description/urdf/tidybot.gazebo.xacro (robot description, xacro)
@@ -8,5 +8,4 @@
       </plugin>
       <plugin name="ignition::gazebo::systems::Sensors" filename="libignition-gazebo-sensors-system.so"/>
-      <!-- <self_collide>true</self_collide> -->
   </gazebo>
   <!-- <gazebo>

File: src/tidybot_description/urdf/tidybot.ros2_control.xacro (robot description, xacro)
@@ -36,10 +36,40 @@
         </xacro:if>
         <xacro:if value="${gripper == 'robotiq_2f_85'}">
-            <xacro:add_joint name="right_inner_finger_joint" gain="0.1" cmd_interface="position"/>
-            <xacro:add_joint name="right_outer_knuckle_joint" gain="0.1" cmd_interface="position"/>
-            <xacro:add_joint name="right_inner_knuckle_joint" gain="0.1" cmd_interface="position"/>
-            <xacro:add_joint name="left_inner_finger_joint" gain="0.1" cmd_interface="position"/>
-            <xacro:add_joint name="left_outer_knuckle_joint" gain="0.1" cmd_interface="position"/>
-            <xacro:add_joint name="left_inner_knuckle_joint" gain="0.1" cmd_interface="position"/>
+            <joint name ="left_outer_knuckle_joint">
+                <command_interface name="position"/>
+                <state_interface name="position"/>
+                <state_interface name="velocity"/>
+                <param name="position_proportional_gain">0.1</param>
+            </joint>
+            <joint name ="right_inner_finger_joint">
+                <param name="mimic">left_outer_knuckle_joint</param>
+                <param name="multiplier">-1.0</param>
+                <state_interface name="position"/>
+                <state_interface name="velocity"/>
+            </joint>
+            <joint name ="right_outer_knuckle_joint">
+                <param name="mimic">left_outer_knuckle_joint</param>
+                <param name="multiplier">1.0</param>
+                <state_interface name="position"/>
+                <state_interface name="velocity"/>
+            </joint>
+            <joint name ="right_inner_knuckle_joint">
+                <param name="mimic">left_outer_knuckle_joint</param>
+                <param name="multiplier">1.0</param>
+                <state_interface name="position"/>
+                <state_interface name="velocity"/>
+            </joint>
+            <joint name ="left_inner_finger_joint">
+                <param name="mimic">left_outer_knuckle_joint</param>
+                <param name="multiplier">-1.0</param>
+                <state_interface name="position"/>
+                <state_interface name="velocity"/>
+            </joint>
+            <joint name ="left_inner_knuckle_joint">
+                <param name="mimic">left_outer_knuckle_joint</param>
+                <param name="multiplier">1.0</param>
+                <state_interface name="position"/>
+                <state_interface name="velocity"/>
+            </joint>
         </xacro:if>
         </ros2_control>

File: src/tidybot_description/urdf/tidybot.urdf (robot description, URDF)
Before this commit: robot tidybot, 30 links, 29 joints
Links:
- added link finger_link
Joints:
- added joint finger_joint: type revolute, parent end_effector_link, child finger_link, origin xyz=0 0 0 rpy=0 0 0, axis 1 0 0, limit lower=0 upper=0.81 effort=1000 velocity=1.0
- joint left_inner_finger_joint: limit lower=-0.8757 upper=0.8757 effort=1000 velocity=2.0 -> lower=-1.0 upper=1.0 effort=1000 velocity=1.0; mimic (none) -> joint=left_outer_knuckle_joint multiplier=-1 offset=0
- joint left_inner_knuckle_joint: limit lower=-0.01 upper=0.8757 effort=1000 velocity=2.0 -> lower=-1.0 upper=1.0 effort=1000 velocity=1.0; mimic (none) -> joint=left_outer_knuckle_joint multiplier=1 offset=0
- joint left_outer_knuckle_joint: limit lower=-0.01 upper=0.8 effort=1000 velocity=2.0 -> lower=-1.0 upper=1.0 effort=1000 velocity=1.0
- joint right_inner_finger_joint: limit lower=-0.8757 upper=0.8757 effort=1000 velocity=2.0 -> lower=-1.0 upper=1.0 effort=1000 velocity=1.0; mimic (none) -> joint=left_outer_knuckle_joint multiplier=-1 offset=0
- joint right_inner_knuckle_joint: limit lower=-0.01 upper=0.8757 effort=1000 velocity=2.0 -> lower=-1.0 upper=1.0 effort=1000 velocity=1.0; mimic (none) -> joint=left_outer_knuckle_joint multiplier=1 offset=0
- joint right_outer_knuckle_joint: limit lower=-0.01 upper=0.81 effort=1000 velocity=2.0 -> lower=-1.0 upper=1.0 effort=1000 velocity=1.0; mimic (none) -> joint=left_outer_knuckle_joint multiplier=1 offset=0

Commit message: unified the gripper definition

File: src/tidybot_description/urdf/grippers/robotiq_2f_85/robotiq_2f_85_macro.xacro (robot description, xacro)
@@ -1,19 +1,27 @@
 <?xml version="1.0"?>
+<!--
+  Robotiq 2F-85 Gripper Loader
+  Unified gripper definition compatible with both Isaac Sim and Gazebo.
+  Uses Isaac Sim kinematic structure with closed-loop kinematics.
+-->
 <robot name="robotiq_arg2f_85_model" xmlns:xacro="http://ros.org/wiki/xacro">
   <xacro:macro name="load_gripper" params="parent prefix">
     <xacro:include filename="$(find tidybot_description)/urdf/grippers/robotiq_2f_85/robotiq_arg2f.xacro" />
     <xacro:include filename="$(find tidybot_description)/urdf/grippers/robotiq_2f_85/robotiq_arg2f_85_model_macro.xacro" />
+    <!-- Tool frame -->
     <link name="${prefix}tool_frame"/>
     <joint name="${prefix}tool_frame_joint" type="fixed">
-        <origin xyz="0 0 0.120" rpy="0 0 0" />
-        <parent link="${parent}" />
-        <child link="${prefix}tool_frame" />
-        <axis xyz="0 0 0" />
+      <origin xyz="0 0 0.120" rpy="0 0 0"/>
+      <parent link="${parent}"/>
+      <child link="${prefix}tool_frame"/>
+      <axis xyz="0 0 0"/>
     </joint>
-    <!-- Gripper description -->
+    <!-- Gripper base link -->
     <xacro:robotiq_arg2f_base_link prefix="${prefix}" parent="${parent}"/>
-    <xacro:finger_links prefix="${prefix}" fingerprefix="left" stroke="85"/>
-    <xacro:finger_links prefix="${prefix}" fingerprefix="right" stroke="85"/>
+    <!-- Left finger (reflect=1) -->
+    <xacro:finger_links prefix="${prefix}" fingerprefix="left" reflect="1"/>
     <xacro:left_outer_knuckle_joint prefix="${prefix}"/>
+    <!-- Right finger (reflect=-1) -->
+    <xacro:finger_links prefix="${prefix}" fingerprefix="right" reflect="-1"/>
     <xacro:right_outer_knuckle_joint prefix="${prefix}"/>
   </xacro:macro>

File: src/tidybot_description/urdf/grippers/robotiq_2f_85/robotiq_arg2f.xacro (robot description, xacro)
@@ -1,33 +1,40 @@
 <?xml version="1.0"?>
+<!--
+  Robotiq 2F-85 Gripper Base Link and Assembly Helpers
+  Uses Isaac Sim exported mesh and inertial properties for consistency
+  across both Isaac Sim and Gazebo simulators.
+-->
 <robot xmlns:xacro="http://ros.org/wiki/xacro">
+  <!-- Mesh directory -->
+  <xacro:property name="mesh_dir" value="file://$(find tidybot_description)/meshes/grippers/robotiq_2f_85"/>
+  <!-- Base link macro -->
   <xacro:macro name="robotiq_arg2f_base_link" params="parent prefix">
     <xacro:include filename="$(find tidybot_description)/urdf/grippers/robotiq_2f_85/robotiq_arg2f_85_model_macro.xacro" />
-    <!-- This joint was added by Kinova -->
+    <!-- Gripper base joint (added by Kinova) -->
     <joint name="${prefix}gripper_base_joint" type="fixed">
-        <parent link="${parent}"/>
-        <child link="${prefix}robotiq_arg2f_base_link"/>
-        <origin rpy="0.0 0.0 1.57" xyz="0.0 0.0 0.0"/>
+      <parent link="${parent}"/>
+      <child link="${prefix}robotiq_arg2f_base_link"/>
+      <origin rpy="0.0 0.0 1.57" xyz="0.0 0.0 0.0"/>
     </joint>
+    <!-- Base link with Isaac Sim inertial properties -->
     <link name="${prefix}robotiq_arg2f_base_link">
       <inertial>
-        <origin xyz="8.625E-08 -4.6583E-06 0.03145" rpy="0 0 0" />
-        <mass value="0.22652" />
-        <inertia ixx="0.00020005" ixy="-4.2442E-10" ixz="-2.9069E-10" iyy="0.00017832" iyz="-3.4402E-08" izz="0.00013478" />
+        <origin xyz="0.0000228 -0.0000006 0.0323229" rpy="0. 0. 0."/>
+        <mass value="0.6098911"/>
+        <inertia ixx="0.0005407" ixy="0." ixz="-0." iyy="0.0003629" iyz="-0." izz="0.0004747"/>
       </inertial>
       <visual>
-        <origin xyz="0 0 0" rpy="0 0 0" />
+        <origin xyz="0. 0. 0." rpy="${pi/2} 0. ${pi/2}"/>
         <geometry>
-          <!-- The DAE file doesn't show well in Gazebo so we're using the STL instead -->
-          <!-- <mesh filename="file://$(find simulation)/meshes/grippers/robotiq_2f_85/meshes/visual/robotiq_arg2f_85_base_link.dae" scale="0.001 0.001 0.001"/> -->
-          <mesh filename="file://$(find tidybot_description)/meshes/grippers/robotiq_2f_85/collision/robotiq_arg2f_base_link.stl" />
+          <mesh filename="${mesh_dir}/robotiq_arg2f_85_base_link.stl"/>
         </geometry>
         <material name="">
-          <color rgba="0.1 0.1 0.1 1" />
+          <color rgba="0.2 0.2 0.2 1.0"/>
         </material>
       </visual>
       <collision>
-        <origin xyz="0 0 0" rpy="0 0 0" />
+        <origin xyz="0. 0. 0." rpy="${pi/2} 0. ${pi/2}"/>
         <geometry>
-          <mesh filename="file://$(find tidybot_description)/meshes/grippers/robotiq_2f_85/collision/robotiq_arg2f_base_link.stl" />
+          <mesh filename="${mesh_dir}/robotiq_arg2f_85_base_link.stl"/>
         </geometry>
       </collision>
@@ -37,16 +44,3 @@
     </gazebo>
   </xacro:macro>
-  <xacro:macro name="finger_joints" params="prefix fingerprefix reflect">
-    <xacro:outer_finger_joint prefix="${prefix}" fingerprefix="${fingerprefix}"/>
-    <xacro:inner_knuckle_joint prefix="${prefix}" fingerprefix="${fingerprefix}" reflect="${reflect}"/>
-    <xacro:inner_finger_joint prefix="${prefix}" fingerprefix="${fingerprefix}"/>
-    <xacro:inner_finger_pad_joint prefix="${prefix}" fingerprefix="${fingerprefix}"/>
-  </xacro:macro>
-  <xacro:macro name="finger_links" params="prefix fingerprefix stroke">
-    <xacro:outer_knuckle prefix="${prefix}" fingerprefix="${fingerprefix}" stroke="${stroke}"/>
-    <xacro:outer_finger prefix="${prefix}" fingerprefix="${fingerprefix}" stroke="${stroke}"/>
-    <xacro:inner_finger prefix="${prefix}" fingerprefix="${fingerprefix}" stroke="${stroke}"/>
-    <xacro:inner_finger_pad prefix="${prefix}" fingerprefix="${fingerprefix}"/>
-    <xacro:inner_knuckle prefix="${prefix}" fingerprefix="${fingerprefix}" stroke="${stroke}"/>
-  </xacro:macro>
 </robot>
