Commit message: add real environment launch configuration

File: src/tidybot_description/urdf/grippers/robotiq_2f_85/robotiq_arg2f_85_model_macro.xacro (robot description, xacro)
@@ -138,5 +138,5 @@
       <axis xyz="1 0 0" />
       <limit lower="0" upper="0.8757" velocity="2.0" effort="1000" />
-      <!-- <mimic joint="${prefix}finger_joint" multiplier="1" offset="0" /> -->
+      <mimic joint="${prefix}finger_joint" multiplier="1" offset="0" />
     </joint>
     <transmission name="{prefix}${fingerprefix}_inner_knuckle_joint_trans">
@@ -155,5 +155,5 @@
       <axis xyz="1 0 0" />
       <limit lower="-0.8757" upper="0.8757" velocity="2.0" effort="1000" />
-      <!-- <mimic joint="${prefix}finger_joint" multiplier="-1" offset="0" /> -->
+      <mimic joint="${prefix}finger_joint" multiplier="-1" offset="0" />
     </joint>
     <transmission name="${prefix}${fingerprefix}_inner_finger_joint_trans">
@@ -198,5 +198,5 @@
       <axis xyz="1 0 0" />
       <limit lower="0" upper="0.81" velocity="2.0" effort="1000" />
-      <!-- <mimic joint="${prefix}finger_joint" multiplier="1" offset="0" /> -->
+      <mimic joint="${prefix}finger_joint" multiplier="1" offset="0" />
     </joint>
     <transmission name="$${prefix}right_outer_knuckle_joint_trans">

File: src/tidybot_description/urdf/tidybot.xacro (robot description, xacro)
@@ -4,5 +4,5 @@
     <xacro:arg name="hardware_plugin" default="gz_ros2_control/GazeboSimSystem" />
     <xacro:arg name="arm" default="gen3_7dof" />
-    <xacro:arg name="gripper" default="gen3_lite_2f" />
+    <xacro:arg name="gripper" default="robotiq_2f_85" />
     <xacro:arg name="vision" default="true" />
     <xacro:arg name="prefix" default="" />

Commit message: add gripper joint_trajectory recorder

File: src/tidybot_description/urdf/grippers/robotiq_2f_85/robotiq_arg2f_85_model_macro.xacro (robot description, xacro)
@@ -137,14 +137,7 @@
       <child link="${prefix}${fingerprefix}_inner_knuckle" />
       <axis xyz="1 0 0" />
-      <limit lower="0" upper="0.8757" velocity="2.0" effort="1000" />
+      <limit lower="-0.01" upper="0.8757" velocity="2.0" effort="1000" />
       <!-- <mimic joint="${prefix}finger_joint" multiplier="1" offset="0" /> -->
     </joint>
-    <transmission name="${prefix}${fingerprefix}_inner_knuckle_joint_trans">
-      <type>transmission_interface/SimpleTransmission</type>
-      <joint name="${prefix}${fingerprefix}_inner_knuckle_joint" />
-      <actuator name="${prefix}${fingerprefix}_inner_knuckle_joint_motor">
-          <mechanicalReduction>1</mechanicalReduction>
-      </actuator>
-    </transmission>
   </xacro:macro>
   <xacro:macro name="inner_finger_joint" params="prefix fingerprefix">
@@ -157,11 +150,4 @@
       <!-- <mimic joint="${prefix}finger_joint" multiplier="-1" offset="0" /> -->
     </joint>
-    <transmission name="${prefix}${fingerprefix}_inner_finger_joint_trans">
-      <type>transmission_interface/SimpleTransmission</type>
-      <joint name="${prefix}${fingerprefix}_inner_finger_joint" />
-      <actuator name="${prefix}${fingerprefix}_inner_finger_joint_motor">
-          <mechanicalReduction>1</mechanicalReduction>
-      </actuator>
-    </transmission>
   </xacro:macro>
   <xacro:macro name="inner_finger_pad_joint" params="prefix fingerprefix">
@@ -174,19 +160,12 @@
   </xacro:macro>
   <xacro:include filename="$(find tidybot_description)/urdf/grippers/robotiq_2f_85/robotiq_arg2f.xacro" />
-  <xacro:macro name="finger_joint" params="prefix">
-    <joint name="${prefix}finger_joint" type="revolute">
+  <xacro:macro name="left_outer_knuckle_joint" params="prefix">
+    <joint name="${prefix}left_outer_knuckle_joint" type="revolute">
       <origin xyz="0 -0.0306011 0.054904" rpy="0 0 ${pi}"/>
       <parent link="${prefix}robotiq_arg2f_base_link" />
       <child link="${prefix}left_outer_knuckle" />
       <axis xyz="1 0 0" />
-      <limit lower="0" upper="0.8" velocity="2.0" effort="1000" />
-    </joint>
-    <transmission name="${prefix}finger_joint_trans">
-      <type>transmission_interface/SimpleTransmission</type>
-      <joint name="${prefix}finger_joint" />
-      <actuator name="${prefix}finger_joint_motor">
-          <mechanicalReduction>1</mechanicalReduction>
-      </actuator>
-    </transmission>
+      <limit lower="-0.01" upper="0.8" velocity="2.0" effort="1000" />
+    </joint>
     <xacro:finger_joints prefix="${prefix}" fingerprefix="left" reflect="1.0"/>
   </xacro:macro>
@@ -197,14 +176,7 @@
       <child link="${prefix}right_outer_knuckle" />
       <axis xyz="1 0 0" />
-      <limit lower="0" upper="0.81" velocity="2.0" effort="1000" />
+      <limit lower="-0.01" upper="0.81" velocity="2.0" effort="1000" />
       <!-- <mimic joint="${prefix}finger_joint" multiplier="1" offset="0" /> -->
     </joint>
-    <transmission name="${prefix}right_outer_knuckle_joint_trans">
-      <type>transmission_interface/SimpleTransmission</type>
-      <joint name="${prefix}right_outer_knuckle_joint" />
-      <actuator name="${prefix}right_outer_knuckle_joint_motor">
-          <mechanicalReduction>1</mechanicalReduction>
-      </actuator>
-    </transmission>
     <xacro:finger_joints prefix="${prefix}" fingerprefix="right" reflect="-1.0"/>
   </xacro:macro>
@@ -223,5 +195,5 @@
     <xacro:finger_links prefix="${prefix}" fingerprefix="left" stroke="85"/>
     <xacro:finger_links prefix="${prefix}" fingerprefix="right" stroke="85"/>
-    <xacro:finger_joint prefix="${prefix}"/>
+    <xacro:left_outer_knuckle_joint prefix="${prefix}"/>
     <xacro:right_outer_knuckle_joint prefix="${prefix}"/>
     <!-- Transmissions are loaded in the generic kortex xacro when simulation is enabled -->

File: src/tidybot_description/urdf/tidybot.gazebo.xacro (robot description, xacro)
@@ -52,4 +52,6 @@
   <xacro:include filename="$(find tidybot_description)/urdf/base/base_transmission.xacro" />
   <xacro:load_base_transmission prefix="${prefix}" />
+  <xacro:include filename="$(find tidybot_description)/urdf/grippers/robotiq_2f_85/robotiq_2f_85_transmission.xacro" />
+  <xacro:load_gripper_transmission prefix="${prefix}" />
 </xacro:macro>
 </robot>

File: src/tidybot_description/urdf/tidybot.ros2_control.xacro (robot description, xacro)
@@ -39,7 +39,7 @@
             <xacro:add_joint name="right_outer_knuckle_joint" gain="0.1" cmd_interface="position"/>
             <xacro:add_joint name="right_inner_knuckle_joint" gain="0.1" cmd_interface="position"/>
-            <!-- <xacro:add_joint name="left_inner_finger_joint" gain="0.1" cmd_interface="position"/>
+            <xacro:add_joint name="left_inner_finger_joint" gain="0.1" cmd_interface="position"/>
             <xacro:add_joint name="left_outer_knuckle_joint" gain="0.1" cmd_interface="position"/>
-            <xacro:add_joint name="left_inner_knuckle_joint" gain="0.1" cmd_interface="position"/> -->
+            <xacro:add_joint name="left_inner_knuckle_joint" gain="0.1" cmd_interface="position"/>
         </xacro:if>
         </ros2_control>

File: src/tidybot_description/urdf/tidybot.urdf (robot description, URDF)
Before this commit: robot tidybot, 29 links, 28 joints
Links:
- link left_inner_finger: geometry visual mesh filename=file:///home/yuandi/tidybot_platform/install/tidybot_descri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 scale=0.001 0.001 0.001
- link left_inner_finger_pad: geometry visual box size=0.022 0.00635 0.0375
- link left_inner_knuckle: geometry visual mesh filename=file:///home/yuandi/tidybot_platform/install/tidybot_descri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 scale=0.001 0.001 0.001
- link left_outer_finger: geometry visual mesh filename=file:///home/yuandi/tidybot_platform/install/tidybot_descri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 scale=0.001 0.001 0.001
- link left_outer_knuckle: geometry visual mesh filename=file:///home/yuandi/tidybot_platform/install/tidybot_descri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 scale=0.001 0.001 0.001
- link right_inner_finger: geometry visual mesh filename=file:///home/yuandi/tidybot_platform/install/tidybot_descri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 scale=0.001 0.001 0.001
- link right_inner_finger_pad: geometry visual box size=0.022 0.00635 0.0375
- link right_inner_knuckle: geometry visual mesh filename=file:///home/yuandi/tidybot_platform/install/tidybot_descri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 scale=0.001 0.001 0.001
- link right_outer_finger: geometry visual mesh filename=file:///home/yuandi/tidybot_platform/install/tidybot_descri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 scale=0.001 0.001 0.001
- link right_outer_knuckle: geometry visual mesh filename=file:///home/yuandi/tidybot_platform/install/tidybot_descri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 scale=0.001 0.001 0.001
Joints:
- removed joint finger_joint
- added joint left_outer_knuckle_joint: type revolute, parent robotiq_arg2f_base_link, child left_outer_knuckle, origin xyz=0 -0.0306011 0.054904 rpy=0 0 3.141592653589793, axis 1 0 0, limit lower=0 upper=0.8 effort=1000 velocity=2.0

Commit message: change the gripper controller to position_controllers/JointGroupPositionController

File: src/tidybot_description/urdf/grippers/robotiq_2f_85/robotiq_arg2f_85_model_macro.xacro (robot description, xacro)
@@ -137,5 +137,5 @@
       <child link="${prefix}${fingerprefix}_inner_knuckle" />
       <axis xyz="1 0 0" />
-      <limit lower="-0.01" upper="0.8757" velocity="2.0" effort="1000" />
+      <limit lower="-1.0" upper="1.0" velocity="1.0" effort="1000" />
       <!-- <mimic joint="${prefix}finger_joint" multiplier="1" offset="0" /> -->
     </joint>
@@ -147,5 +147,5 @@
       <child link="${prefix}${fingerprefix}_inner_finger" />
       <axis xyz="1 0 0" />
-      <limit lower="-0.8757" upper="0.8757" velocity="2.0" effort="1000" />
+      <limit lower="-1.0" upper="1.0" velocity="1.0" effort="1000" />
       <!-- <mimic joint="${prefix}finger_joint" multiplier="-1" offset="0" /> -->
     </joint>
@@ -166,5 +166,5 @@
       <child link="${prefix}left_outer_knuckle" />
       <axis xyz="1 0 0" />
-      <limit lower="-0.01" upper="0.8" velocity="2.0" effort="1000" />
+      <limit lower="-1.0" upper="1.0" velocity="1.0" effort="1000" />
     </joint>
     <xacro:finger_joints prefix="${prefix}" fingerprefix="left" reflect="1.0"/>
@@ -176,5 +176,5 @@
       <child link="${prefix}right_outer_knuckle" />
       <axis xyz="1 0 0" />
-      <limit lower="-0.01" upper="0.81" velocity="2.0" effort="1000" />
+      <limit lower="-1.0" upper="1.0" velocity="1.0" effort="1000" />
       <!-- <mimic joint="${prefix}finger_joint" multiplier="1" offset="0" /> -->
     </joint>

File: src/tidybot_description/urdf/tidybot.urdf (robot description, URDF)
Before this commit: robot tidybot, 29 links, 28 joints
Links:
- removed link camera_link
- added link arm_camera_link
- added link base_camera_link
- link arm_base_link: geometry collision mesh filename=file:///home/janchen/Documents/tidybot_platform/install/tid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; visual mesh filename=file:///home/janchen/Documents/tidybot_platform/install/tid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
- link base: mass 60.0 -> 34; geometry collision mesh filename=file:///home/janchen/Documents/tidybot_platform/install/tid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; visual mesh filename=file:///home/janchen/Documents/tidybot_platform/install/tid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
- link bracelet_link: geometry collision mesh filename=file:///home/janchen/Documents/tidybot_platform/install/tid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; visual mesh filename=file:///home/janchen/Documents/tidybot_platform/install/tid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
- link forearm_link: geometry collision mesh filename=file:///home/janchen/Documents/tidybot_platform/install/tid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; visual mesh filename=file:///home/janchen/Documents/tidybot_platform/install/tid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
- link half_arm_1_link: geometry collision mesh filename=file:///home/janchen/Documents/tidybot_platform/install/tid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; visual mesh filename=file:///home/janchen/Documents/tidybot_platform/install/tid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
- link half_arm_2_link: geometry collision mesh filename=file:///home/janchen/Documents/tidybot_platform/install/tid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; visual mesh filename=file:///home/janchen/Documents/tidybot_platform/install/tid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
- link left_inner_finger: geometry collision mesh filename=file:///home/janchen/Documents/tidybot_platform/install/tid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 scale=0.001 0.001 0.001; visual mesh filename=file:///home/janchen/Documents/tidybot_platform/install/tid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 scale=0.001 0.001 0.001
- link left_inner_finger_pad: geometry collision box size=0.022 0.00635 0.0375; visual box size=0.022 0.00635 0.0375
- link left_inner_knuckle: geometry collision mesh filename=file:///home/janchen/Documents/tidybot_platform/install/tid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 scale=0.001 0.001 0.001; visual mesh filename=file:///home/janchen/Documents/tidybot_platform/install/tid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 scale=0.001 0.001 0.001
- link left_outer_finger: geometry collision mesh filename=file:///home/janchen/Documents/tidybot_platform/install/tid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 scale=0.001 0.001 0.001; visual mesh filename=file:///home/janchen/Documents/tidybot_platform/install/tid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 scale=0.001 0.001 0.001
- link left_outer_knuckle: geometry collision mesh filename=file:///home/janchen/Documents/tidybot_platform/install/tid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 scale=0.001 0.001 0.001; visual mesh filename=file:///home/janchen/Documents/tidybot_platform/install/tid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 scale=0.001 0.001 0.001
- link right_inner_finger: geometry collision mesh filename=file:///home/janchen/Documents/tidybot_platform/install/tid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 scale=0.001 0.001 0.001; visual mesh filename=file:///home/janchen/Documents/tidybot_platform/install/tid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 scale=0.001 0.001 0.001
- link right_inner_finger_pad: geometry collision box size=0.022 0.00635 0.0375; visual box size=0.022 0.00635 0.0375
- link right_inner_knuckle: geometry collision mesh filename=file:///home/janchen/Documents/tidybot_platform/install/tid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 scale=0.001 0.001 0.001; visual mesh filename=file:///home/janchen/Documents/tidybot_platform/install/tid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 scale=0.001 0.001 0.001
- link right_outer_finger: geometry collision mesh filename=file:///home/janchen/Documents/tidybot_platform/install/tid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 scale=0.001 0.001 0.001; visual mesh filename=file:///home/janchen/Documents/tidybot_platform/install/tid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 scale=0.001 0.001 0.001
- link right_outer_knuckle: geometry collision mesh filename=file:///home/janchen/Documents/tidybot_platform/install/tid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 scale=0.001 0.001 0.001; visual mesh filename=file:///home/janchen/Documents/tidybot_platform/install/tid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 scale=0.001 0.001 0.001
- link robotiq_arg2f_base_link: geometry collision mesh filename=file:///home/janchen/Documents/tidybot_platform/install/tid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; visual mesh filename=file:///home/janchen/Documents/tidybot_platform/install/tid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
- link shoulder_link: geometry collision mesh filename=file:///home/janchen/Documents/tidybot_platform/install/tid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; visual mesh filename=file:///home/janchen/Documents/tidybot_platform/install/tid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
- link spherical_wrist_1_link: geometry collision mesh filename=file:///home/janchen/Documents/tidybot_platform/install/tid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; visual mesh filename=file:///home/janchen/Documents/tidybot_platform/install/tid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
- link spherical_wrist_2_link: geometry collision mesh filename=file:///home/janchen/Documents/tidybot_platform/install/tid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; visual mesh filename=file:///home/janchen/Documents/tidybot_platform/install/tid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
Joints:
- added joint base_camera_joint: type fixed, parent base, child base_camera_link, origin xyz=0.2525 0.0 0.315 rpy=0 0.7853981634 0
- joint arm_base_joint: origin xyz=0 0 0.33 rpy=0 0 0 -> xyz=0.12 3.76986e-15 0.374775 rpy=0 0 0
- joint camera_module: child camera_link -> arm_camera_link
- joint left_inner_knuckle_joint: limit lower=0 upper=0.8757 effort=1000 velocity=2.0 -> lower=-0.01 upper=0.8757 effort=1000 velocity=2.0
- joint left_outer_knuckle_joint: limit lower=0 upper=0.8 effort=1000 velocity=2.0 -> lower=-0.01 upper=0.8 effort=1000 velocity=2.0
- joint right_inner_knuckle_joint: limit lower=0 upper=0.8757 effort=1000 velocity=2.0 -> lower=-0.01 upper=0.8757 effort=1000 velocity=2.0
- joint right_outer_knuckle_joint: limit lower=0 upper=0.81 effort=1000 velocity=2.0 -> lower=-0.01 upper=0.81 effort=1000 velocity=2.0

File: src/tidybot_moveit_config/config/tidybot.ros2_control.xacro (robot description, xacro)
@@ -57,32 +57,4 @@
                 <state_interface name="velocity"/>
             </joint>
-            <joint name="left_finger_bottom_joint">
-                <command_interface name="position"/>
-                <state_interface name="position">
-                  <param name="initial_value">${initial_positions['left_finger_bottom_joint']}</param>
-                </state_interface>
-                <state_interface name="velocity"/>
-            </joint>
-            <joint name="left_finger_tip_joint">
-                <command_interface name="position"/>
-                <state_interface name="position">
-                  <param name="initial_value">${initial_positions['left_finger_tip_joint']}</param>
-                </state_interface>
-                <state_interface name="velocity"/>
-            </joint>
-            <joint name="right_finger_bottom_joint">
-                <command_interface name="position"/>
-                <state_interface name="position">
-                  <param name="initial_value">${initial_positions['right_finger_bottom_joint']}</param>
-                </state_interface>
-                <state_interface name="velocity"/>
-            </joint>
-            <joint name="right_finger_tip_joint">
-                <command_interface name="position"/>
-                <state_interface name="position">
-                  <param name="initial_value">${initial_positions['right_finger_tip_joint']}</param>
-                </state_interface>
-                <state_interface name="velocity"/>
-            </joint>
         </ros2_control>
     </xacro:macro>
