Commit message: added multi-stage-planner and drawer policy; refactored robot control logic in Gazebo

File: src/tidybot_description/urdf/grippers/robotiq_2f_85/robotiq_arg2f_85_model_macro.xacro (robot description, xacro)
@@ -84,10 +84,11 @@
         </material>
       </visual>
-      <collision>
+      <!-- Collision disabled (Kinematic Inversion Fix) -->
+      <!-- <collision>
         <origin xyz="-0.0292492 0.0556365 0." rpy="0. 0. 3.1171339"/>
         <geometry>
           <mesh filename="${mesh_dir}/robotiq_arg2f_85_outer_knuckle.stl"/>
         </geometry>
-      </collision>
+      </collision> -->
     </link>
     <gazebo reference="${prefix}right_outer_knuckle">
@@ -140,10 +141,11 @@
         </material>
       </visual>
-      <collision>
+      <!-- Collision disabled (Kinematic Inversion Fix) -->
+      <!-- <collision>
         <origin xyz="0.062026 0.0503723 0." rpy="3.1415927 0. 0."/>
         <geometry>
           <mesh filename="${mesh_dir}/robotiq_arg2f_85_outer_finger.stl"/>
         </geometry>
-      </collision>
+      </collision> -->
     </link>
     <gazebo reference="${prefix}right_outer_finger">
@@ -224,5 +226,6 @@
         </material>
       </visual>
-      <collision>
+      <!-- Collision disabled (Kinematic Inversion Fix) -->
+      <!-- <collision>
         <origin xyz="0.071171 -0.0956936 -0.0133" rpy="0. 0. 0.0244594"/>
         <geometry>
@@ -235,5 +238,5 @@
           <mesh filename="${mesh_dir}/robotiq_arg2f_85_pad.stl"/>
         </geometry>
-      </collision>
+      </collision> -->
     </link>
     <gazebo reference="${prefix}right_inner_finger">
@@ -286,10 +289,11 @@
         </material>
       </visual>
-      <collision>
+      <!-- Collision disabled (Kinematic Inversion Fix) -->
+      <!-- <collision>
         <origin xyz="0.0483511 -0.1051343 0." rpy="0. 0. -0.0244597"/>
         <geometry>
           <mesh filename="${mesh_dir}/robotiq_arg2f_85_inner_knuckle.stl"/>
         </geometry>
-      </collision>
+      </collision> -->
     </link>
     <gazebo reference="${prefix}right_inner_knuckle">
@@ -353,7 +357,6 @@
       <parent link="${prefix}robotiq_arg2f_base_link"/>
       <child link="${prefix}right_outer_knuckle"/>
-      <axis xyz="0. 0. -1."/>
-      <limit lower="0." upper="0.8203047" effort="26." velocity="174.5329252"/>
-      <mimic joint="${prefix}finger_joint" multiplier="1.0" offset="0"/>
+      <axis xyz="0. 0. 1."/>
+      <limit lower="-0.8203047" upper="0.8203047" effort="26." velocity="2.5562093"/>
       <dynamics damping="1.0" friction="0.5"/>
     </joint>
@@ -367,5 +370,5 @@
       <axis xyz="0 0 1"/>
       <limit lower="0.0" upper="0.0" effort="100" velocity="100"/>
-      <mimic joint="${prefix}finger_joint" multiplier="0.0" offset="0"/>
+      <mimic joint="${prefix}right_outer_knuckle_joint" multiplier="0.0" offset="0"/>
       <dynamics damping="10.0" friction="10.0"/>
     </joint>
@@ -379,5 +382,5 @@
       <axis xyz="0. 0. 1."/>
       <limit lower="-3.1415927" upper="3.1415927" effort="26." velocity="174.5329252"/>
-      <mimic joint="${prefix}finger_joint" multiplier="1.0" offset="0"/>
+      <mimic joint="${prefix}right_outer_knuckle_joint" multiplier="-1.0" offset="0"/>
       <dynamics damping="1.0" friction="0.5"/>
     </joint>
@@ -391,5 +394,5 @@
       <axis xyz="0. 0. 1."/>
       <limit lower="-3.1415927" upper="3.1415927" effort="26." velocity="174.5329252"/>
-      <mimic joint="${prefix}finger_joint" multiplier="-1.0" offset="0"/>
+      <mimic joint="${prefix}right_outer_knuckle_joint" multiplier="1.0" offset="0"/>
       <dynamics damping="1.0" friction="0.5"/>
     </joint>

File: src/tidybot_description/urdf/tidybot.gazebo.xacro (robot description, xacro)
@@ -1,83 +1,81 @@
 <?xml version="1.0"?>
 <robot xmlns:xacro="http://ros.org/wiki/xacro">
-<xacro:macro name="load_gazebo_plugins" params="config_path prefix arm vision">
-  <gazebo>
+  <xacro:macro name="load_gazebo_plugins" params="config_path prefix arm vision">
+    <gazebo>
       <plugin name="gz_ros2_control::GazeboSimROS2ControlPlugin" filename="gz_ros2_control-system">
-          <parameters>${config_path}</parameters>
-          <robot_description_param>robot_description</robot_description_param>
+        <parameters>${config_path}</parameters>
+        <robot_description_param>robot_description</robot_description_param>
       </plugin>
       <plugin name="ignition::gazebo::systems::Sensors" filename="libignition-gazebo-sensors-system.so"/>
-  </gazebo>
-  <!-- <gazebo>
+    </gazebo>
+    <!-- <gazebo>
     <plugin filename="ignition-gazebo-joint-state-publisher-system" name="ignition::gazebo::systems::JointStatePublisher"/>
-    <plugin
-        filename="ignition-gazebo-pose-publisher-system"
-        name="ignition::gazebo::systems::PosePublisher">
+    <plugin filename="ignition-gazebo-pose-publisher-system" name="ignition::gazebo::systems::PosePublisher">
         <publish_link_pose>true</publish_link_pose>
         <use_pose_vector_msg>true</use_pose_vector_msg>
     </plugin>
   </gazebo> -->
-  <xacro:if value="${vision}">
-    <gazebo reference="${prefix}arm_camera_link">
-      <sensor name="${prefix}arm_camera" type="rgbd_camera">
-        <always_on>1</always_on>
-        <update_rate>30</update_rate>
-        <visualize>true</visualize>
-        <pose>0 -0.01 0.03 0 4.7124 1.5708</pose>
-				<topic>/arm_camera</topic>
-        <gz_frame_id>${prefix}arm_camera_link</gz_frame_id>
-        <camera>
-          <horizontal_fov>1.247</horizontal_fov>
-          <image>
-            <width>640</width>
-            <height>480</height>
-            <format>R8G8B8</format>
-          </image>
-          <clip>
-            <near>0.03</near>
-            <far>3.0</far>
-          </clip>
-          <noise>
-            <type>gaussian</type>
-            <mean>0.0</mean>
-            <stddev>0.007</stddev>
-          </noise>
-        </camera>
-      </sensor>
-    </gazebo>
-    <gazebo reference="${prefix}base_camera_link">
-      <sensor name="${prefix}base_camera" type="rgbd_camera">
-        <always_on>1</always_on>
-        <update_rate>30</update_rate>
-        <visualize>true</visualize>
-        <pose>0 0 0 0 0 0</pose>
-				<topic>/base_camera</topic>
-        <gz_frame_id>${prefix}base_camera_link</gz_frame_id>
-        <camera>
-          <horizontal_fov>1.434</horizontal_fov>
-          <image>
-            <width>640</width>
-            <height>360</height>
-            <format>R8G8B8</format>
-          </image>
-          <clip>
-            <near>0.03</near>
-            <far>3.0</far>
-          </clip>
-          <noise>
-            <type>gaussian</type>
-            <mean>0.0</mean>
-            <stddev>0.007</stddev>
-          </noise>
-        </camera>
-      </sensor>
-    </gazebo>
-  </xacro:if>
-  <xacro:include filename="$(find tidybot_description)/urdf/arms/${arm}/${arm}_transmission.xacro" />
-  <xacro:load_arm_transmission prefix="${prefix}" />
-  <xacro:include filename="$(find tidybot_description)/urdf/base/tidybot++/base_kinova_transmission.xacro" />
-  <xacro:load_base_transmission prefix="${prefix}" />
-  <xacro:include filename="$(find tidybot_description)/urdf/grippers/robotiq_2f_85/robotiq_2f_85_transmission.xacro" />
-  <xacro:load_gripper_transmission prefix="${prefix}" />
-</xacro:macro>
+    <xacro:if value="${vision}">
+      <gazebo reference="${prefix}arm_camera_link">
+        <sensor name="${prefix}arm_camera" type="rgbd_camera">
+          <always_on>1</always_on>
+          <update_rate>30</update_rate>
+          <visualize>true</visualize>
+          <pose>0 -0.01 0.03 0 4.7124 1.5708</pose>
+          <topic>/arm_camera</topic>
+          <gz_frame_id>${prefix}arm_camera_link</gz_frame_id>
+          <camera>
+            <horizontal_fov>1.247</horizontal_fov>
+            <image>
+              <width>640</width>
+              <height>480</height>
+              <format>R8G8B8</format>
+            </image>
+            <clip>
+              <near>0.03</near>
+              <far>3.0</far>
+            </clip>
+            <noise>
+              <type>gaussian</type>
+              <mean>0.0</mean>
+              <stddev>0.007</stddev>
+            </noise>
+          </camera>
+        </sensor>
+      </gazebo>
+      <gazebo reference="${prefix}base_camera_link">
+        <sensor name="${prefix}base_camera" type="rgbd_camera">
+          <always_on>1</always_on>
+          <update_rate>30</update_rate>
+          <visualize>true</visualize>
+          <pose>0 0 0 0 0 0</pose>
+          <topic>/base_camera</topic>
+          <gz_frame_id>${prefix}base_camera_link</gz_frame_id>
+          <camera>
+            <horizontal_fov>1.434</horizontal_fov>
+            <image>
+              <width>640</width>
+              <height>360</height>
+              <format>R8G8B8</format>
+            </image>
+            <clip>
+              <near>0.03</near>
+              <far>3.0</far>
+            </clip>
+            <noise>
+              <type>gaussian</type>
+              <mean>0.0</mean>
+              <stddev>0.007</stddev>
+            </noise>
+          </camera>
+        </sensor>
+      </gazebo>
+    </xacro:if>
+    <xacro:include filename="$(find tidybot_description)/urdf/arms/${arm}/${arm}_transmission.xacro" />
+    <xacro:load_arm_transmission prefix="${prefix}" />
+    <xacro:include filename="$(find tidybot_description)/urdf/base/tidybot++/base_kinova_transmission.xacro" />
+    <xacro:load_base_transmission prefix="${prefix}" />
+    <xacro:include filename="$(find tidybot_description)/urdf/grippers/robotiq_2f_85/robotiq_2f_85_transmission.xacro" />
+    <xacro:load_gripper_transmission prefix="${prefix}" />
+  </xacro:macro>
 </robot>

File: src/tidybot_description/urdf/tidybot.ros2_control.xacro (robot description, xacro)
@@ -50,7 +50,7 @@
                 </joint>
                 <!-- Right outer knuckle (mimic, same numeric value for symmetric closing) -->
+                <!-- Right driver joint (formerly right_outer_knuckle_joint) -->
                 <joint name="right_outer_knuckle_joint">
-                    <param name="mimic">finger_joint</param>
-                    <param name="multiplier">1.0</param>
+                    <command_interface name="position"/>
                     <state_interface name="position">
                         <param name="initial_value">0.0</param>
@@ -69,5 +69,5 @@
                 <!-- Right inner finger (mimic) -->
                 <joint name="right_inner_finger_joint">
-                    <param name="mimic">finger_joint</param>
+                    <param name="mimic">right_outer_knuckle_joint</param>
                     <param name="multiplier">1.0</param>
                     <state_interface name="position">
@@ -87,5 +87,5 @@
                 <!-- Right inner finger knuckle (mimic, connects inner finger to inner knuckle) -->
                 <joint name="right_inner_finger_knuckle_joint">
-                    <param name="mimic">finger_joint</param>
+                    <param name="mimic">right_outer_knuckle_joint</param>
                     <param name="multiplier">-1.0</param>
                     <state_interface name="position">
