Commit message: update base urdf model

File: src/tidybot_description/urdf/arms/gen3_7dof/gen3_7dof_macro.xacro (robot description, xacro)
@@ -5,5 +5,5 @@
   <xacro:macro name="load_arm" params="parent:='' vision prefix *origin">
     <joint name="${prefix}arm_base_joint" type="fixed">
-      <origin xyz="0 0 0.33" rpy="0 0 0" />
+      <origin xyz="0.12 3.76986e-15 0.374775" rpy="0 0 0" />
       <parent link="${parent}" />
       <child link="${prefix}arm_base_link" />

File: src/tidybot_description/urdf/base/tidybot/base_macro.xacro (robot description, xacro)
@@ -13,5 +13,5 @@
                 <origin xyz="-1.3915598211675165e-07 -2.058962502098711e-07 0.05386474576457055" rpy="-2.442021632452952 -1.5707963267948966 0.0"/>
                 <geometry>
-                    <mesh filename="file://$(find tidybot_description)/meshes/base/bumper.stl"/>
+                    <mesh filename="file://$(find tidybot_description)/meshes/base/tidybot/bumper.stl"/>
                 </geometry>
                 <material name="white"/>
@@ -20,5 +20,5 @@
                 <origin xyz="-1.3915598211675165e-07 -2.058962502098711e-07 0.05386474576457055" rpy="-2.442021632452952 -1.5707963267948966 0.0"/>
                 <geometry>
-                    <mesh filename="file://$(find tidybot_description)/meshes/base/bumper.stl"/>
+                    <mesh filename="file://$(find tidybot_description)/meshes/base/tidybot/bumper.stl"/>
                 </geometry>
             </collision>
@@ -26,5 +26,5 @@
                 <origin xyz="4.155854111430312e-11 1.8201972332496634e-11 0.08495000004768373" rpy="1.6659662035857206 -1.5707963267948966 0.0"/>
                 <geometry>
-                    <mesh filename="file://$(find tidybot_description)/meshes/base/bottom_plate.stl"/>
+                    <mesh filename="file://$(find tidybot_description)/meshes/base/tidybot/bottom_plate.stl"/>
                 </geometry>
                 <material name="white"/>
@@ -33,5 +33,5 @@
                 <origin xyz="4.155854111430312e-11 1.8201972332496634e-11 0.08495000004768373" rpy="1.6659662035857206 -1.5707963267948966 0.0"/>
                 <geometry>
-                    <mesh filename="file://$(find tidybot_description)/meshes/base/bottom_plate.stl"/>
+                    <mesh filename="file://$(find tidybot_description)/meshes/base/tidybot/bottom_plate.stl"/>
                 </geometry>
             </collision>
@@ -39,5 +39,5 @@
                 <origin xyz="7.590768644441668e-06 -6.000635064190085e-10 0.20330222068596052" rpy="-1.5707963267948966 -1.570779305272103 3.141592653589793"/>
                 <geometry>
-                    <mesh filename="file://$(find tidybot_description)/meshes/base/body.stl"/>
+                    <mesh filename="file://$(find tidybot_description)/meshes/base/tidybot/body.stl"/>
                 </geometry>
                 <material name="white"/>
@@ -46,5 +46,5 @@
                 <origin xyz="7.590768644441668e-06 -6.000635064190085e-10 0.20330222068596052" rpy="-1.5707963267948966 -1.570779305272103 3.141592653589793"/>
                 <geometry>
-                    <mesh filename="file://$(find tidybot_description)/meshes/base/body.stl"/>
+                    <mesh filename="file://$(find tidybot_description)/meshes/base/tidybot/body.stl"/>
                 </geometry>
             </collision>
@@ -52,5 +52,5 @@
                 <origin xyz="-2.9658670629084936e-11 -3.476524862019053e-11 0.3216499984264373" rpy="1.6906681075416252 -1.5707963267948966 0.0"/>
                 <geometry>
-                    <mesh filename="file://$(find tidybot_description)/meshes/base/top_plate.stl"/>
+                    <mesh filename="file://$(find tidybot_description)/meshes/base/tidybot/top_plate.stl"/>
                 </geometry>
                 <material name="white"/>
@@ -59,5 +59,5 @@
                 <origin xyz="-2.9658670629084936e-11 -3.476524862019053e-11 0.3216499984264373" rpy="1.6906681075416252 -1.5707963267948966 0.0"/>
                 <geometry>
-                    <mesh filename="file://$(find tidybot_description)/meshes/base/top_plate.stl"/>
+                    <mesh filename="file://$(find tidybot_description)/meshes/base/tidybot/top_plate.stl"/>
                 </geometry>
             </collision>
@@ -65,5 +65,5 @@
                 <origin xyz="-2.7580994002430455e-12 -3.3382504263355704e-12 0.32999999883475684" rpy="1.5707963267948966 -1.5707963267948966 0.0"/>
                 <geometry>
-                    <mesh filename="file://$(find tidybot_description)/meshes/base/arm_plate.stl"/>
+                    <mesh filename="file://$(find tidybot_description)/meshes/base/tidybot/arm_plate.stl"/>
                 </geometry>
                 <material name="white"/>
@@ -72,5 +72,5 @@
                 <origin xyz="-2.7580994002430455e-12 -3.3382504263355704e-12 0.32999999883475684" rpy="1.5707963267948966 -1.5707963267948966 0.0"/>
                 <geometry>
-                    <mesh filename="file://$(find tidybot_description)/meshes/base/arm_plate.stl"/>
+                    <mesh filename="file://$(find tidybot_description)/meshes/base/tidybot/arm_plate.stl"/>
                 </geometry>
             </collision>

File: src/tidybot_description/urdf/bot.xacro (robot description, xacro)
@@ -5,5 +5,5 @@
     <xacro:include filename="$(find tidybot_description)/urdf/arms/${arm}/${arm}_macro.xacro" />
     <xacro:include filename="$(find tidybot_description)/urdf/grippers/${gripper}/${gripper}_macro.xacro" />
-    <xacro:include filename="$(find tidybot_description)/urdf/base/base_macro.xacro" />
+    <xacro:include filename="$(find tidybot_description)/urdf/base/tidybot++/base_kinova_macro.xacro" />
     <!-- load the base -->
     <xacro:load_base parent="" prefix="${prefix}" />

File: src/tidybot_description/urdf/tidybot.gazebo.xacro (robot description, xacro)
@@ -50,5 +50,5 @@
   <xacro:include filename="$(find tidybot_description)/urdf/arms/${arm}/${arm}_transmission.xacro" />
   <xacro:load_arm_transmission prefix="${prefix}" />
-  <xacro:include filename="$(find tidybot_description)/urdf/base/base_transmission.xacro" />
+  <xacro:include filename="$(find tidybot_description)/urdf/base/tidybot++/base_kinova_transmission.xacro" />
   <xacro:load_base_transmission prefix="${prefix}" />
 </xacro:macro>

Commit message: add base camera to the simulation

File: src/tidybot_description/urdf/arms/gen3_7dof/gen3_7dof_macro.xacro (robot description, xacro)
@@ -341,9 +341,9 @@
     </joint>
     <xacro:if value="${vision}">
-      <link name="${prefix}camera_link" />
+      <link name="${prefix}arm_camera_link" />
       <joint name="${prefix}camera_module" type="fixed">
         <origin xyz="0 0.05639 -0.00305" rpy="3.14159265358979 3.14159265358979 0" />
         <parent link="${prefix}end_effector_link" />
-        <child  link="${prefix}camera_link" />
+        <child  link="${prefix}arm_camera_link" />
       </joint>
       <link name="${prefix}camera_depth_frame" />

File: src/tidybot_description/urdf/base/tidybot++/base_kinova_macro.xacro (robot description, xacro)
@@ -2,5 +2,5 @@
 <robot name="tidybot_base" xmlns:xacro="http://ros.org/wiki/xacro">
     <xacro:property name="last_base_link" value="base"/>
-    <xacro:macro name="load_base" params="parent:='' prefix">
+    <xacro:macro name="load_base" params="parent:='' prefix vision">
         <link name="world"></link>
         <link name="${prefix}base">
@@ -12,5 +12,5 @@
             <!-- Part kinova -->
             <visual>
-                <origin xyz="-0.3066 0.064 0.085" rpy="0 -0 0"/>
+                <origin xyz="-0.3066 0.06523 0.085" rpy="0 -0 0"/>
                 <geometry>
                     <mesh filename="file://$(find tidybot_description)/meshes/base/tidybot++/Kinova.stl"/>
@@ -21,5 +21,5 @@
             </visual>
             <collision>
-                <origin xyz="-0.3066 0.064 0.085" rpy="0 -0 0"/>
+                <origin xyz="-0.3066 0.06523 0.085" rpy="0 -0 0"/>
                 <geometry>
                     <mesh filename="file://$(find tidybot_description)/meshes/base/tidybot++/Kinova.stl"/>
@@ -27,4 +27,21 @@
             </collision>
         </link>
+        <xacro:if value="${vision}">
+            <link name="${prefix}base_camera_link" />
+            <joint type="fixed" name="${prefix}base_camera_joint">
+                <origin xyz="0.2285 0.0 0.315" rpy="0.0 1.57079632679 0.0"/>
+                <parent link="${prefix}base"/>
+                <child link="${prefix}base_camera_link"/>
+                <visual>
+                    <origin xyz="0.2285 0.0 0.315" rpy="0.0 0.0 0.0"/>
+                    <geometry>
+                        <box size="0.1 0.1 0.1"/>
+                    </geometry>
+                    <material name="red">
+                        <color rgba="1 0 0 1"/>
+                    </material>
+                </visual>
+            </joint>
+        </xacro:if>
         <link name="joint_x_jointbody">
             <inertial>

File: src/tidybot_description/urdf/bot.xacro (robot description, xacro)
@@ -7,5 +7,5 @@
     <xacro:include filename="$(find tidybot_description)/urdf/base/tidybot++/base_kinova_macro.xacro" />
     <!-- load the base -->
-    <xacro:load_base parent="" prefix="${prefix}" />
+    <xacro:load_base parent="" prefix="${prefix}" vision="${vision}" />
     <!-- load the arm -->
     <xacro:load_arm parent="${last_base_link}" vision="${vision}" prefix="${prefix}">

File: src/tidybot_description/urdf/tidybot.gazebo.xacro (robot description, xacro)
@@ -20,12 +20,39 @@
   </gazebo> -->
   <xacro:if value="${vision}">
-    <gazebo reference="${prefix}camera_link">
-      <sensor name="${prefix}camera" type="rgbd_camera">
+    <gazebo reference="${prefix}arm_camera_link">
+      <sensor name="${prefix}arm_camera" type="rgbd_camera">
         <always_on>1</always_on>
         <update_rate>30</update_rate>
         <visualize>true</visualize>
         <pose>0 -0.01 0.03 0 4.7124 1.5708</pose>
-				<topic>/camera</topic>
-        <gz_frame_id>${prefix}camera_link</gz_frame_id>
+				<topic>/arm_camera</topic>
+        <gz_frame_id>${prefix}arm_camera_link</gz_frame_id>
+        <camera>
+          <horizontal_fov>1.047</horizontal_fov>
+          <image>
+            <width>640</width>
+            <height>480</height>
+            <format>R8G8B8</format>
+          </image>
+          <clip>
+            <near>0.03</near>
+            <far>3.0</far>
+          </clip>
+          <noise>
+            <type>gaussian</type>
+            <mean>0.0</mean>
+            <stddev>0.007</stddev>
+          </noise>
+        </camera>
+      </sensor>
+    </gazebo>
+    <gazebo reference="${prefix}base_camera_link">
+      <sensor name="${prefix}base_camera" type="rgbd_camera">
+        <always_on>1</always_on>
+        <update_rate>30</update_rate>
+        <visualize>true</visualize>
+        <pose>0 0 0 0 4.7124 0</pose>
+				<topic>/base_camera</topic>
+        <gz_frame_id>${prefix}base_camera_link</gz_frame_id>
         <camera>
           <horizontal_fov>1.047</horizontal_fov>

File: src/tidybot_description/urdf/tidybot.xacro (robot description, xacro)
@@ -16,4 +16,4 @@
     <!-- load gazebo plugins -->
     <xacro:include filename="$(find tidybot_description)/urdf/tidybot.gazebo.xacro" />
-    <xacro:load_gazebo_plugins config_path="$(arg ros2_control_config_path)" prefix="$(arg prefix) " arm="$(arg arm)" vision="$(arg vision)" />
+    <xacro:load_gazebo_plugins config_path="$(arg ros2_control_config_path)" prefix="$(arg prefix)" arm="$(arg arm)" vision="$(arg vision)" />
 </robot>

Commit message: update the urdf and add fetch_cube demo

File: src/tidybot_description/urdf/arms/gen3_7dof/gen3_7dof_macro.xacro (robot description, xacro)
@@ -343,5 +343,5 @@
       <link name="${prefix}arm_camera_link" />
       <joint name="${prefix}camera_module" type="fixed">
-        <origin xyz="0 0.05639 -0.00305" rpy="3.14159265358979 3.14159265358979 0" />
+        <origin xyz="0 0.05639 -0.00405" rpy="3.14159265358979 3.14159265358979 0" />
         <parent link="${prefix}end_effector_link" />
         <child  link="${prefix}arm_camera_link" />

File: src/tidybot_description/urdf/tidybot.gazebo.xacro (robot description, xacro)
@@ -28,5 +28,5 @@
         <gz_frame_id>${prefix}arm_camera_link</gz_frame_id>
         <camera>
-          <horizontal_fov>1.047</horizontal_fov>
+          <horizontal_fov>1.147</horizontal_fov>
           <image>
             <width>640</width>

Commit message: add tidybot pretrained policy demo

File: src/tidybot_description/urdf/arms/gen3_7dof/gen3_7dof_macro.xacro (robot description, xacro)
@@ -5,5 +5,5 @@
   <xacro:macro name="load_arm" params="parent:='' vision prefix *origin">
     <joint name="${prefix}arm_base_joint" type="fixed">
-      <origin xyz="0.12 3.76986e-15 0.374775" rpy="0 0 0" />
+      <origin xyz="0 0 0.33" rpy="0 0 0" />
       <parent link="${parent}" />
       <child link="${prefix}arm_base_link" />

File: src/tidybot_description/urdf/base/tidybot/base_macro.xacro (robot description, xacro)
@@ -2,5 +2,5 @@
 <robot name="tidybot_base" xmlns:xacro="http://ros.org/wiki/xacro">
     <xacro:property name="last_base_link" value="base"/>
-    <xacro:macro name="load_base" params="parent:='' prefix">
+    <xacro:macro name="load_base" params="parent:='' prefix vision">
         <link name="world"></link>
         <link name="${prefix}base">
@@ -15,5 +15,5 @@
                     <mesh filename="file://$(find tidybot_description)/meshes/base/tidybot/bumper.stl"/>
                 </geometry>
-                <material name="white"/>
+                <material name="grey"/>
             </visual>
             <collision name="bumper">
@@ -28,5 +28,5 @@
                     <mesh filename="file://$(find tidybot_description)/meshes/base/tidybot/bottom_plate.stl"/>
                 </geometry>
-                <material name="white"/>
+                <material name="grey"/>
             </visual>
             <collision name="bottom_plate">
@@ -41,5 +41,5 @@
                     <mesh filename="file://$(find tidybot_description)/meshes/base/tidybot/body.stl"/>
                 </geometry>
-                <material name="white"/>
+                <material name="grey"/>
             </visual>
             <collision name="body">
@@ -54,5 +54,5 @@
                     <mesh filename="file://$(find tidybot_description)/meshes/base/tidybot/top_plate.stl"/>
                 </geometry>
-                <material name="white"/>
+                <material name="grey"/>
             </visual>
             <collision name="top_plate">
@@ -67,5 +67,5 @@
                     <mesh filename="file://$(find tidybot_description)/meshes/base/tidybot/arm_plate.stl"/>
                 </geometry>
-                <material name="white"/>
+                <material name="grey"/>
             </visual>
             <collision name="arm_plate">
@@ -76,4 +76,21 @@
             </collision>
         </link>
+        <xacro:if value="${vision}">
+            <link name="${prefix}base_camera_link" />
+            <joint type="fixed" name="${prefix}base_camera_joint">
+                <origin xyz="0.2525 0.0 0.315" rpy="0 0.7853981634 0"/>
+                <parent link="${prefix}base"/>
+                <child link="${prefix}base_camera_link"/>
+                <visual>
+                    <origin xyz="0.2285 0.0 0.315" rpy="0 0 0"/>
+                    <geometry>
+                        <box size="0.1 0.1 0.1"/>
+                    </geometry>
+                    <material name="red">
+                        <color rgba="1 0 0 1"/>
+                    </material>
+                </visual>
+            </joint>
+        </xacro:if>
         <link name="joint_x_jointbody">
             <inertial>
@@ -128,6 +145,6 @@
             <limit lower="0.0" upper="0.0" effort="100" velocity="100"/>
         </joint>
-        <material name="white">
-            <color rgba="1 1 1 1"/>
+        <material name="grey">
+            <color rgba="0.5 0.5 0.5 1"/>
         </material>
     </xacro:macro>

File: src/tidybot_description/urdf/bot.xacro (robot description, xacro)
@@ -5,5 +5,5 @@
     <xacro:include filename="$(find tidybot_description)/urdf/arms/${arm}/${arm}_macro.xacro" />
     <xacro:include filename="$(find tidybot_description)/urdf/grippers/${gripper}/${gripper}_macro.xacro" />
-    <xacro:include filename="$(find tidybot_description)/urdf/base/tidybot++/base_kinova_macro.xacro" />
+    <xacro:include filename="$(find tidybot_description)/urdf/base/tidybot/base_macro.xacro" />
     <!-- load the base -->
     <xacro:load_base parent="" prefix="${prefix}" vision="${vision}" />

File: src/tidybot_description/urdf/tidybot.gazebo.xacro (robot description, xacro)
@@ -76,5 +76,5 @@
   <xacro:include filename="$(find tidybot_description)/urdf/arms/${arm}/${arm}_transmission.xacro" />
   <xacro:load_arm_transmission prefix="${prefix}" />
-  <xacro:include filename="$(find tidybot_description)/urdf/base/tidybot++/base_kinova_transmission.xacro" />
+  <xacro:include filename="$(find tidybot_description)/urdf/base/tidybot/base_transmission.xacro" />
   <xacro:load_base_transmission prefix="${prefix}" />
   <xacro:include filename="$(find tidybot_description)/urdf/grippers/robotiq_2f_85/robotiq_2f_85_transmission.xacro" />

File: src/tidybot_description/urdf/tidybot.ros2_control.xacro (robot description, xacro)
@@ -26,5 +26,5 @@
         <xacro:add_joint name="joint_3" gain="0.1" cmd_interface="position" init_pos="3.141522"/>
         <xacro:add_joint name="joint_4" gain="0.1" cmd_interface="position" init_pos="-2.548368"/>
-        <xacro:add_joint name="joint_5" gain="0.1" cmd_interface="position" init_pos="-3.195793"/>
+        <xacro:add_joint name="joint_5" gain="0.1" cmd_interface="position" init_pos="-3.131593"/>
         <xacro:add_joint name="joint_6" gain="0.1" cmd_interface="position" init_pos="0.872947"/>
         <xacro:if value="${arm == 'gen3_7dof'}">

Commit message: update joystick control and REAME files

File: src/tidybot_description/urdf/arms/gen3_7dof/gen3_7dof_macro.xacro (robot description, xacro)
@@ -5,5 +5,5 @@
   <xacro:macro name="load_arm" params="parent:='' vision prefix *origin">
     <joint name="${prefix}arm_base_joint" type="fixed">
-      <origin xyz="0.12 3.76986e-15 0.374775" rpy="0 0 0" />
+      <xacro:insert_block name="origin"/>
       <parent link="${parent}" />
       <child link="${prefix}arm_base_link" />

File: src/tidybot_description/urdf/bot.xacro (robot description, xacro)
@@ -10,5 +10,5 @@
     <!-- load the arm -->
     <xacro:load_arm parent="${last_base_link}" vision="${vision}" prefix="${prefix}">
-        <origin xyz="0 0 0" rpy="0 0 0" />
+        <origin xyz="0.12 3.76986e-15 0.374775" rpy="0 0 0" />
     </xacro:load_arm>
     <!-- load the gripper -->

File: src/tidybot_description/urdf/tidybot.ros2_control.xacro (robot description, xacro)
@@ -20,11 +20,11 @@
         <xacro:add_joint name="joint_th" gain="0.1" cmd_interface="${base_mode}" init_pos="0.0"/>
         <xacro:add_joint name="joint_1" gain="0.1" cmd_interface="position" init_pos="0.0"/>
-        <xacro:add_joint name="joint_2" gain="0.1" cmd_interface="position" init_pos="-0.348927"/>
+        <xacro:add_joint name="joint_2" gain="0.1" cmd_interface="position" init_pos="-0.35"/>
         <xacro:add_joint name="joint_3" gain="0.1" cmd_interface="position" init_pos="3.141522"/>
-        <xacro:add_joint name="joint_4" gain="0.1" cmd_interface="position" init_pos="-2.548368"/>
-        <xacro:add_joint name="joint_5" gain="0.1" cmd_interface="position" init_pos="-3.195793"/>
-        <xacro:add_joint name="joint_6" gain="0.1" cmd_interface="position" init_pos="0.872947"/>
-        <xacro:if value="${arm == 'gen3_7dof'}">
-            <xacro:add_joint name="joint_7" gain="0.1" cmd_interface="position" init_pos="-1.574186"/>
+        <xacro:add_joint name="joint_4" gain="0.1" cmd_interface="position" init_pos="-2.36"/>
+        <xacro:add_joint name="joint_5" gain="0.1" cmd_interface="position" init_pos="0.0"/>
+        <xacro:add_joint name="joint_6" gain="0.1" cmd_interface="position" init_pos="-1.13"/>
+        <xacro:if value="${'$(arg arm)' == 'gen3_7dof'}">
+            <xacro:add_joint name="joint_7" gain="0.1" cmd_interface="position" init_pos="1.574186"/>
         </xacro:if>
         <xacro:if value="${gripper == 'gen3_lite_2f'}">

Commit message: Remove camera_depth and camera_color frame from robot description (published by ros2_kortex_vision)

File: src/tidybot_description/urdf/arms/gen3_7dof/gen3_7dof_macro.xacro (robot description, xacro)
@@ -341,21 +341,9 @@
     </joint>
     <xacro:if value="${vision}">
-      <link name="${prefix}arm_camera_link" />
-      <joint name="${prefix}camera_module" type="fixed">
-        <origin xyz="0 0.05639 -0.00405" rpy="3.14159265358979 3.14159265358979 0" />
+      <link name="${prefix}camera_link" />
+      <joint name="${prefix}camera_mount_joint" type="fixed">
+        <origin xyz="0 0.05639 -0.00405" rpy="${pi} ${pi} 0" />
         <parent link="${prefix}end_effector_link" />
-        <child  link="${prefix}arm_camera_link" />
-      </joint>
-      <link name="${prefix}camera_depth_frame" />
-      <joint name="${prefix}depth_module" type="fixed">
-        <origin xyz="0.0275 0.066 -0.00305" rpy="3.14159265358979 3.14159265358979 0" />
-        <parent link="${prefix}end_effector_link" />
-        <child  link="${prefix}camera_depth_frame" />
-      </joint>
-      <link name="${prefix}camera_color_frame" />
-      <joint name="${prefix}color_module" type="fixed">
-        <origin xyz="0 0.05639 -0.00305" rpy="3.14159265358979 3.14159265358979 0" />
-        <parent link="${prefix}end_effector_link" />
-        <child  link="${prefix}camera_color_frame" />
+        <child  link="${prefix}camera_link" />
       </joint>
     </xacro:if>
